Commit message: Update configuration and URDF files for Rizon robot

File: urdf/common/rizon_common.xacro (robot description, xacro)
@@ -13,5 +13,6 @@
         <origin xyz="0 0 0" rpy="0 0 0" />
         <geometry>
-          <mesh filename="package://${shell_config.mesh.package}/${shell_config.mesh.path}" />
+          <mesh
+            filename="package://${shell_config['mesh']['package']}/${shell_config['mesh']['path']}" />
         </geometry>
       </visual>
@@ -21,10 +22,10 @@
         <xacro:property name="ring_config" value="${visual_config['ring']}" lazy_eval="false" />
         <origin
-          xyz="${ring_config.origin.x} ${ring_config.origin.y} ${ring_config.origin.z}"
-          rpy="${ring_config.origin.roll} ${ring_config.origin.pitch} ${ring_config.origin.yaw}" />
+          xyz="${ring_config['origin']['x']} ${ring_config['origin']['y']} ${ring_config['origin']['z']}"
+          rpy="${ring_config['origin']['roll']} ${ring_config['origin']['pitch']} ${ring_config['origin']['yaw']}" />
         <geometry>
           <mesh
-            filename="package://${ring_config.mesh.package}/${ring_config.mesh.path}"
-            scale="${ring_config.mesh.scale}" />
+            filename="package://${ring_config['mesh']['package']}/${ring_config['mesh']['path']}"
+            scale="${ring_config['mesh']['scale']}" />
         </geometry>
       </visual>
@@ -42,5 +43,5 @@
       <geometry>
         <mesh
-          filename="package://${collision_config.mesh.package}/${collision_config.mesh.path}" />
+          filename="package://${collision_config['mesh']['package']}/${collision_config['mesh']['path']}" />
       </geometry>
     </collision>
@@ -52,8 +53,9 @@
   <xacro:macro name="get_joint_limits" params="name">
     <xacro:property name="limits" value="${sec_joint_limits[name]}" lazy_eval="false" />
-    <limit lower="${limits.lower}" upper="${limits.upper}" effort="${limits.effort}"
-      velocity="${limits.velocity}" />
-    <safety_controller k_position="100.0" k_velocity="40.0" soft_lower_limit="${limits.soft_lower}"
-      soft_upper_limit="${limits.soft_upper}" />
+    <limit lower="${limits['lower']}" upper="${limits['upper']}" effort="${limits['effort']}"
+      velocity="${limits['velocity']}" />
+    <safety_controller k_position="100.0" k_velocity="40.0"
+      soft_lower_limit="${limits['soft_lower']}"
+      soft_upper_limit="${limits['soft_upper']}" />
   </xacro:macro>
   <!--
@@ -63,6 +65,6 @@
   <xacro:macro name="get_kinematics" params="name">
     <xacro:property name="kinematics" value="${sec_kinematics[name]}" lazy_eval="false" />
-    <origin xyz="${kinematics.x} ${kinematics.y} ${kinematics.z}"
-      rpy="${kinematics.roll} ${kinematics.pitch} ${kinematics.yaw}" />
+    <origin xyz="${kinematics['x']} ${kinematics['y']} ${kinematics['z']}"
+      rpy="${kinematics['roll']} ${kinematics['pitch']} ${kinematics['yaw']}" />
   </xacro:macro>
   <!--
@@ -72,10 +74,11 @@
   <xacro:macro name="get_inertias" params="name">
     <xacro:property name="inertias" value="${sec_inertia_parameters[name]}" lazy_eval="false" />
-    <origin xyz="${inertias.origin.x} ${inertias.origin.y} ${inertias.origin.z}"
-      rpy="${inertias.origin.roll} ${inertias.origin.pitch} ${inertias.origin.yaw}" />
-    <mass value="${inertias.mass}" />
-    <inertia ixx="${inertias.inertia.ixx}" ixy="${inertias.inertia.ixy}"
-      ixz="${inertias.inertia.ixz}" iyy="${inertias.inertia.iyy}" iyz="${inertias.inertia.iyz}"
-      izz="${inertias.inertia.izz}" />
+    <origin xyz="${inertias['origin']['x']} ${inertias['origin']['y']} ${inertias['origin']['z']}"
+      rpy="${inertias['origin']['roll']} ${inertias['origin']['pitch']} ${inertias['origin']['yaw']}" />
+    <mass value="${inertias['mass']}" />
+    <inertia ixx="${inertias['inertia']['ixx']}" ixy="${inertias['inertia']['ixy']}"
+      ixz="${inertias['inertia']['ixz']}" iyy="${inertias['inertia']['iyy']}"
+      iyz="${inertias['inertia']['iyz']}"
+      izz="${inertias['inertia']['izz']}" />
   </xacro:macro>
   <!--

File: urdf/common/rizon_robot.xacro (robot description, xacro)
@@ -26,5 +26,5 @@
     <!-- Load gripper -->
     <xacro:if value="${load_gripper and gripper_name=='Flexiv-GN01'}">
-      <xacro:include filename="$(find flexiv_description)/urdf/grav_macro.xacro" />
+      <xacro:include filename="$(find flexiv_description)/urdf/common/grav_macro.xacro" />
       <xacro:flexiv_GN01 prefix="${prefix}" mesh_prefix_path="package://flexiv_description/" />
     </xacro:if>

File: urdf/rizon.urdf.xacro (robot description, xacro)
@@ -8,19 +8,34 @@
   <xacro:arg name="arm_prefix" default="" />
   <xacro:arg name="robot_sn" default="" />
-  <xacro:arg name="rdk_control_mode" default="joint_position" />
+  <xacro:arg name="joint_limits_parameters_file"
+    default="$(find flexiv_description)/config/$(arg rizon_type)/joint_limits.yaml" />
+  <xacro:arg name="kinematics_parameters_file"
+    default="$(find flexiv_description)/config/$(arg rizon_type)/default_kinematics.yaml" />
+  <xacro:arg name="inertia_parameters_file"
+    default="$(find flexiv_description)/config/$(arg rizon_type)/inertia_parameters.yaml" />
+  <xacro:arg name="visual_parameters_file"
+    default="$(find flexiv_description)/config/$(arg rizon_type)/visual_parameters.yaml" />
   <xacro:arg name="load_gripper" default="false" />
   <xacro:arg name="gripper_name" default="Flexiv-GN01" />
   <xacro:arg name="load_mounted_ft_sensor" default="false" />
+  <!-- ros2_control related parameters -->
+  <xacro:arg name="ros2_control" default="false" />
+  <xacro:arg name="rdk_control_mode" default="joint_position" />
   <xacro:arg name="use_fake_hardware" default="false" />
   <xacro:arg name="fake_sensor_commands" default="false" />
   <xacro:rizon_robot
     rizon_type="$(arg rizon_type)"
+    robot_sn="$(arg robot_sn)"
+    joint_limits_parameters_file="$(arg joint_limits_parameters_file)"
+    kinematics_parameters_file="$(arg kinematics_parameters_file)"
+    inertia_parameters_file="$(arg inertia_parameters_file)"
+    visual_parameters_file="$(arg visual_parameters_file)"
     arm_prefix="$(arg arm_prefix)"
-    robot_sn="$(arg robot_sn)"
-    rdk_control_mode="$(arg rdk_control_mode)"
     load_gripper="$(arg load_gripper)"
     gripper_name="$(arg gripper_name)"
+    load_mounted_ft_sensor="$(arg load_mounted_ft_sensor)"
+    ros2_control="$(arg ros2_control)"
+    rdk_control_mode="$(arg rdk_control_mode)"
     use_fake_hardware="$(arg use_fake_hardware)"
-    load_mounted_ft_sensor="$(arg load_mounted_ft_sensor)"
     fake_sensor_commands="$(arg fake_sensor_commands)">
   </xacro:rizon_robot>
