Commit message: Refactor rizon_robot.xacro to conditionally set prefix and update rizon.urdf.xacro to use rizon_type argument for robot name

File: urdf/common/rizon_robot.xacro (robot description, xacro)
@@ -19,5 +19,5 @@
     ">
     <!-- Prefix defaults to 'arm_prefix_robot_sn' -->
-    <xacro:property name="prefix" value="${arm_prefix + robot_sn + '_'}" />
+    <xacro:property name="prefix" value="${(arm_prefix + robot_sn + '_') if (arm_prefix + robot_sn) != '' else ''}" />
     <!-- FT sensor mounting only supported for Rizon4, Rizon4R and Rizon10 -->
     <xacro:unless value="${rizon_type=='Rizon4' or rizon_type=='Rizon4R' or rizon_type=='Rizon10'}">

File: urdf/rizon.urdf.xacro (robot description, xacro)
@@ -1,4 +1,4 @@
 <?xml version="1.0" encoding="utf-8"?>
-<robot xmlns:xacro="http://www.ros.org/wiki/xacro" name="rizon">
+<robot xmlns:xacro="http://www.ros.org/wiki/xacro" name="$(arg rizon_type)">
   <!-- 'rizon_type' values: Rizon4, Rizon4s, Rizon4M, Rizon4R, Rizon10, Rizon10s -->
   <xacro:arg name="rizon_type" default="Rizon4" />

Commit message: Refactor URDF file naming convention to prepend arm prefix and improve prefix property logic in Xacro

File: urdf/common/rizon_robot.xacro (robot description, xacro)
@@ -19,5 +19,6 @@
     ">
     <!-- Prefix defaults to 'arm_prefix_robot_sn' -->
-    <xacro:property name="prefix" value="${(arm_prefix + robot_sn + '_') if (arm_prefix + robot_sn) != '' else ''}" />
+    <xacro:property name="prefix"
+      value="${(arm_prefix + '_' + robot_sn + '_') if arm_prefix != '' and robot_sn != '' else (arm_prefix + robot_sn + '_') if (arm_prefix + robot_sn) != '' else ''}" />
     <!-- FT sensor mounting only supported for Rizon4, Rizon4R and Rizon10 -->
     <xacro:unless value="${rizon_type=='Rizon4' or rizon_type=='Rizon4R' or rizon_type=='Rizon10'}">
