Commit message: Add dual arm setup with initial positions and launch configuration

File: urdf/common/rizon.ros2_control.xacro (robot description, xacro)
@@ -8,5 +8,7 @@
     use_fake_hardware:=false
     fake_sensor_commands:=false
+    initial_positions_file
     ">
+    <xacro:property name="initial_positions" value="${xacro.load_yaml(initial_positions_file)['initial_positions']}"/>
     <ros2_control name="FlexivHardwareInterface" type="system">
       <hardware>
@@ -28,5 +30,5 @@
         <command_interface name="effort" />
         <state_interface name="position">
-          <param name="initial_value">0.0</param>
+          <param name="initial_value">${initial_positions['joint1']}</param>
         </state_interface>
         <state_interface name="velocity" />
@@ -38,5 +40,5 @@
         <command_interface name="effort" />
         <state_interface name="position">
-          <param name="initial_value">-0.69813</param>
+          <param name="initial_value">${initial_positions['joint2']}</param>
         </state_interface>
         <state_interface name="velocity" />
@@ -48,5 +50,5 @@
         <command_interface name="effort" />
         <state_interface name="position">
-          <param name="initial_value">0.0</param>
+          <param name="initial_value">${initial_positions['joint3']}</param>
         </state_interface>
         <state_interface name="velocity" />
@@ -58,5 +60,5 @@
         <command_interface name="effort" />
         <state_interface name="position">
-          <param name="initial_value">1.570796</param>
+          <param name="initial_value">${initial_positions['joint4']}</param>
         </state_interface>
         <state_interface name="velocity" />
@@ -68,5 +70,5 @@
         <command_interface name="effort" />
         <state_interface name="position">
-          <param name="initial_value">0.0</param>
+          <param name="initial_value">${initial_positions['joint5']}</param>
         </state_interface>
         <state_interface name="velocity" />
@@ -78,5 +80,5 @@
         <command_interface name="effort" />
         <state_interface name="position">
-          <param name="initial_value">0.69813</param>
+          <param name="initial_value">${initial_positions['joint6']}</param>
         </state_interface>
         <state_interface name="velocity" />
@@ -88,5 +90,5 @@
         <command_interface name="effort" />
         <state_interface name="position">
-          <param name="initial_value">0.0</param>
+          <param name="initial_value">${initial_positions['joint7']}</param>
         </state_interface>
         <state_interface name="velocity" />

File: urdf/common/rizon_arm.xacro (robot description, xacro)
@@ -10,4 +10,5 @@
     visual_parameters_file
     load_mounted_ft_sensor:=false
+    add_world_link:=true
     ">
     <!-- Load configuration data from the YAML files -->
@@ -88,6 +89,8 @@
     </joint>
     <!-- LINKS -->
-    <link name="world">
-    </link>
+    <xacro:if value="${add_world_link}">
+      <link name="world">
+      </link>
+    </xacro:if>
     <link name="${prefix}base_link">
       <xacro:get_inertias name="base_link" />

File: urdf/common/rizon_robot.xacro (robot description, xacro)
@@ -17,4 +17,6 @@
     use_fake_hardware:=false
     fake_sensor_commands:=false
+    add_world_link:=true
+    initial_positions_file:='$(find flexiv_description)/config/initial_positions.yaml'
     ">
     <!-- Prefix defaults to 'arm_prefix_robot_sn' -->
@@ -37,4 +39,5 @@
       inertia_parameters_file="${inertia_parameters_file}"
       visual_parameters_file="${visual_parameters_file}"
+      add_world_link="${add_world_link}"
     />
     <xacro:if value="${ros2_control}">
@@ -45,4 +48,5 @@
         use_fake_hardware="${use_fake_hardware}"
         fake_sensor_commands="${fake_sensor_commands}"
+        initial_positions_file="${initial_positions_file}"
       />
     </xacro:if>

File: urdf/rizon.urdf.xacro (robot description, xacro)
@@ -24,4 +24,5 @@
   <xacro:arg name="use_fake_hardware" default="false" />
   <xacro:arg name="fake_sensor_commands" default="false" />
+  <xacro:arg name="initial_positions_file" default="$(find flexiv_description)/config/initial_positions.yaml" />
   <xacro:rizon_robot
     rizon_type="$(arg rizon_type)"
@@ -38,5 +39,6 @@
     rdk_control_mode="$(arg rdk_control_mode)"
     use_fake_hardware="$(arg use_fake_hardware)"
-    fake_sensor_commands="$(arg fake_sensor_commands)">
+    fake_sensor_commands="$(arg fake_sensor_commands)"
+    initial_positions_file="$(arg initial_positions_file)">
   </xacro:rizon_robot>
 </robot>
