Commit message: Remove deprecated URDF files for Rizon4 and Rizon4R robot models, consolidating joint and link definitions to streamline the robot description.

File: urdf/common/rizon_arm.xacro (robot description, xacro)
@@ -94,10 +94,5 @@
       <xacro:get_visuals name="base_link" />
       <xacro:get_collisions name="base_link" />
-      <workspace>
-        <origin rpy="0 0 0" xyz="0 0 0.365" />
-        <geometry>
-          <sphere radius="0.890" />
-        </geometry>
-      </workspace>
+      <xacro:get_workspace name="base_link" />
     </link>
     <link name="${prefix}link1">

File: urdf/common/rizon_common.xacro (robot description, xacro)
@@ -11,5 +11,12 @@
       <visual name="shell">
         <xacro:property name="shell_config" value="${visual_config['shell']}" lazy_eval="false" />
-        <origin xyz="0 0 0" rpy="0 0 0" />
+        <xacro:if value="${'origin' in shell_config}">
+          <origin
+            xyz="${shell_config['origin']['x']} ${shell_config['origin']['y']} ${shell_config['origin']['z']}"
+            rpy="${shell_config['origin']['roll']} ${shell_config['origin']['pitch']} ${shell_config['origin']['yaw']}" />
+        </xacro:if>
+        <xacro:unless value="${'origin' in shell_config}">
+          <origin xyz="0 0 0" rpy="0 0 0" />
+        </xacro:unless>
         <geometry>
           <mesh
@@ -40,5 +47,12 @@
       lazy_eval="false" />
     <collision name="convex_mesh">
-      <origin xyz="0 0 0" rpy="0 0 0" />
+      <xacro:if value="${'origin' in collision_config}">
+        <origin
+          xyz="${collision_config['origin']['x']} ${collision_config['origin']['y']} ${collision_config['origin']['z']}"
+          rpy="${collision_config['origin']['roll']} ${collision_config['origin']['pitch']} ${collision_config['origin']['yaw']}" />
+      </xacro:if>
+      <xacro:unless value="${'origin' in collision_config}">
+        <origin xyz="0 0 0" rpy="0 0 0" />
+      </xacro:unless>
       <geometry>
         <mesh
@@ -132,3 +146,21 @@
     </xacro:unless>
   </xacro:macro>
+  <!--
+    Extract workspace parameters from the config file
+    name: name of the link
+  -->
+  <xacro:macro name="get_workspace" params="name">
+    <xacro:if value="${'workspace' in sec_visual_parameters[name]}">
+      <xacro:property name="workspace_config" value="${sec_visual_parameters[name]['workspace']}"
+        lazy_eval="false" />
+      <workspace>
+        <origin
+          xyz="${workspace_config['origin']['x']} ${workspace_config['origin']['y']} ${workspace_config['origin']['z']}"
+          rpy="${workspace_config['origin']['roll']} ${workspace_config['origin']['pitch']} ${workspace_config['origin']['yaw']}" />
+        <geometry>
+          <sphere radius="${workspace_config['sphere']['radius']}" />
+        </geometry>
+      </workspace>
+    </xacro:if>
+  </xacro:macro>
 </robot>

Commit message: Add dual arm setup support with updated scripts and configurations

File: urdf/common/rizon_arm.xacro (robot description, xacro)
@@ -11,4 +11,6 @@
     load_mounted_ft_sensor:=false
     add_world_link:=true
+    base_xyz:='0.0 0.0 0.0'
+    base_rpy:='0.0 0.0 0.0'
     ">
     <!-- Load configuration data from the YAML files -->
@@ -27,5 +29,5 @@
       <parent link="world" />
       <child link="${prefix}base_link" />
-      <origin xyz="0.0 0.0 0.0" rpy="0.0 0.0 0.0" />
+      <origin xyz="${base_xyz}" rpy="${base_rpy}" />
     </joint>
     <joint name="${prefix}joint1" type="revolute">

File: urdf/common/rizon_dual.ros2_control.xacro (robot description, xacro)
@@ -12,4 +12,10 @@
     initial_positions_file_left
     initial_positions_file_right
+    translation_left_x:=0.0
+    translation_left_y:=0.0
+    translation_left_z:=0.0
+    translation_right_x:=0.0
+    translation_right_y:=0.0
+    translation_right_z:=0.0
     ">
     <xacro:property name="initial_positions_left" value="${xacro.load_yaml(initial_positions_file_left)['initial_positions']}"/>
@@ -29,4 +35,10 @@
           <param name="prefix_right">${prefix_right}</param>
           <param name="rdk_control_mode">${rdk_control_mode}</param>
+          <param name="translation_left_x">${translation_left_x}</param>
+          <param name="translation_left_y">${translation_left_y}</param>
+          <param name="translation_left_z">${translation_left_z}</param>
+          <param name="translation_right_x">${translation_right_x}</param>
+          <param name="translation_right_y">${translation_right_y}</param>
+          <param name="translation_right_z">${translation_right_z}</param>
         </xacro:unless>
       </hardware>

File: urdf/common/rizon_robot.xacro (robot description, xacro)
@@ -19,4 +19,6 @@
     add_world_link:=true
     initial_positions_file:='$(find flexiv_description)/config/initial_positions.yaml'
+    base_xyz:='0.0 0.0 0.0'
+    base_rpy:='0.0 0.0 0.0'
     ">
     <!-- Prefix defaults to 'arm_prefix_robot_sn' -->
@@ -40,4 +42,6 @@
       visual_parameters_file="${visual_parameters_file}"
       add_world_link="${add_world_link}"
+      base_xyz="${base_xyz}"
+      base_rpy="${base_rpy}"
     />
     <xacro:if value="${ros2_control}">

File: urdf/rizon_dual.urdf.xacro (robot description, xacro)
@@ -18,4 +18,5 @@
   <xacro:arg name="initial_positions_file_left" default="$(find flexiv_description)/config/left_initial_positions.yaml" />
   <xacro:arg name="initial_positions_file_right" default="$(find flexiv_description)/config/right_initial_positions.yaml" />
+  <xacro:arg name="translations_file" default="$(find flexiv_description)/config/dual_arm_translations.yaml" />
   <xacro:include filename="$(find flexiv_description)/urdf/common/rizon_robot.xacro" />
   <xacro:include filename="$(find flexiv_description)/urdf/common/rizon_dual.ros2_control.xacro" />
@@ -23,4 +24,5 @@
   <xacro:property name="prefix_left" value="left_$(arg robot_sn_left)_" />
   <xacro:property name="prefix_right" value="right_$(arg robot_sn_right)_" />
+  <xacro:property name="translations" value="${xacro.load_yaml('$(arg translations_file)')}" />
   <link name="world" />
   <!-- Left Robot -->
@@ -38,4 +40,6 @@
     ros2_control="false"
     add_world_link="false"
+    base_xyz="${translations['translations']['left']['x']} ${translations['translations']['left']['y']} ${translations['translations']['left']['z']}"
+    base_rpy="0 0 0"
   />
   <!-- Right Robot -->
@@ -53,4 +57,6 @@
     ros2_control="false"
     add_world_link="false"
+    base_xyz="${translations['translations']['right']['x']} ${translations['translations']['right']['y']} ${translations['translations']['right']['z']}"
+    base_rpy="0 0 0"
   />
   <!-- Dual ROS 2 Control -->
@@ -66,4 +72,10 @@
       initial_positions_file_left="$(arg initial_positions_file_left)"
       initial_positions_file_right="$(arg initial_positions_file_right)"
+      translation_left_x="${translations['translations']['left']['x']}"
+      translation_left_y="${translations['translations']['left']['y']}"
+      translation_left_z="${translations['translations']['left']['z']}"
+      translation_right_x="${translations['translations']['right']['x']}"
+      translation_right_y="${translations['translations']['right']['y']}"
+      translation_right_z="${translations['translations']['right']['z']}"
     />
   </xacro:if>

Commit message: Feature/Add Rizon Dual Arm Setup (#4)
* Add dual arm setup with initial positions and launch configuration
* Refactor launch configuration for dual arm setup to improve clarity and organization
* Add dual arm setup support with updated scripts and configurations

File: urdf/common/rizon_arm.xacro (robot description, xacro)
@@ -10,4 +10,7 @@
     visual_parameters_file
     load_mounted_ft_sensor:=false
+    add_world_link:=true
+    base_xyz:='0.0 0.0 0.0'
+    base_rpy:='0.0 0.0 0.0'
     ">
     <!-- Load configuration data from the YAML files -->
@@ -26,5 +29,5 @@
       <parent link="world" />
       <child link="${prefix}base_link" />
-      <origin xyz="0.0 0.0 0.0" rpy="0.0 0.0 0.0" />
+      <origin xyz="${base_xyz}" rpy="${base_rpy}" />
     </joint>
     <joint name="${prefix}joint1" type="revolute">
@@ -88,6 +91,8 @@
     </joint>
     <!-- LINKS -->
-    <link name="world">
-    </link>
+    <xacro:if value="${add_world_link}">
+      <link name="world">
+      </link>
+    </xacro:if>
     <link name="${prefix}base_link">
       <xacro:get_inertias name="base_link" />

File: urdf/common/rizon_robot.xacro (robot description, xacro)
@@ -17,4 +17,8 @@
     use_fake_hardware:=false
     fake_sensor_commands:=false
+    add_world_link:=true
+    initial_positions_file:='$(find flexiv_description)/config/initial_positions.yaml'
+    base_xyz:='0.0 0.0 0.0'
+    base_rpy:='0.0 0.0 0.0'
     ">
     <!-- Prefix defaults to 'arm_prefix_robot_sn' -->
@@ -37,4 +41,7 @@
       inertia_parameters_file="${inertia_parameters_file}"
       visual_parameters_file="${visual_parameters_file}"
+      add_world_link="${add_world_link}"
+      base_xyz="${base_xyz}"
+      base_rpy="${base_rpy}"
     />
     <xacro:if value="${ros2_control}">
@@ -45,4 +52,5 @@
         use_fake_hardware="${use_fake_hardware}"
         fake_sensor_commands="${fake_sensor_commands}"
+        initial_positions_file="${initial_positions_file}"
       />
     </xacro:if>

Commit message: Add launch files and URDF for AICO1 and AICO2

File: urdf/common/rizon_arm.xacro (robot description, xacro)
@@ -11,4 +11,5 @@
     load_mounted_ft_sensor:=false
     add_world_link:=true
+    create_base_joint:=true
     base_xyz:='0.0 0.0 0.0'
     base_rpy:='0.0 0.0 0.0'
@@ -26,9 +27,11 @@
     />
     <!-- JOINTS -->
-    <joint name="${prefix}base_joint" type="fixed">
-      <parent link="world" />
-      <child link="${prefix}base_link" />
-      <origin xyz="${base_xyz}" rpy="${base_rpy}" />
-    </joint>
+    <xacro:if value="${create_base_joint}">
+      <joint name="${prefix}base_joint" type="fixed">
+        <parent link="world" />
+        <child link="${prefix}base_link" />
+        <origin xyz="${base_xyz}" rpy="${base_rpy}" />
+      </joint>
+    </xacro:if>
     <joint name="${prefix}joint1" type="revolute">
       <parent link="${prefix}base_link" />

File: urdf/common/rizon_robot.xacro (robot description, xacro)
@@ -18,4 +18,5 @@
     fake_sensor_commands:=false
     add_world_link:=true
+    create_base_joint:=true
     initial_positions_file:='$(find flexiv_description)/config/initial_positions.yaml'
     base_xyz:='0.0 0.0 0.0'
@@ -42,4 +43,5 @@
       visual_parameters_file="${visual_parameters_file}"
       add_world_link="${add_world_link}"
+      create_base_joint="${create_base_joint}"
       base_xyz="${base_xyz}"
       base_rpy="${base_rpy}"
