Commit message: Update joint limits for AICO2-X1 platform in URDF file

File: urdf/common/aico2_platform_x1.xacro (robot description, xacro)
@@ -8,5 +8,5 @@
       <child link="${prefix}aico2_x1_link1" />
       <axis xyz="0 0 1" />
-      <limit lower="-3.14" upper="3.14" effort="165" velocity="1" />
+      <limit lower="-1.57" upper="1.57" effort="400" velocity="1.05" />
     </joint>
     <joint name="${prefix}aico2_x1_joint2" type="revolute">
