Commit message: Fix GPIO configuration for dual robot setup by adjusting digital IO ports count and structure

File: urdf/common/rizon_dual.ros2_control.xacro (robot description, xacro)
@@ -69,13 +69,16 @@
       <xacro:configure_joint joint_name="${prefix_right}joint6" initial_pos="${initial_positions_right['joint6']}" />
       <xacro:configure_joint joint_name="${prefix_right}joint7" initial_pos="${initial_positions_right['joint7']}" />
-      <!-- 36 digital IO ports (18 per robot) -->
-      <gpio name="dual_arm_gpio">
-        <xacro:macro name="loop_gpio" params="idx">
-          <command_interface name="digital_output_${idx}" />
-          <state_interface name="digital_input_${idx}" />
-          <xacro:if value="${idx &lt; 35}">
-            <xacro:loop_gpio idx="${idx+1}" />
-          </xacro:if>
-        </xacro:macro>
+      <!-- 18 digital IO ports per robot -->
+      <xacro:macro name="loop_gpio" params="idx">
+        <command_interface name="digital_output_${idx}" />
+        <state_interface name="digital_input_${idx}" />
+        <xacro:if value="${idx &lt; 17}">
+          <xacro:loop_gpio idx="${idx+1}" />
+        </xacro:if>
+      </xacro:macro>
+      <gpio name="${prefix_left}gpio">
+        <xacro:loop_gpio idx="0" />
+      </gpio>
+      <gpio name="${prefix_right}gpio">
         <xacro:loop_gpio idx="0" />
       </gpio>

Commit message: Add joint configuration macro for dual robot control

File: urdf/common/rizon_dual.ros2_control.xacro (robot description, xacro)
@@ -46,4 +46,16 @@
         </xacro:unless>
       </hardware>
+      <xacro:macro name="configure_joint" params="joint_name initial_pos">
+        <joint name="${joint_name}">
+          <command_interface name="position" />
+          <command_interface name="velocity" />
+          <command_interface name="effort" />
+          <state_interface name="position">
+            <param name="initial_value">${initial_pos}</param>
+          </state_interface>
+          <state_interface name="velocity" />
+          <state_interface name="effort" />
+        </joint>
+      </xacro:macro>
       <xacro:configure_joint joint_name="${prefix_left}joint1" initial_pos="${initial_positions_left['joint1']}" />
       <xacro:configure_joint joint_name="${prefix_left}joint2" initial_pos="${initial_positions_left['joint2']}" />

Commit message: Feature/Add AICO meshes and URDF (#9)

File: urdf/common/rizon_dual.ros2_control.xacro (robot description, xacro)
@@ -18,4 +18,7 @@
     translation_right_y:=0.0
     translation_right_z:=0.0
+    platform_name:=''
+    platform_type:=''
+    platform_prefix:=''
     ">
     <xacro:property name="initial_positions_left" value="${xacro.load_yaml(initial_positions_file_left)['initial_positions']}"/>
@@ -62,4 +65,51 @@
       <xacro:configure_joint joint_name="${prefix_left}joint6" initial_pos="${initial_positions_left['joint6']}" />
       <xacro:configure_joint joint_name="${prefix_left}joint7" initial_pos="${initial_positions_left['joint7']}" />
+      <!-- Platform joints -->
+      <xacro:if value="${platform_name == 'aico2'}">
+        <xacro:if value="${platform_type == 'X1'}">
+          <joint name="${platform_prefix}aico2_x1_joint1">
+            <command_interface name="position" />
+            <command_interface name="velocity" />
+            <command_interface name="effort" />
+            <state_interface name="position">
+              <param name="initial_value">0.0</param>
+            </state_interface>
+            <state_interface name="velocity" />
+            <state_interface name="effort" />
+          </joint>
+          <joint name="${platform_prefix}aico2_x1_joint2">
+            <command_interface name="position" />
+            <command_interface name="velocity" />
+            <command_interface name="effort" />
+            <state_interface name="position">
+              <param name="initial_value">0.0</param>
+            </state_interface>
+            <state_interface name="velocity" />
+            <state_interface name="effort" />
+          </joint>
+        </xacro:if>
+        <xacro:if value="${platform_type == 'X2'}">
+          <joint name="${platform_prefix}aico2_x2_joint1">
+            <command_interface name="position" />
+            <command_interface name="velocity" />
+            <command_interface name="effort" />
+            <state_interface name="position">
+              <param name="initial_value">0.0</param>
+            </state_interface>
+            <state_interface name="velocity" />
+            <state_interface name="effort" />
+          </joint>
+          <joint name="${platform_prefix}aico2_x2_joint2">
+            <command_interface name="position" />
+            <command_interface name="velocity" />
+            <command_interface name="effort" />
+            <state_interface name="position">
+              <param name="initial_value">0.0</param>
+            </state_interface>
+            <state_interface name="velocity" />
+            <state_interface name="effort" />
+          </joint>
+        </xacro:if>
+      </xacro:if>
       <xacro:configure_joint joint_name="${prefix_right}joint1" initial_pos="${initial_positions_right['joint1']}" />
       <xacro:configure_joint joint_name="${prefix_right}joint2" initial_pos="${initial_positions_right['joint2']}" />

File: urdf/common/rizon_robot.xacro (robot description, xacro)
@@ -18,7 +18,11 @@
     fake_sensor_commands:=false
     add_world_link:=true
+    create_base_joint:=true
     initial_positions_file:='$(find flexiv_description)/config/initial_positions.yaml'
     base_xyz:='0.0 0.0 0.0'
     base_rpy:='0.0 0.0 0.0'
+    platform_name:=''
+    platform_type:=''
+    platform_prefix:=''
     ">
     <!-- Prefix defaults to 'arm_prefix_robot_sn' -->
@@ -42,4 +46,5 @@
       visual_parameters_file="${visual_parameters_file}"
       add_world_link="${add_world_link}"
+      create_base_joint="${create_base_joint}"
       base_xyz="${base_xyz}"
       base_rpy="${base_rpy}"
@@ -53,4 +58,7 @@
         fake_sensor_commands="${fake_sensor_commands}"
         initial_positions_file="${initial_positions_file}"
+        platform_name="${platform_name}"
+        platform_type="${platform_type}"
+        platform_prefix="${platform_prefix}"
       />
     </xacro:if>
