Commit message: Rename AICO series name

File: urdf/common/aico1_4s_v1.xacro (robot description, xacro)
@@ -1,26 +1,26 @@
 <?xml version="1.0" encoding="utf-8"?>
 <robot xmlns:xacro="http://wiki.ros.org/xacro">
-  <xacro:macro name="aico1_platform_x1" params="prefix arm_prefix mesh_prefix_path">
-    <joint name="${prefix}aico1_x1_joint1" type="fixed">
+  <xacro:macro name="aico1_4s_v1" params="prefix arm_prefix mesh_prefix_path">
+    <joint name="${prefix}aico1_4s_v1_joint1" type="fixed">
       <origin xyz="0 0 0.768" rpy="0 0 0" />
-      <parent link="${prefix}aico1_x1_base_link" />
-      <child link="${prefix}aico1_x1_link1" />
+      <parent link="${prefix}aico1_4s_v1_base_link" />
+      <child link="${prefix}aico1_4s_v1_link1" />
       <axis xyz="0 0 1" />
       <limit lower="0" upper="0.3" effort="100" velocity="1" />
     </joint>
-    <joint name="${prefix}aico1_x1_joint2" type="revolute">
+    <joint name="${prefix}aico1_4s_v1_joint2" type="revolute">
       <origin xyz="0.1385 0.204 0.183" rpy="0 0 0" />
-      <parent link="${prefix}aico1_x1_link1" />
-      <child link="${prefix}aico1_x1_link2" />
+      <parent link="${prefix}aico1_4s_v1_link1" />
+      <child link="${prefix}aico1_4s_v1_link2" />
       <axis xyz="0 1 0" />
       <limit lower="0" upper="1.57" effort="365" velocity="1" />
     </joint>
-    <joint name="${prefix}aico1_x1_arm_adapter" type="fixed">
+    <joint name="${prefix}aico1_4s_v1_arm_adapter" type="fixed">
       <origin xyz="0.0037763 0.0 0.3214" rpy="1.5708 0 0" />
-      <parent link="${prefix}aico1_x1_link2" />
+      <parent link="${prefix}aico1_4s_v1_link2" />
       <child link="${arm_prefix}base_link" />
       <axis xyz="0 0 0" />
     </joint>
-    <link name="${prefix}aico1_x1_base_link">
+    <link name="${prefix}aico1_4s_v1_base_link">
       <inertial>
         <origin xyz="0.00266 0.000754 0.34" rpy="0 0 0" />
@@ -32,5 +32,5 @@
         <geometry>
           <mesh
-            filename="${mesh_prefix_path}meshes/AICO1-X1/visual/base_link.obj" />
+            filename="${mesh_prefix_path}meshes/AICO1-4s-V1/visual/base_link.obj" />
         </geometry>
         <material name="">
@@ -42,9 +42,9 @@
         <geometry>
           <mesh
-            filename="${mesh_prefix_path}meshes/AICO1-X1/collision/base_link.stl" />
+            filename="${mesh_prefix_path}meshes/AICO1-4s-V1/collision/base_link.stl" />
         </geometry>
       </collision>
     </link>
-    <link name="${prefix}aico1_x1_link1">
+    <link name="${prefix}aico1_4s_v1_link1">
       <inertial>
         <origin xyz="0.017 0.014 -0.075" rpy="0 0 0" />
@@ -56,5 +56,5 @@
         <geometry>
           <mesh
-            filename="${mesh_prefix_path}meshes/AICO1-X1/visual/rise_link.obj" />
+            filename="${mesh_prefix_path}meshes/AICO1-4s-V1/visual/rise_link.obj" />
         </geometry>
         <material name="">
@@ -66,5 +66,5 @@
         <geometry>
           <mesh
-            filename="${mesh_prefix_path}meshes/AICO1-X1/collision/rise_link_bottom.stl" />
+            filename="${mesh_prefix_path}meshes/AICO1-4s-V1/collision/rise_link_bottom.stl" />
         </geometry>
       </collision>
@@ -73,9 +73,9 @@
         <geometry>
           <mesh
-            filename="${mesh_prefix_path}meshes/AICO1-X1/collision/rise_link_top.stl" />
+            filename="${mesh_prefix_path}meshes/AICO1-4s-V1/collision/rise_link_top.stl" />
         </geometry>
       </collision>
     </link>
-    <link name="${prefix}aico1_x1_link2">
+    <link name="${prefix}aico1_4s_v1_link2">
       <inertial>
         <origin xyz="0.0303 -0.092 0.255" rpy="0 0 0" />
@@ -87,5 +87,5 @@
         <geometry>
           <mesh
-            filename="${mesh_prefix_path}meshes/AICO1-X1/visual/pitch_link.obj" />
+            filename="${mesh_prefix_path}meshes/AICO1-4s-V1/visual/pitch_link.obj" />
         </geometry>
         <material name="">
@@ -97,5 +97,5 @@
         <geometry>
           <mesh
-            filename="${mesh_prefix_path}meshes/AICO1-X1/collision/pitch_link.stl" />
+            filename="${mesh_prefix_path}meshes/AICO1-4s-V1/collision/pitch_link.stl" />
         </geometry>
       </collision>

File: urdf/common/aico1_4s_v2.xacro (robot description, xacro)
@@ -1,39 +1,39 @@
 <?xml version="1.0" encoding="utf-8"?>
 <robot xmlns:xacro="http://wiki.ros.org/xacro">
-  <xacro:macro name="aico1_platform_x2" params="prefix arm_prefix mesh_prefix_path">
-    <joint name="${prefix}aico1_x2_base_to_agv" type="fixed">
+  <xacro:macro name="aico1_4s_v2" params="prefix arm_prefix mesh_prefix_path">
+    <joint name="${prefix}aico1_4s_v2_base_to_agv" type="fixed">
       <origin xyz="0.004 0.1255 0.695" rpy="0.0 0.0 0.0" />
-      <parent link="${prefix}aico1_x2_agv" />
-      <child link="${prefix}aico1_x2_base_link" />
+      <parent link="${prefix}aico1_4s_v2_agv" />
+      <child link="${prefix}aico1_4s_v2_base_link" />
       <axis xyz="0 0 0" />
     </joint>
-    <joint name="${prefix}aico1_x2_joint1" type="revolute">
+    <joint name="${prefix}aico1_4s_v2_joint1" type="revolute">
       <origin xyz="-0.122 0.1066 0.164" rpy="0 0 0" />
-      <parent link="${prefix}aico1_x2_base_link" />
-      <child link="${prefix}aico1_x2_link1" />
+      <parent link="${prefix}aico1_4s_v2_base_link" />
+      <child link="${prefix}aico1_4s_v2_link1" />
       <axis xyz="0 1 0" />
       <limit lower="-0.523598775598" upper="1.57079632679" effort="1000"
         velocity="1" />
     </joint>
-    <joint name="${prefix}aico1_x2_joint2" type="revolute">
+    <joint name="${prefix}aico1_4s_v2_joint2" type="revolute">
       <origin xyz="-0.005 -0.0991 0.47875" rpy="0 0 0" />
-      <parent link="${prefix}aico1_x2_link1" />
-      <child link="${prefix}aico1_x2_neck_link" />
+      <parent link="${prefix}aico1_4s_v2_link1" />
+      <child link="${prefix}aico1_4s_v2_neck_link" />
       <axis xyz="0 0 1" />
       <limit lower="-1.57079632679" upper="1.57079632679" effort="50" velocity="1" />
     </joint>
-    <joint name="${prefix}aico1_x2_joint_head" type="revolute">
+    <joint name="${prefix}aico1_4s_v2_joint_head" type="revolute">
       <origin xyz="-0.025 0 0.088" rpy="0 0 0" />
-      <parent link="${prefix}aico1_x2_neck_link" />
-      <child link="${prefix}aico1_x2_head_link" />
+      <parent link="${prefix}aico1_4s_v2_neck_link" />
+      <child link="${prefix}aico1_4s_v2_head_link" />
       <axis xyz="0 1 0" />
       <limit lower="0" upper="0.436332312999" effort="80" velocity="1" />
     </joint>
-    <joint name="${prefix}aico1_x2_arm_adapter" type="fixed">
-      <parent link="${prefix}aico1_x2_link1" />
+    <joint name="${prefix}aico1_4s_v2_arm_adapter" type="fixed">
+      <parent link="${prefix}aico1_4s_v2_link1" />
       <child link="${arm_prefix}base_link" />
       <origin xyz="0.0 0.016 0.320" rpy="1.57079632679 0.0 0.0" />
     </joint>
-    <link name="${prefix}aico1_x2_agv">
+    <link name="${prefix}aico1_4s_v2_agv">
       <inertial>
         <origin xyz="0 0 0" rpy="0 0 0" />
@@ -45,5 +45,5 @@
         <geometry>
           <mesh
-            filename="${mesh_prefix_path}meshes/AICO1-X2/visual/agv.obj" />
+            filename="${mesh_prefix_path}meshes/AICO1-4s-V2/visual/agv.obj" />
         </geometry>
         <material name="">
@@ -55,9 +55,9 @@
         <geometry>
           <mesh
-            filename="${mesh_prefix_path}meshes/AICO1-X2/collision/agv.stl" />
+            filename="${mesh_prefix_path}meshes/AICO1-4s-V2/collision/agv.stl" />
         </geometry>
       </collision>
     </link>
-    <link name="${prefix}aico1_x2_base_link">
+    <link name="${prefix}aico1_4s_v2_base_link">
       <inertial>
         <origin xyz="-0.0372 -0.00251 0.0448" rpy="0 0 0" />
@@ -69,5 +69,5 @@
         <geometry>
           <mesh
-            filename="${mesh_prefix_path}meshes/AICO1-X2/visual/base_link.obj" />
+            filename="${mesh_prefix_path}meshes/AICO1-4s-V2/visual/base_link.obj" />
         </geometry>
         <material name="">
@@ -79,9 +79,9 @@
         <geometry>
           <mesh
-            filename="${mesh_prefix_path}meshes/AICO1-X2/collision/base_link.stl" />
+            filename="${mesh_prefix_path}meshes/AICO1-4s-V2/collision/base_link.stl" />
         </geometry>
       </collision>
     </link>
-    <link name="${prefix}aico1_x2_link1">
+    <link name="${prefix}aico1_4s_v2_link1">
       <inertial>
         <origin xyz="-0.00141 -0.0922 0.106" rpy="0 0 0" />
@@ -93,5 +93,5 @@
         <geometry>
           <mesh
-            filename="${mesh_prefix_path}meshes/AICO1-X2/visual/link1.obj" />
+            filename="${mesh_prefix_path}meshes/AICO1-4s-V2/visual/link1.obj" />
         </geometry>
         <material name="">
@@ -103,9 +103,9 @@
         <geometry>
           <mesh
-            filename="${mesh_prefix_path}meshes/AICO1-X2/collision/link1.stl" />
+            filename="${mesh_prefix_path}meshes/AICO1-4s-V2/collision/link1.stl" />
         </geometry>
       </collision>
     </link>
-    <link name="${prefix}aico1_x2_neck_link">
+    <link name="${prefix}aico1_4s_v2_neck_link">
       <inertial>
         <origin xyz="-0.0149 7E-07 0.0547" rpy="0 0 0" />
@@ -117,5 +117,5 @@
         <geometry>
           <mesh
-            filename="${mesh_prefix_path}meshes/AICO1-X2/visual/neck_link.obj" />
+            filename="${mesh_prefix_path}meshes/AICO1-4s-V2/visual/neck_link.obj" />
         </geometry>
         <material name="">
@@ -127,9 +127,9 @@
         <geometry>
           <mesh
-            filename="${mesh_prefix_path}meshes/AICO1-X2/collision/neck_link.stl" />
+            filename="${mesh_prefix_path}meshes/AICO1-4s-V2/collision/neck_link.stl" />
         </geometry>
       </collision>
     </link>
-    <link name="${prefix}aico1_x2_head_link">
+    <link name="${prefix}aico1_4s_v2_head_link">
       <inertial>
         <origin xyz="0.017 0.000125 0.0594" rpy="0 0 0" />
@@ -141,5 +141,5 @@
         <geometry>
           <mesh
-            filename="${mesh_prefix_path}meshes/AICO1-X2/visual/head_link.obj" />
+            filename="${mesh_prefix_path}meshes/AICO1-4s-V2/visual/head_link.obj" />
         </geometry>
         <material name="">
@@ -151,5 +151,5 @@
         <geometry>
           <mesh
-            filename="${mesh_prefix_path}meshes/AICO1-X2/collision/head_link.stl" />
+            filename="${mesh_prefix_path}meshes/AICO1-4s-V2/collision/head_link.stl" />
         </geometry>
       </collision>

File: urdf/common/aico2_10_v1.xacro (robot description, xacro)
@@ -1,33 +1,33 @@
 <?xml version="1.0" encoding="utf-8"?>
 <robot xmlns:xacro="http://wiki.ros.org/xacro">
-  <xacro:macro name="aico2_platform_x2"
+  <xacro:macro name="aico2_10_v1"
     params="prefix left_arm_prefix right_arm_prefix mesh_prefix_path">
-    <joint name="${prefix}aico2_x2_joint1" type="revolute">
+    <joint name="${prefix}aico2_10_v1_joint1" type="revolute">
       <origin xyz="0 0 0.804" rpy="0 0 0" />
-      <parent link="${prefix}aico2_x2_base_link" />
-      <child link="${prefix}aico2_x2_link1" />
+      <parent link="${prefix}aico2_10_v1_base_link" />
+      <child link="${prefix}aico2_10_v1_link1" />
       <axis xyz="0 0 1" />
       <limit lower="-1.57" upper="1.57" effort="1000" velocity="1" />
     </joint>
-    <joint name="${prefix}aico2_x2_joint2" type="revolute">
+    <joint name="${prefix}aico2_10_v1_joint2" type="revolute">
       <origin xyz="0 0 0.116" rpy="0 0 0" />
-      <parent link="${prefix}aico2_x2_link1" />
-      <child link="${prefix}aico2_x2_link2" />
+      <parent link="${prefix}aico2_10_v1_link1" />
+      <child link="${prefix}aico2_10_v1_link2" />
       <axis xyz="0 1 0" />
       <limit lower="0" upper="1.57" effort="1900" velocity="1" />
     </joint>
-    <joint name="${prefix}aico2_x2_left_arm_adapter" type="fixed">
+    <joint name="${prefix}aico2_10_v1_left_arm_adapter" type="fixed">
       <origin xyz="0 -0.0375 0.33" rpy="-1.5708 1.5708 0" />
-      <parent link="${prefix}aico2_x2_link2" />
+      <parent link="${prefix}aico2_10_v1_link2" />
       <child link="${left_arm_prefix}base_link" />
       <axis xyz="0 0 0" />
     </joint>
-    <joint name="${prefix}aico2_x2_right_arm_adapter" type="fixed">
+    <joint name="${prefix}aico2_10_v1_right_arm_adapter" type="fixed">
       <origin xyz="0 0.0375 0.33" rpy="1.5708 -1.5708 0" />
-      <parent link="${prefix}aico2_x2_link2" />
+      <parent link="${prefix}aico2_10_v1_link2" />
       <child link="${right_arm_prefix}base_link" />
       <axis xyz="0 0 0" />
     </joint>
-    <link name="${prefix}aico2_x2_base_link">
+    <link name="${prefix}aico2_10_v1_base_link">
       <inertial>
         <origin xyz="-0.006 -0.00638 0.157" rpy="0 0 0" />
@@ -38,5 +38,5 @@
         <origin xyz="0 0 0" rpy="0 0 0" />
         <geometry>
-          <mesh filename="${mesh_prefix_path}meshes/AICO2-X2/visual/base_link.obj" />
+          <mesh filename="${mesh_prefix_path}meshes/AICO2-10-V1/visual/base_link.obj" />
         </geometry>
         <material name="">
@@ -47,9 +47,9 @@
         <origin xyz="0 0 0" rpy="0 0 0" />
         <geometry>
-          <mesh filename="${mesh_prefix_path}meshes/AICO2-X2/collision/base_link.stl" />
+          <mesh filename="${mesh_prefix_path}meshes/AICO2-10-V1/collision/base_link.stl" />
         </geometry>
       </collision>
     </link>
-    <link name="${prefix}aico2_x2_link1">
+    <link name="${prefix}aico2_10_v1_link1">
       <inertial>
         <origin xyz="-0.00685 -0.00021 -0.073" rpy="0 0 0" />
@@ -60,5 +60,5 @@
         <origin xyz="0 0 0" rpy="0 0 0" />
         <geometry>
-          <mesh filename="${mesh_prefix_path}meshes/AICO2-X2/visual/link1.obj" />
+          <mesh filename="${mesh_prefix_path}meshes/AICO2-10-V1/visual/link1.obj" />
         </geometry>
         <material name="">
@@ -69,9 +69,9 @@
         <origin xyz="0 0 0" rpy="0 0 0" />
         <geometry>
-          <mesh filename="${mesh_prefix_path}meshes/AICO2-X2/collision/link1.stl" />
+          <mesh filename="${mesh_prefix_path}meshes/AICO2-10-V1/collision/link1.stl" />
         </geometry>
       </collision>
     </link>
-    <link name="${prefix}aico2_x2_link2">
+    <link name="${prefix}aico2_10_v1_link2">
       <inertial>
         <origin xyz="0.00217 3E-05 0.3" rpy="0 0 0" />
@@ -82,5 +82,5 @@
         <origin xyz="0 0 0" rpy="0 0 0" />
         <geometry>
-          <mesh filename="${mesh_prefix_path}meshes/AICO2-X2/visual/link2.obj" />
+          <mesh filename="${mesh_prefix_path}meshes/AICO2-10-V1/visual/link2.obj" />
         </geometry>
         <material name="">
@@ -91,5 +91,5 @@
         <origin xyz="0 0 0" rpy="0 0 0" />
         <geometry>
-          <mesh filename="${mesh_prefix_path}meshes/AICO2-X2/collision/link2.stl" />
+          <mesh filename="${mesh_prefix_path}meshes/AICO2-10-V1/collision/link2.stl" />
         </geometry>
       </collision>

File: urdf/common/aico2_4_v1.xacro (robot description, xacro)
@@ -1,33 +1,33 @@
 <?xml version="1.0" encoding="utf-8"?>
 <robot xmlns:xacro="http://wiki.ros.org/xacro">
-  <xacro:macro name="aico2_platform_x1"
+  <xacro:macro name="aico2_4_v1"
     params="prefix left_arm_prefix right_arm_prefix mesh_prefix_path">
-    <joint name="${prefix}aico2_x1_joint1" type="revolute">
+    <joint name="${prefix}aico2_4_v1_joint1" type="revolute">
       <origin xyz="0 0 0.307" rpy="0 0 0" />
-      <parent link="${prefix}aico2_x1_base_link" />
-      <child link="${prefix}aico2_x1_link1" />
+      <parent link="${prefix}aico2_4_v1_base_link" />
+      <child link="${prefix}aico2_4_v1_link1" />
       <axis xyz="0 0 1" />
       <limit lower="-1.57" upper="1.57" effort="400" velocity="1.05" />
     </joint>
-    <joint name="${prefix}aico2_x1_joint2" type="revolute">
+    <joint name="${prefix}aico2_4_v1_joint2" type="revolute">
       <origin xyz="0.025 0 0" rpy="0 0 0" />
-      <parent link="${prefix}aico2_x1_link1" />
-      <child link="${prefix}aico2_x1_link2" />
+      <parent link="${prefix}aico2_4_v1_link1" />
+      <child link="${prefix}aico2_4_v1_link2" />
       <axis xyz="0 1 0" />
       <limit lower="0" upper="1.57" effort="365" velocity="1" />
     </joint>
-    <joint name="${prefix}aico2_x1_left_arm_adapter" type="fixed">
+    <joint name="${prefix}aico2_4_v1_left_arm_adapter" type="fixed">
       <origin xyz="0 -0.035 0.2885" rpy="-1.5708 0 0" />
-      <parent link="${prefix}aico2_x1_link2" />
+      <parent link="${prefix}aico2_4_v1_link2" />
       <child link="${left_arm_prefix}base_link" />
       <axis xyz="0 0 0" />
     </joint>
-    <joint name="${prefix}aico2_x1_right_arm_adapter" type="fixed">
+    <joint name="${prefix}aico2_4_v1_right_arm_adapter" type="fixed">
       <origin xyz="0 0.035 0.2885" rpy="1.5708 0 0" />
-      <parent link="${prefix}aico2_x1_link2" />
+      <parent link="${prefix}aico2_4_v1_link2" />
       <child link="${right_arm_prefix}base_link" />
       <axis xyz="0 0 0" />
     </joint>
-    <link name="${prefix}aico2_x1_base_link">
+    <link name="${prefix}aico2_4_v1_base_link">
       <inertial>
         <origin xyz="0.0052 -0.0154 0.258" rpy="0 0 0" />
@@ -38,5 +38,5 @@
         <origin xyz="0 0 0" rpy="0 0 1.5708" />
         <geometry>
-          <mesh filename="${mesh_prefix_path}meshes/AICO2-X1/visual/base_link.obj"
+          <mesh filename="${mesh_prefix_path}meshes/AICO2-4-V1/visual/base_link.obj"
             scale="0.001 0.001 0.001" />
         </geometry>
@@ -48,9 +48,9 @@
         <origin xyz="0 0 0" rpy="0 0 0" />
         <geometry>
-          <mesh filename="${mesh_prefix_path}meshes/AICO2-X1/collision/base_link.stl" />
+          <mesh filename="${mesh_prefix_path}meshes/AICO2-4-V1/collision/base_link.stl" />
         </geometry>
       </collision>
     </link>
-    <link name="${prefix}aico2_x1_link1">
+    <link name="${prefix}aico2_4_v1_link1">
       <inertial>
         <origin xyz="0.0484 -6.38E-05 -0.134" rpy="0 0 0" />
@@ -61,5 +61,5 @@
         <origin xyz="0 0 0" rpy="0 0 1.5708" />
         <geometry>
-          <mesh filename="${mesh_prefix_path}meshes/AICO2-X1/visual/link1.obj" />
+          <mesh filename="${mesh_prefix_path}meshes/AICO2-4-V1/visual/link1.obj" />
         </geometry>
         <material name="">
@@ -70,9 +70,9 @@
         <origin xyz="0 0 0" rpy="0 0 0" />
         <geometry>
-          <mesh filename="${mesh_prefix_path}meshes/AICO2-X1/collision/link1.stl" />
+          <mesh filename="${mesh_prefix_path}meshes/AICO2-4-V1/collision/link1.stl" />
         </geometry>
       </collision>
     </link>
-    <link name="${prefix}aico2_x1_link2">
+    <link name="${prefix}aico2_4_v1_link2">
       <inertial>
         <origin xyz="-0.0155 0.00056 0.25" rpy="0 0 0" />
@@ -83,5 +83,5 @@
         <origin xyz="0 0 0" rpy="0 0 1.5708" />
         <geometry>
-          <mesh filename="${mesh_prefix_path}meshes/AICO2-X1/visual/link2.obj" />
+          <mesh filename="${mesh_prefix_path}meshes/AICO2-4-V1/visual/link2.obj" />
         </geometry>
         <material name="">
@@ -92,5 +92,5 @@
         <origin xyz="0 0 0" rpy="0 0 0" />
         <geometry>
-          <mesh filename="${mesh_prefix_path}meshes/AICO2-X1/collision/link2.stl" />
+          <mesh filename="${mesh_prefix_path}meshes/AICO2-4-V1/collision/link2.stl" />
         </geometry>
       </collision>
