Commit message: Rename AICO1-4 robot model

File: urdf/common/aico1_4_v1.xacro (robot description, xacro)
@@ -1,26 +1,26 @@
 <?xml version="1.0" encoding="utf-8"?>
 <robot xmlns:xacro="http://wiki.ros.org/xacro">
-  <xacro:macro name="aico1_4s_v1" params="prefix arm_prefix mesh_prefix_path">
-    <joint name="${prefix}aico1_4s_v1_joint1" type="fixed">
+  <xacro:macro name="aico1_4_v1" params="prefix arm_prefix mesh_prefix_path">
+    <joint name="${prefix}aico1_4_v1_joint1" type="fixed">
       <origin xyz="0 0 0.768" rpy="0 0 0" />
-      <parent link="${prefix}aico1_4s_v1_base_link" />
-      <child link="${prefix}aico1_4s_v1_link1" />
+      <parent link="${prefix}aico1_4_v1_base_link" />
+      <child link="${prefix}aico1_4_v1_link1" />
       <axis xyz="0 0 1" />
       <limit lower="0" upper="0.3" effort="100" velocity="1" />
     </joint>
-    <joint name="${prefix}aico1_4s_v1_joint2" type="revolute">
+    <joint name="${prefix}aico1_4_v1_joint2" type="revolute">
       <origin xyz="0.1385 0.204 0.183" rpy="0 0 0" />
-      <parent link="${prefix}aico1_4s_v1_link1" />
-      <child link="${prefix}aico1_4s_v1_link2" />
+      <parent link="${prefix}aico1_4_v1_link1" />
+      <child link="${prefix}aico1_4_v1_link2" />
       <axis xyz="0 1 0" />
       <limit lower="0" upper="1.57" effort="365" velocity="1" />
     </joint>
-    <joint name="${prefix}aico1_4s_v1_arm_adapter" type="fixed">
+    <joint name="${prefix}aico1_4_v1_arm_adapter" type="fixed">
       <origin xyz="0.0037763 0.0 0.3214" rpy="1.5708 0 0" />
-      <parent link="${prefix}aico1_4s_v1_link2" />
+      <parent link="${prefix}aico1_4_v1_link2" />
       <child link="${arm_prefix}base_link" />
       <axis xyz="0 0 0" />
     </joint>
-    <link name="${prefix}aico1_4s_v1_base_link">
+    <link name="${prefix}aico1_4_v1_base_link">
       <inertial>
         <origin xyz="0.00266 0.000754 0.34" rpy="0 0 0" />
@@ -32,5 +32,5 @@
         <geometry>
           <mesh
-            filename="${mesh_prefix_path}meshes/AICO1-4s-V1/visual/base_link.obj" />
+            filename="${mesh_prefix_path}meshes/AICO1-4-V1/visual/base_link.obj" />
         </geometry>
         <material name="">
@@ -42,9 +42,9 @@
         <geometry>
           <mesh
-            filename="${mesh_prefix_path}meshes/AICO1-4s-V1/collision/base_link.stl" />
+            filename="${mesh_prefix_path}meshes/AICO1-4-V1/collision/base_link.stl" />
         </geometry>
       </collision>
     </link>
-    <link name="${prefix}aico1_4s_v1_link1">
+    <link name="${prefix}aico1_4_v1_link1">
       <inertial>
         <origin xyz="0.017 0.014 -0.075" rpy="0 0 0" />
@@ -56,5 +56,5 @@
         <geometry>
           <mesh
-            filename="${mesh_prefix_path}meshes/AICO1-4s-V1/visual/rise_link.obj" />
+            filename="${mesh_prefix_path}meshes/AICO1-4-V1/visual/rise_link.obj" />
         </geometry>
         <material name="">
@@ -66,5 +66,5 @@
         <geometry>
           <mesh
-            filename="${mesh_prefix_path}meshes/AICO1-4s-V1/collision/rise_link_bottom.stl" />
+            filename="${mesh_prefix_path}meshes/AICO1-4-V1/collision/rise_link_bottom.stl" />
         </geometry>
       </collision>
@@ -73,9 +73,9 @@
         <geometry>
           <mesh
-            filename="${mesh_prefix_path}meshes/AICO1-4s-V1/collision/rise_link_top.stl" />
+            filename="${mesh_prefix_path}meshes/AICO1-4-V1/collision/rise_link_top.stl" />
         </geometry>
       </collision>
     </link>
-    <link name="${prefix}aico1_4s_v1_link2">
+    <link name="${prefix}aico1_4_v1_link2">
       <inertial>
         <origin xyz="0.0303 -0.092 0.255" rpy="0 0 0" />
@@ -87,5 +87,5 @@
         <geometry>
           <mesh
-            filename="${mesh_prefix_path}meshes/AICO1-4s-V1/visual/pitch_link.obj" />
+            filename="${mesh_prefix_path}meshes/AICO1-4-V1/visual/pitch_link.obj" />
         </geometry>
         <material name="">
@@ -97,5 +97,5 @@
         <geometry>
           <mesh
-            filename="${mesh_prefix_path}meshes/AICO1-4s-V1/collision/pitch_link.stl" />
+            filename="${mesh_prefix_path}meshes/AICO1-4-V1/collision/pitch_link.stl" />
         </geometry>
       </collision>

File: urdf/common/aico1_4_v2.xacro (robot description, xacro)
@@ -1,39 +1,39 @@
 <?xml version="1.0" encoding="utf-8"?>
 <robot xmlns:xacro="http://wiki.ros.org/xacro">
-  <xacro:macro name="aico1_4s_v2" params="prefix arm_prefix mesh_prefix_path">
-    <joint name="${prefix}aico1_4s_v2_base_to_agv" type="fixed">
+  <xacro:macro name="aico1_4_v2" params="prefix arm_prefix mesh_prefix_path">
+    <joint name="${prefix}aico1_4_v2_base_to_agv" type="fixed">
       <origin xyz="0.004 0.1255 0.695" rpy="0.0 0.0 0.0" />
-      <parent link="${prefix}aico1_4s_v2_agv" />
-      <child link="${prefix}aico1_4s_v2_base_link" />
+      <parent link="${prefix}aico1_4_v2_agv" />
+      <child link="${prefix}aico1_4_v2_base_link" />
       <axis xyz="0 0 0" />
     </joint>
-    <joint name="${prefix}aico1_4s_v2_joint1" type="revolute">
+    <joint name="${prefix}aico1_4_v2_joint1" type="revolute">
       <origin xyz="-0.122 0.1066 0.164" rpy="0 0 0" />
-      <parent link="${prefix}aico1_4s_v2_base_link" />
-      <child link="${prefix}aico1_4s_v2_link1" />
+      <parent link="${prefix}aico1_4_v2_base_link" />
+      <child link="${prefix}aico1_4_v2_link1" />
       <axis xyz="0 1 0" />
       <limit lower="-0.523598775598" upper="1.57079632679" effort="1000"
         velocity="1" />
     </joint>
-    <joint name="${prefix}aico1_4s_v2_joint2" type="revolute">
+    <joint name="${prefix}aico1_4_v2_joint2" type="revolute">
       <origin xyz="-0.005 -0.0991 0.47875" rpy="0 0 0" />
-      <parent link="${prefix}aico1_4s_v2_link1" />
-      <child link="${prefix}aico1_4s_v2_neck_link" />
+      <parent link="${prefix}aico1_4_v2_link1" />
+      <child link="${prefix}aico1_4_v2_neck_link" />
       <axis xyz="0 0 1" />
       <limit lower="-1.57079632679" upper="1.57079632679" effort="50" velocity="1" />
     </joint>
-    <joint name="${prefix}aico1_4s_v2_joint_head" type="revolute">
+    <joint name="${prefix}aico1_4_v2_joint_head" type="revolute">
       <origin xyz="-0.025 0 0.088" rpy="0 0 0" />
-      <parent link="${prefix}aico1_4s_v2_neck_link" />
-      <child link="${prefix}aico1_4s_v2_head_link" />
+      <parent link="${prefix}aico1_4_v2_neck_link" />
+      <child link="${prefix}aico1_4_v2_head_link" />
       <axis xyz="0 1 0" />
       <limit lower="0" upper="0.436332312999" effort="80" velocity="1" />
     </joint>
-    <joint name="${prefix}aico1_4s_v2_arm_adapter" type="fixed">
-      <parent link="${prefix}aico1_4s_v2_link1" />
+    <joint name="${prefix}aico1_4_v2_arm_adapter" type="fixed">
+      <parent link="${prefix}aico1_4_v2_link1" />
       <child link="${arm_prefix}base_link" />
       <origin xyz="0.0 0.016 0.320" rpy="1.57079632679 0.0 0.0" />
     </joint>
-    <link name="${prefix}aico1_4s_v2_agv">
+    <link name="${prefix}aico1_4_v2_agv">
       <inertial>
         <origin xyz="0 0 0" rpy="0 0 0" />
@@ -45,5 +45,5 @@
         <geometry>
           <mesh
-            filename="${mesh_prefix_path}meshes/AICO1-4s-V2/visual/agv.obj" />
+            filename="${mesh_prefix_path}meshes/AICO1-4-V2/visual/agv.obj" />
         </geometry>
         <material name="">
@@ -55,9 +55,9 @@
         <geometry>
           <mesh
-            filename="${mesh_prefix_path}meshes/AICO1-4s-V2/collision/agv.stl" />
+            filename="${mesh_prefix_path}meshes/AICO1-4-V2/collision/agv.stl" />
         </geometry>
       </collision>
     </link>
-    <link name="${prefix}aico1_4s_v2_base_link">
+    <link name="${prefix}aico1_4_v2_base_link">
       <inertial>
         <origin xyz="-0.0372 -0.00251 0.0448" rpy="0 0 0" />
@@ -69,5 +69,5 @@
         <geometry>
           <mesh
-            filename="${mesh_prefix_path}meshes/AICO1-4s-V2/visual/base_link.obj" />
+            filename="${mesh_prefix_path}meshes/AICO1-4-V2/visual/base_link.obj" />
         </geometry>
         <material name="">
@@ -79,9 +79,9 @@
         <geometry>
           <mesh
-            filename="${mesh_prefix_path}meshes/AICO1-4s-V2/collision/base_link.stl" />
+            filename="${mesh_prefix_path}meshes/AICO1-4-V2/collision/base_link.stl" />
         </geometry>
       </collision>
     </link>
-    <link name="${prefix}aico1_4s_v2_link1">
+    <link name="${prefix}aico1_4_v2_link1">
       <inertial>
         <origin xyz="-0.00141 -0.0922 0.106" rpy="0 0 0" />
@@ -93,5 +93,5 @@
         <geometry>
           <mesh
-            filename="${mesh_prefix_path}meshes/AICO1-4s-V2/visual/link1.obj" />
+            filename="${mesh_prefix_path}meshes/AICO1-4-V2/visual/link1.obj" />
         </geometry>
         <material name="">
@@ -103,9 +103,9 @@
         <geometry>
           <mesh
-            filename="${mesh_prefix_path}meshes/AICO1-4s-V2/collision/link1.stl" />
+            filename="${mesh_prefix_path}meshes/AICO1-4-V2/collision/link1.stl" />
         </geometry>
       </collision>
     </link>
-    <link name="${prefix}aico1_4s_v2_neck_link">
+    <link name="${prefix}aico1_4_v2_neck_link">
       <inertial>
         <origin xyz="-0.0149 7E-07 0.0547" rpy="0 0 0" />
@@ -117,5 +117,5 @@
         <geometry>
           <mesh
-            filename="${mesh_prefix_path}meshes/AICO1-4s-V2/visual/neck_link.obj" />
+            filename="${mesh_prefix_path}meshes/AICO1-4-V2/visual/neck_link.obj" />
         </geometry>
         <material name="">
@@ -127,9 +127,9 @@
         <geometry>
           <mesh
-            filename="${mesh_prefix_path}meshes/AICO1-4s-V2/collision/neck_link.stl" />
+            filename="${mesh_prefix_path}meshes/AICO1-4-V2/collision/neck_link.stl" />
         </geometry>
       </collision>
     </link>
-    <link name="${prefix}aico1_4s_v2_head_link">
+    <link name="${prefix}aico1_4_v2_head_link">
       <inertial>
         <origin xyz="0.017 0.000125 0.0594" rpy="0 0 0" />
@@ -141,5 +141,5 @@
         <geometry>
           <mesh
-            filename="${mesh_prefix_path}meshes/AICO1-4s-V2/visual/head_link.obj" />
+            filename="${mesh_prefix_path}meshes/AICO1-4-V2/visual/head_link.obj" />
         </geometry>
         <material name="">
@@ -151,5 +151,5 @@
         <geometry>
           <mesh
-            filename="${mesh_prefix_path}meshes/AICO1-4s-V2/collision/head_link.stl" />
+            filename="${mesh_prefix_path}meshes/AICO1-4-V2/collision/head_link.stl" />
         </geometry>
       </collision>

Commit message: Update robot inertia parameters for AICO models

File: urdf/common/aico1_4_v1.xacro (robot description, xacro)
@@ -24,7 +24,7 @@
     <link name="${prefix}aico1_4_v1_base_link">
       <inertial>
-        <origin xyz="0.00266 0.000754 0.34" rpy="0 0 0" />
-        <mass value="6.6" />
-        <inertia ixx="0.45" ixy="-0.0018" ixz="-0.0051" iyy="0.234" iyz="-0.00059" izz="0.3" />
+        <origin xyz="0.00266 0.00075403 0.34014" rpy="0 0 0" />
+        <mass value="6.6026" />
+        <inertia ixx="0.45058" ixy="-0.0017625" ixz="-0.0050778" iyy="0.23454" iyz="-0.00059237" izz="0.2993" />
       </inertial>
       <visual>
@@ -48,7 +48,7 @@
     <link name="${prefix}aico1_4_v1_link1">
       <inertial>
-        <origin xyz="0.017 0.014 -0.075" rpy="0 0 0" />
-        <mass value="6.3" />
-        <inertia ixx="0.35" ixy="-0.002" ixz="-0.0059" iyy="0.197" iyz="-0.0096" izz="0.241" />
+        <origin xyz="0.017065 0.014003 -0.075525" rpy="0 0 0" />
+        <mass value="6.2889" />
+        <inertia ixx="0.35138" ixy="-0.0019964" ixz="-0.0059424" iyy="0.19696" iyz="-0.0095617" izz="0.24113" />
       </inertial>
       <visual>
@@ -79,7 +79,7 @@
     <link name="${prefix}aico1_4_v1_link2">
       <inertial>
-        <origin xyz="0.0303 -0.092 0.255" rpy="0 0 0" />
-        <mass value="3.68" />
-        <inertia ixx="0.0804" ixy="4.3E-05" ixz="-0.0025" iyy="0.0484" iyz="-0.0063" izz="0.047" />
+        <origin xyz="0.030313 -0.09201 0.25487" rpy="0 0 0" />
+        <mass value="3.6794" />
+        <inertia ixx="0.080449" ixy="4.3268E-05" ixz="-0.0025222" iyy="0.048422" iyz="-0.0063047" izz="0.046989" />
       </inertial>
       <visual>

File: urdf/common/aico1_4_v2.xacro (robot description, xacro)
@@ -2,13 +2,13 @@
 <robot xmlns:xacro="http://wiki.ros.org/xacro">
   <xacro:macro name="aico1_4_v2" params="prefix arm_prefix mesh_prefix_path">
-    <joint name="${prefix}aico1_4_v2_base_to_agv" type="fixed">
+    <joint name="${prefix}aico1_4_v2_base_to_torso_mount" type="fixed">
       <origin xyz="0.004 0.1255 0.695" rpy="0.0 0.0 0.0" />
-      <parent link="${prefix}aico1_4_v2_agv" />
-      <child link="${prefix}aico1_4_v2_base_link" />
+      <parent link="${prefix}aico1_4_v2_base_link" />
+      <child link="${prefix}aico1_4_v2_torso_mount"/>
       <axis xyz="0 0 0" />
     </joint>
     <joint name="${prefix}aico1_4_v2_joint1" type="revolute">
       <origin xyz="-0.122 0.1066 0.164" rpy="0 0 0" />
-      <parent link="${prefix}aico1_4_v2_base_link" />
+      <parent link="${prefix}aico1_4_v2_torso_mount" />
       <child link="${prefix}aico1_4_v2_link1" />
       <axis xyz="0 1 0" />
@@ -35,33 +35,9 @@
       <origin xyz="0.0 0.016 0.320" rpy="1.57079632679 0.0 0.0" />
     </joint>
-    <link name="${prefix}aico1_4_v2_agv">
+    <link name="${prefix}aico1_4_v2_base_link">
       <inertial>
         <origin xyz="0 0 0" rpy="0 0 0" />
         <mass value="60" />
-        <inertia ixx="0.029" ixy="2.8E-05" ixz="-2.82E-05" iyy="0.089" iyz="4.6E-05" izz="0.105" />
-      </inertial>
-      <visual>
-        <origin xyz="0 0 0" rpy="0 0 0" />
-        <geometry>
-          <mesh
-            filename="${mesh_prefix_path}meshes/AICO1-4-V2/visual/agv.obj" />
-        </geometry>
-        <material name="">
-          <color rgba="0.75294 0.75294 0.75294 1" />
-        </material>
-      </visual>
-      <collision>
-        <origin xyz="0 0 0" rpy="0 0 0" />
-        <geometry>
-          <mesh
-            filename="${mesh_prefix_path}meshes/AICO1-4-V2/collision/agv.stl" />
-        </geometry>
-      </collision>
-    </link>
-    <link name="${prefix}aico1_4_v2_base_link">
-      <inertial>
-        <origin xyz="-0.0372 -0.00251 0.0448" rpy="0 0 0" />
-        <mass value="3.9" />
-        <inertia ixx="0.029" ixy="2.8E-05" ixz="-2.82E-05" iyy="0.089" iyz="4.6E-05" izz="0.105" />
+        <inertia ixx="0.029184" ixy="2.8373E-05" ixz="-2.82E-05" iyy="0.089571" iyz="4.6654E-05" izz="0.10508" />
       </inertial>
       <visual>
@@ -83,9 +59,33 @@
       </collision>
     </link>
+    <link name="${prefix}aico1_4_v2_torso_mount">
+      <inertial>
+        <origin xyz="-0.037217 -0.002506 0.044824" rpy="0 0 0" />
+        <mass value="3.9443" />
+        <inertia ixx="0.029184" ixy="2.8373E-05" ixz="-2.82E-05" iyy="0.089571" iyz="4.6654E-05" izz="0.10508" />
+      </inertial>
+      <visual>
+        <origin xyz="0 0 0" rpy="0 0 0" />
+        <geometry>
+          <mesh
+            filename="${mesh_prefix_path}meshes/AICO1-4-V2/visual/torso_mount.obj" />
+        </geometry>
+        <material name="">
+          <color rgba="0.75294 0.75294 0.75294 1" />
+        </material>
+      </visual>
+      <collision>
+        <origin xyz="0 0 0" rpy="0 0 0" />
+        <geometry>
+          <mesh
+            filename="${mesh_prefix_path}meshes/AICO1-4-V2/collision/torso_mount.stl" />
+        </geometry>
+      </collision>
+    </link>
     <link name="${prefix}aico1_4_v2_link1">
       <inertial>
-        <origin xyz="-0.00141 -0.0922 0.106" rpy="0 0 0" />
-        <mass value="2.76" />
-        <inertia ixx="0.039" ixy="-8.02E-05" ixz="-0.00091" iyy="0.04" iyz="0.0017" izz="0.026" />
+        <origin xyz="-0.0014123 -0.092235 0.10641" rpy="0 0 0" />
+        <mass value="2.7625" />
+        <inertia ixx="0.039793" ixy="-8.0219E-05" ixz="-0.00090994" iyy="0.039722" iyz="0.0017219" izz="0.026481" />
       </inertial>
       <visual>
@@ -109,7 +109,7 @@
     <link name="${prefix}aico1_4_v2_neck_link">
       <inertial>
-        <origin xyz="-0.0149 7E-07 0.0547" rpy="0 0 0" />
-        <mass value="0.078" />
-        <inertia ixx="0.00013" ixy="-1.6E-09" ixz="1.4E-05" iyy="7.7E-05" iyz="9.9E-10" izz="8E-05" />
+        <origin xyz="-0.014922 7.085E-07 0.054696" rpy="0 0 0" />
+        <mass value="0.078627" />
+        <inertia ixx="0.00013359" ixy="-1.6505E-09" ixz="1.4077E-05" iyy="7.7245E-05" iyz="9.9064E-10" izz="8.0068E-05" />
       </inertial>
       <visual>
@@ -133,7 +133,7 @@
     <link name="${prefix}aico1_4_v2_head_link">
       <inertial>
-        <origin xyz="0.017 0.000125 0.0594" rpy="0 0 0" />
-        <mass value="6.97" />
-        <inertia ixx="0.062" ixy="-1.05E-06" ixz="0.00041" iyy="0.03" iyz="2.35E-06" izz="0.057" />
+        <origin xyz="0.017357 0.00012518 0.059446" rpy="0 0 0" />
+        <mass value="6.9698" />
+        <inertia ixx="0.061947" ixy="-1.0452E-06" ixz="0.00041384" iyy="0.029712" iyz="2.3512E-06" izz="0.057242" />
       </inertial>
       <visual>

File: urdf/common/aico2_10_v1.xacro (robot description, xacro)
@@ -31,7 +31,7 @@
     <link name="${prefix}aico2_10_v1_base_link">
       <inertial>
-        <origin xyz="-0.006 -0.00638 0.157" rpy="0 0 0" />
-        <mass value="30.4" />
-        <inertia ixx="0.67" ixy="-0.0021" ixz="0.006" iyy="0.65" iyz="0.0004" izz="1.13" />
+        <origin xyz="-0.0059929 -0.0063778 0.15742" rpy="0 0 0" />
+        <mass value="30.358" />
+        <inertia ixx="0.66978" ixy="-0.0020934" ixz="0.0059521" iyy="0.64823" iyz="0.00043467" izz="1.1261" />
       </inertial>
       <visual>
@@ -53,7 +53,7 @@
     <link name="${prefix}aico2_10_v1_link1">
       <inertial>
-        <origin xyz="-0.00685 -0.00021 -0.073" rpy="0 0 0" />
-        <mass value="3.3" />
-        <inertia ixx="0.19" ixy="-9E-06" ixz="0.00231" iyy="0.12" iyz="0.00012" izz="0.083" />
+        <origin xyz="-0.0068471 -0.00020586 -0.072697" rpy="0 0 0" />
+        <mass value="3.3142" />
+        <inertia ixx="0.18573" ixy="-9.5323E-06" ixz="0.0023109" iyy="0.12383" iyz="0.00012341" izz="0.082964" />
       </inertial>
       <visual>
@@ -75,7 +75,7 @@
     <link name="${prefix}aico2_10_v1_link2">
       <inertial>
-        <origin xyz="0.00217 3E-05 0.3" rpy="0 0 0" />
-        <mass value="4" />
-        <inertia ixx="0.167" ixy="6.9E-06" ixz="-0.00029" iyy="0.082" iyz="-3.7E-06" izz="0.125" />
+        <origin xyz="0.0021658 3.0022E-05 0.2996" rpy="0 0 0" />
+        <mass value="4.0152" />
+        <inertia ixx="0.16718" ixy="6.9054E-06" ixz="-0.00029293" iyy="0.081637" iyz="-3.6515E-06" izz="0.12478" />
       </inertial>
       <visual>

File: urdf/common/aico2_4_v1.xacro (robot description, xacro)
@@ -31,7 +31,7 @@
     <link name="${prefix}aico2_4_v1_base_link">
       <inertial>
-        <origin xyz="0.0052 -0.0154 0.258" rpy="0 0 0" />
-        <mass value="53.5" />
-        <inertia ixx="1.61" ixy="0.00049" ixz="0.0047" iyy="0.81" iyz="-0.0133" izz="1.86" />
+        <origin xyz="0.0052047 -0.015452 0.25843" rpy="0 0 0" />
+        <mass value="53.522" />
+        <inertia ixx="1.6095" ixy="0.00048511" ixz="0.004696" iyy="0.80577" iyz="-0.013343" izz="1.8645" />
       </inertial>
       <visual>
@@ -54,7 +54,7 @@
     <link name="${prefix}aico2_4_v1_link1">
       <inertial>
-        <origin xyz="0.0484 -6.38E-05 -0.134" rpy="0 0 0" />
-        <mass value="11.5" />
-        <inertia ixx="0.549" ixy="3.3E-05" ixz="-0.061" iyy="0.48" iyz="-5.7E-05" izz="0.218" />
+        <origin xyz="0.048352 -6.38E-05 -0.13411" rpy="0 0 0" />
+        <mass value="11.466" />
+        <inertia ixx="0.54861" ixy="3.301E-05" ixz="-0.061055" iyy="0.4792" iyz="-5.73E-05" izz="0.21847" />
       </inertial>
       <visual>
@@ -76,7 +76,7 @@
     <link name="${prefix}aico2_4_v1_link2">
       <inertial>
-        <origin xyz="-0.0155 0.00056 0.25" rpy="0 0 0" />
-        <mass value="8.6" />
-        <inertia ixx="0.28" ixy="0.00029" ixz="-0.0073" iyy="0.19" iyz="7.7E-05" izz="0.175" />
+        <origin xyz="-0.015519 0.00056005 0.24987" rpy="0 0 0" />
+        <mass value="8.6001" />
+        <inertia ixx="0.27997" ixy="0.00028956" ixz="-0.0072546" iyy="0.19124" iyz="7.7035E-05" izz="0.17514" />
       </inertial>
       <visual>

File: urdf/common/aico2_4_v2.xacro (robot description, xacro)
@@ -30,7 +30,7 @@
     <link name="${prefix}aico2_4_v2_base_link">
       <inertial>
-        <origin xyz="-0.009 0.0011 0.21" rpy="0 0 0" />
-        <mass value="42.5" />
-        <inertia ixx="0.73" ixy="-0.003" ixz="0.005" iyy="0.68" iyz="0.0004" izz="1.2" />
+        <origin xyz="-0.0088021 0.0011052 0.21091" rpy="0 0 0" />
+        <mass value="42.488" />
+        <inertia ixx="0.72999" ixy="-0.003102" ixz="0.0053601" iyy="0.67864" iyz="0.00041913" izz="1.2009" />
       </inertial>
       <visual>
@@ -52,7 +52,7 @@
     <link name="${prefix}aico2_4_v2_link1">
       <inertial>
-        <origin xyz="-0.005 9.74E-06 -0.15" rpy="0 0 0" />
-        <mass value="3.2" />
-        <inertia ixx="0.17" ixy="2.5E-06" ixz="0.0016" iyy="0.12" iyz="1.65E-05" izz="0.07" />
+        <origin xyz="-0.0053448 9.7381E-06 -0.1462" rpy="0 0 0" />
+        <mass value="3.1883" />
+        <inertia ixx="0.17302" ixy="2.5419E-06" ixz="0.001552" iyy="0.11904" iyz="1.6546E-05" izz="0.069933" />
       </inertial>
       <visual>
@@ -74,7 +74,7 @@
     <link name="${prefix}aico2_4_v2_link2">
       <inertial>
-        <origin xyz="0.004 -6E-05 0.26" rpy="0 0 0" />
-        <mass value="3.4" />
-        <inertia ixx="0.12" ixy="1.9E-06" ixz="0.0003" iyy="0.048" iyz="-1.8E-05" izz="0.08" />
+        <origin xyz="0.0039028 -6.035E-05 0.25637" rpy="0 0 0" />
+        <mass value="3.4291" />
+        <inertia ixx="0.11689" ixy="1.8994E-06" ixz="0.00030188" iyy="0.048162" iyz="-1.7709E-05" izz="0.079268" />
       </inertial>
       <visual>
