Commit message: Release/flexiv_description Lyrical v3.1 (#43)

File: urdf/common/aico1_4_v1.xacro (robot description, xacro)
@@ -7,5 +7,6 @@
       <child link="${prefix}aico1_4_v1_link1" />
       <axis xyz="0 0 1" />
-      <limit lower="0" upper="0.3" effort="100" velocity="1" />
+      <limit lower="0" upper="0.3" effort="100" velocity="1"
+        acceleration="4" deceleration="4" jerk="32" />
     </joint>
     <joint name="${prefix}aico1_4_v1_joint2" type="revolute">
@@ -14,8 +15,9 @@
       <child link="${prefix}aico1_4_v1_link2" />
       <axis xyz="0 1 0" />
-      <limit lower="0" upper="1.57" effort="365" velocity="1" />
+      <limit lower="0" upper="1.57" effort="365" velocity="1"
+        acceleration="4" deceleration="4" jerk="32" />
     </joint>
     <joint name="${prefix}aico1_4_v1_arm_adapter" type="fixed">
-      <origin xyz="0.0037763 0.0 0.3214" rpy="1.5708 0 0" />
+      <origin xyz="0.0037763 7.8713E-05 0.3214" rpy="1.5708 0 0" />
       <parent link="${prefix}aico1_4_v1_link2" />
       <child link="${arm_prefix}base_link" />

File: urdf/common/aico1_4_v2.xacro (robot description, xacro)
@@ -14,19 +14,15 @@
       <axis xyz="0 1 0" />
       <limit lower="-0.523598775598" upper="1.57079632679" effort="1000"
-        velocity="1" />
+        velocity="1" acceleration="4" deceleration="4" jerk="32" />
     </joint>
-    <joint name="${prefix}aico1_4_v2_joint2" type="revolute">
+    <joint name="${prefix}aico1_4_v2_joint2" type="fixed">
       <origin xyz="-0.005 -0.0991 0.47875" rpy="0 0 0" />
       <parent link="${prefix}aico1_4_v2_link1" />
       <child link="${prefix}aico1_4_v2_neck_link" />
-      <axis xyz="0 0 1" />
-      <limit lower="-1.57079632679" upper="1.57079632679" effort="50" velocity="1" />
     </joint>
-    <joint name="${prefix}aico1_4_v2_joint_head" type="revolute">
+    <joint name="${prefix}aico1_4_v2_joint_head" type="fixed">
       <origin xyz="-0.025 0 0.088" rpy="0 0 0" />
       <parent link="${prefix}aico1_4_v2_neck_link" />
       <child link="${prefix}aico1_4_v2_head_link" />
-      <axis xyz="0 1 0" />
-      <limit lower="0" upper="0.436332312999" effort="80" velocity="1" />
     </joint>
     <joint name="${prefix}aico1_4_v2_arm_adapter" type="fixed">

File: urdf/common/flexiv_common.xacro (robot description, xacro)
@@ -79,9 +79,21 @@
   <xacro:macro name="get_joint_limits" params="name">
     <xacro:property name="limits" value="${sec_joint_limits[name]}" lazy_eval="false" />
-    <limit lower="${limits['lower']}" upper="${limits['upper']}" effort="${limits['effort']}"
-      velocity="${limits['velocity']}" />
-    <safety_controller k_position="100.0" k_velocity="40.0"
-      soft_lower_limit="${limits['soft_lower']}"
-      soft_upper_limit="${limits['soft_upper']}" />
+    <!-- URDF 1.2 dynamic limits; a YAML without them leaves the parser at infinity -->
+    <xacro:if value="${'acceleration' in limits}">
+      <limit lower="${limits['lower']}" upper="${limits['upper']}" effort="${limits['effort']}"
+        velocity="${limits['velocity']}" acceleration="${limits['acceleration']}"
+        deceleration="${limits.get('deceleration', limits['acceleration'])}"
+        jerk="${limits['jerk']}" />
+    </xacro:if>
+    <xacro:unless value="${'acceleration' in limits}">
+      <limit lower="${limits['lower']}" upper="${limits['upper']}" effort="${limits['effort']}"
+        velocity="${limits['velocity']}" />
+    </xacro:unless>
+    <!-- Soft limits are optional: the MICO torso joints have none -->
+    <xacro:if value="${'soft_lower' in limits}">
+      <safety_controller k_position="100.0" k_velocity="40.0"
+        soft_lower_limit="${limits['soft_lower']}"
+        soft_upper_limit="${limits['soft_upper']}" />
+    </xacro:if>
   </xacro:macro>
   <!--
@@ -108,11 +120,13 @@
   <xacro:macro name="get_inertias" params="name">
     <xacro:property name="inertias" value="${sec_inertia_parameters[name]}" lazy_eval="false" />
-    <origin xyz="${inertias['origin']['x']} ${inertias['origin']['y']} ${inertias['origin']['z']}"
-      rpy="${inertias['origin']['roll']} ${inertias['origin']['pitch']} ${inertias['origin']['yaw']}" />
-    <mass value="${inertias['mass']}" />
-    <inertia ixx="${inertias['inertia']['ixx']}" ixy="${inertias['inertia']['ixy']}"
-      ixz="${inertias['inertia']['ixz']}" iyy="${inertias['inertia']['iyy']}"
-      iyz="${inertias['inertia']['iyz']}"
-      izz="${inertias['inertia']['izz']}" />
+    <inertial>
+      <origin xyz="${inertias['origin']['x']} ${inertias['origin']['y']} ${inertias['origin']['z']}"
+        rpy="${inertias['origin']['roll']} ${inertias['origin']['pitch']} ${inertias['origin']['yaw']}" />
+      <mass value="${inertias['mass']}" />
+      <inertia ixx="${inertias['inertia']['ixx']}" ixy="${inertias['inertia']['ixy']}"
+        ixz="${inertias['inertia']['ixz']}" iyy="${inertias['inertia']['iyy']}"
+        iyz="${inertias['inertia']['iyz']}"
+        izz="${inertias['inertia']['izz']}" />
+    </inertial>
   </xacro:macro>
   <!--

File: urdf/common/grav_macro.xacro (robot description, xacro)
@@ -185,6 +185,6 @@
       </collision>
     </link>
-    <!-- TCP links -->
-    <link name="${prefix}grav_tcp"><!-- open finger, used by RCA -->
+    <!-- TCP between the open finger tips -->
+    <link name="${prefix}grav_tcp">
       <inertial>
         <origin rpy="0 0 0" xyz="0 0 0" />
@@ -193,36 +193,9 @@
       </inertial>
     </link>
-    <link name="${prefix}closed_fingers_tcp">
-      <inertial>
-        <origin rpy="0 0 0" xyz="0 0 0" />
-        <mass value="0" />
-        <inertia ixx="0" ixy="0" ixz="0" iyy="0" iyz="0" izz="0" />
-      </inertial>
-    </link>
-    <link name="${prefix}left_finger_tcp">
-      <inertial>
-        <origin rpy="0 0 0" xyz="0 0 0" />
-        <mass value="0" />
-        <inertia ixx="0" ixy="0" ixz="0" iyy="0" iyz="0" izz="0" />
-      </inertial>
-    </link>
-    <link name="${prefix}right_finger_tcp">
-      <inertial>
-        <origin rpy="0 0 0" xyz="0 0 0" />
-        <mass value="0" />
-        <inertia ixx="0" ixy="0" ixz="0" iyy="0" iyz="0" izz="0" />
-      </inertial>
-    </link>
     <!-- JOINTS -->
-    <joint name="${prefix}open_fingers_tcp_joint" type="fixed">
-      <origin rpy="0 0 0" xyz="0 0 0.15" />
+    <joint name="${prefix}base_to_tcp" type="fixed">
+      <origin rpy="0 0 0" xyz="0 0 0.18" />
       <parent link="${prefix}grav_base_link" />
       <child link="${prefix}grav_tcp" />
-      <axis xyz="0 0 1" />
-    </joint>
-    <joint name="${prefix}closed_fingers_tcp_joint" type="fixed">
-      <origin rpy="0 0 0" xyz="0 0 0.20" />
-      <parent link="${prefix}grav_base_link" />
-      <child link="${prefix}closed_fingers_tcp" />
       <axis xyz="0 0 1" />
     </joint>
@@ -233,5 +206,6 @@
       <child link="${prefix}left_outer_bar" />
       <axis xyz="1 0 0" />
-      <limit effort="0" lower="-0.155" upper="0.7854" velocity="2.0" />
+      <limit effort="0" lower="-0.155" upper="0.7854" velocity="2.0"
+        acceleration="8" deceleration="8" jerk="64" />
       <mimic joint="${prefix}finger_width_joint" multiplier="9.404" offset="-0.155" />
     </joint>
@@ -241,5 +215,6 @@
       <child link="${prefix}left_inner_bar" />
       <axis xyz="1 0 0" />
-      <limit effort="0" lower="-0.155" upper="0.7854" velocity="2.0" />
+      <limit effort="0" lower="-0.155" upper="0.7854" velocity="2.0"
+        acceleration="8" deceleration="8" jerk="64" />
       <mimic joint="${prefix}left_outer_knuckle_joint" multiplier="1" offset="0" />
     </joint>
@@ -249,5 +224,6 @@
       <child link="${prefix}left_finger_mount" />
       <axis xyz="1 0 0" />
-      <limit effort="0" lower="-0.7854" upper="0.155" velocity="2.0" />
+      <limit effort="0" lower="-0.7854" upper="0.155" velocity="2.0"
+        acceleration="8" deceleration="8" jerk="64" />
       <mimic joint="${prefix}left_outer_knuckle_joint" multiplier="-1" offset="0" />
     </joint>
@@ -258,10 +234,4 @@
       <axis xyz="0 0 1" />
     </joint>
-    <joint name="${prefix}left_finger_tcp_joint" type="fixed">
-      <origin rpy="0 0 0" xyz="0 0.0135 0.036" />
-      <parent link="${prefix}left_finger_tip" />
-      <child link="${prefix}left_finger_tcp" />
-      <axis xyz="0 0 1" />
-    </joint>
     <!-- right finger joints -->
     <joint name="${prefix}right_outer_knuckle_joint" type="revolute">
@@ -270,5 +240,6 @@
       <child link="${prefix}right_outer_bar" />
       <axis xyz="1 0 0" />
-      <limit effort="0" lower="-0.155" upper="0.7854" velocity="2.0" />
+      <limit effort="0" lower="-0.155" upper="0.7854" velocity="2.0"
+        acceleration="8" deceleration="8" jerk="64" />
       <mimic joint="${prefix}left_outer_knuckle_joint" multiplier="1" offset="0" />
     </joint>
@@ -278,5 +249,6 @@
       <child link="${prefix}right_inner_bar" />
       <axis xyz="1 0 0" />
-      <limit effort="0" lower="-0.155" upper="0.7854" velocity="2.0" />
+      <limit effort="0" lower="-0.155" upper="0.7854" velocity="2.0"
+        acceleration="8" deceleration="8" jerk="64" />
       <mimic joint="${prefix}left_outer_knuckle_joint" multiplier="1" offset="0" />
     </joint>
@@ -286,5 +258,6 @@
       <child link="${prefix}right_finger_mount" />
       <axis xyz="1 0 0" />
-      <limit effort="0" lower="-0.7854" upper="0.155" velocity="2.0" />
+      <limit effort="0" lower="-0.7854" upper="0.155" velocity="2.0"
+        acceleration="8" deceleration="8" jerk="64" />
       <mimic joint="${prefix}left_outer_knuckle_joint" multiplier="-1" offset="0" />
     </joint>
@@ -293,10 +266,4 @@
       <parent link="${prefix}right_finger_mount" />
       <child link="${prefix}right_finger_tip" />
-      <axis xyz="0 0 1" />
-    </joint>
-    <joint name="${prefix}right_finger_tcp_joint" type="fixed">
-      <origin rpy="0 0 0" xyz="0 0.0135 0.036" />
-      <parent link="${prefix}right_finger_tip" />
-      <child link="${prefix}right_finger_tcp" />
       <axis xyz="0 0 1" />
     </joint>
@@ -313,5 +280,6 @@
       <child link="${prefix}unused_finger_width_link" />
       <axis xyz="1 0 0" />
-      <limit effort="80" lower="0" upper="0.100" velocity="0.2" />
+      <limit effort="80" lower="0" upper="0.100" velocity="0.2"
+        acceleration="0.8" deceleration="0.8" jerk="6.4" />
     </joint>
     <link name="${prefix}unused_finger_width_link">

File: urdf/flexiv.urdf.xacro (robot description, xacro)
@@ -1,4 +1,5 @@
 <?xml version="1.0" encoding="utf-8"?>
-<robot xmlns:xacro="http://www.ros.org/wiki/xacro" name="$(arg robot_type)">
+<!-- URDF 1.2: required for the acceleration/deceleration/jerk joint limits to be parsed -->
+<robot xmlns:xacro="http://www.ros.org/wiki/xacro" name="$(arg robot_type)" version="1.2">
   <!-- Single entry point for every Flexiv robot model. 'robot_type' values:
     Single arm on a mount (one robot_sn):
@@ -13,5 +14,6 @@
     Two paired robots (robot_sn_left + robot_sn_right, 'arm_type_left/right'):
       Rizon-Dual   two arms on a shared mount, no external axis
-      AICO2-4-V1, AICO2-4-V2, AICO2-10-V1
+      AICO2-4-V1, AICO2-4-V2, AICO2-4-D3, AICO2-4E-D1, AICO2-4U-D1
+      AICO2-10-V1, AICO2-10-D2, AICO2-10E-D1, AICO2-10U-D1
   -->
   <xacro:arg name="robot_type" default="Enlight-L" />
@@ -66,6 +68,8 @@
   <xacro:property name="is_dual" value="${is_enlight_ll or is_mico}" />
   <xacro:property name="is_aico1" value="${robot_type_str in ['AICO1-4-V1', 'AICO1-4-V2']}" />
-  <xacro:property name="is_aico2"
-    value="${robot_type_str in ['AICO2-4-V1', 'AICO2-4-V2', 'AICO2-10-V1']}" />
+  <xacro:property name="aico2_types"
+    value="${['AICO2-4-V1', 'AICO2-4-V2', 'AICO2-4-D3', 'AICO2-4E-D1', 'AICO2-4U-D1',
+              'AICO2-10-V1', 'AICO2-10-D2', 'AICO2-10E-D1', 'AICO2-10U-D1']}" />
+  <xacro:property name="is_aico2" value="${robot_type_str in aico2_types}" />
   <xacro:property name="is_rizon_dual" value="${robot_type_str == 'Rizon-Dual'}" />
   <!-- 'Paired' means two robots with two serial numbers, as opposed to one robot
@@ -248,22 +252,22 @@
        one robot with two arms on a single robot_sn. -->
   <xacro:if value="${is_paired}">
-    <!-- AICO2-10-V1 carries two Rizon10; the -4- variants carry a Rizon4 / Rizon4R
-         mirrored pair, which is also the default for a plain Rizon-Dual. -->
-    <xacro:property name="paired_default_left"
-      value="${'Rizon10' if robot_type_str == 'AICO2-10-V1' else 'Rizon4'}" />
+    <!-- The AICO2-10 variants carry two Rizon10; the AICO2-4 ones carry a Rizon4 /
+         Rizon4R mirrored pair, which is also the default for a plain Rizon-Dual. -->
+    <xacro:property name="is_aico2_10" value="${robot_type_str.startswith('AICO2-10')}" />
+    <xacro:property name="paired_default_left" value="${'Rizon10' if is_aico2_10 else 'Rizon4'}" />
     <xacro:property name="paired_default_right"
-      value="${'Rizon10R' if robot_type_str == 'AICO2-10-V1' else 'Rizon4R'}" />
+      value="${'Rizon10R' if is_aico2_10 else 'Rizon4R'}" />
     <xacro:property name="arm_left"
       value="${'$(arg arm_type_left)' if '$(arg arm_type_left)' != '' else paired_default_left}" />
     <xacro:property name="arm_right"
       value="${'$(arg arm_type_right)' if '$(arg arm_type_right)' != '' else paired_default_right}" />
-    <xacro:if value="${robot_type_str in ['AICO2-4-V1', 'AICO2-4-V2']}">
+    <xacro:if value="${is_aico2 and not is_aico2_10}">
       <xacro:unless value="${arm_left in ['Rizon4', 'Rizon4s', 'Rizon4R'] and arm_right in ['Rizon4', 'Rizon4s', 'Rizon4R']}">
         ${xacro.warning(robot_type_str + ' carries Rizon4-class arms. You selected ' + arm_left + ' and ' + arm_right + '.')}
       </xacro:unless>
     </xacro:if>
-    <xacro:if value="${robot_type_str == 'AICO2-10-V1'}">
+    <xacro:if value="${is_aico2_10}">
       <xacro:unless value="${arm_left in ['Rizon10', 'Rizon10R'] and arm_right in ['Rizon10', 'Rizon10R']}">
-        ${xacro.warning('AICO2-10-V1 carries Rizon10-class arms. You selected ' + arm_left + ' and ' + arm_right + '.')}
+        ${xacro.warning(robot_type_str + ' carries Rizon10-class arms. You selected ' + arm_left + ' and ' + arm_right + '.')}
       </xacro:unless>
     </xacro:if>
@@ -280,5 +284,11 @@
       <xacro:include filename="$(find flexiv_description)/urdf/common/aico2_4_v1.xacro" />
       <xacro:include filename="$(find flexiv_description)/urdf/common/aico2_4_v2.xacro" />
+      <xacro:include filename="$(find flexiv_description)/urdf/common/aico2_4_d3.xacro" />
+      <xacro:include filename="$(find flexiv_description)/urdf/common/aico2_4e_d1.xacro" />
+      <xacro:include filename="$(find flexiv_description)/urdf/common/aico2_4u_d1.xacro" />
       <xacro:include filename="$(find flexiv_description)/urdf/common/aico2_10_v1.xacro" />
+      <xacro:include filename="$(find flexiv_description)/urdf/common/aico2_10_d2.xacro" />
+      <xacro:include filename="$(find flexiv_description)/urdf/common/aico2_10e_d1.xacro" />
+      <xacro:include filename="$(find flexiv_description)/urdf/common/aico2_10u_d1.xacro" />
       <joint name="world_to_platform" type="fixed">
         <parent link="world" />
@@ -286,19 +296,9 @@
         <origin xyz="0 0 0" rpy="0 0 0" />
       </joint>
-      <xacro:if value="${robot_type_str == 'AICO2-4-V1'}">
-        <xacro:aico2_4_v1 prefix="$(arg external_axis_prefix)"
-          left_arm_prefix="${prefix_left}" right_arm_prefix="${prefix_right}"
-          mesh_prefix_path="package://flexiv_description/" />
-      </xacro:if>
-      <xacro:if value="${robot_type_str == 'AICO2-4-V2'}">
-        <xacro:aico2_4_v2 prefix="$(arg external_axis_prefix)"
-          left_arm_prefix="${prefix_left}" right_arm_prefix="${prefix_right}"
-          mesh_prefix_path="package://flexiv_description/" />
-      </xacro:if>
-      <xacro:if value="${robot_type_str == 'AICO2-10-V1'}">
-        <xacro:aico2_10_v1 prefix="$(arg external_axis_prefix)"
-          left_arm_prefix="${prefix_left}" right_arm_prefix="${prefix_right}"
-          mesh_prefix_path="package://flexiv_description/" />
-      </xacro:if>
+      <!-- Every AICO2 macro is named after its robot type and takes the same
+           parameters, so the selected one can be called by name. -->
+      <xacro:call macro="${external_axis_type}" prefix="$(arg external_axis_prefix)"
+        left_arm_prefix="${prefix_left}" right_arm_prefix="${prefix_right}"
+        mesh_prefix_path="package://flexiv_description/" />
       <xacro:property name="paired_left_xyz" value="0.0 0.0 0.0" />
       <xacro:property name="paired_left_rpy" value="0.0 0.0 0.0" />
