Commit message: Remove Rizon robot meshes and update URDF xacro files

File: urdf/common/enlight_arm.xacro (robot description, xacro)
@@ -1,5 +1,5 @@
 <?xml version="1.0"?>
 <robot xmlns:xacro="http://wiki.ros.org/xacro">
-  <xacro:include filename="$(find flexiv_description)/urdf/common/rizon_common.xacro" />
+  <xacro:include filename="$(find flexiv_description)/urdf/common/flexiv_common.xacro" />
   <xacro:macro name="enlight_arm"
     params="

File: urdf/common/enlight_robot.xacro (robot description, xacro)
@@ -22,6 +22,4 @@
     base_xyz:='0.0 0.0 0.0'
     base_rpy:='0.0 0.0 0.0'
-    external_axis_type:=''
-    external_axis_prefix:=''
     ">
     <xacro:property name="prefix"
@@ -45,12 +43,10 @@
     />
     <xacro:if value="${ros2_control}">
-      <xacro:include filename="$(find flexiv_description)/urdf/common/rizon.ros2_control.xacro" />
-      <xacro:rizon_ros2_control prefix="${prefix}" robot_sn="${robot_sn}"
+      <xacro:include filename="$(find flexiv_description)/urdf/common/flexiv.ros2_control.xacro" />
+      <xacro:flexiv_ros2_control prefix="${prefix}" robot_sn="${robot_sn}"
         rdk_control_mode="${rdk_control_mode}"
         use_fake_hardware="${use_fake_hardware}"
         fake_sensor_commands="${fake_sensor_commands}"
         initial_positions_file="${initial_positions_file}"
-        external_axis_type="${external_axis_type}"
-        external_axis_prefix="${external_axis_prefix}"
       />
     </xacro:if>

File: urdf/common/flexiv.ros2_control.xacro (robot description, xacro)
@@ -1,5 +1,5 @@
 <?xml version="1.0"?>
 <robot xmlns:xacro="http://www.ros.org/wiki/xacro">
-  <xacro:macro name="rizon_ros2_control"
+  <xacro:macro name="flexiv_ros2_control"
     params="
     prefix
@@ -9,6 +9,4 @@
     fake_sensor_commands:=false
     initial_positions_file
-    external_axis_type:=''
-    external_axis_prefix:=''
     ">
     <xacro:property name="initial_positions" value="${xacro.load_yaml(initial_positions_file)['initial_positions']}"/>
@@ -97,49 +95,4 @@
         <state_interface name="effort" />
       </joint>
-      <!-- External axis joints -->
-      <xacro:if value="${external_axis_type == 'aico1_4_v1'}">
-        <joint name="${external_axis_prefix}aico1_4_v1_joint2">
-          <command_interface name="position" />
-          <command_interface name="velocity" />
-          <command_interface name="effort" />
-          <state_interface name="position">
-            <param name="initial_value">0.0</param>
-          </state_interface>
-          <state_interface name="velocity" />
-          <state_interface name="effort" />
-        </joint>
-      </xacro:if>
-      <xacro:if value="${external_axis_type == 'aico1_4_v2'}">
-        <joint name="${external_axis_prefix}aico1_4_v2_joint1">
-          <command_interface name="position" />
-          <command_interface name="velocity" />
-          <command_interface name="effort" />
-          <state_interface name="position">
-            <param name="initial_value">0.0</param>
-          </state_interface>
-          <state_interface name="velocity" />
-          <state_interface name="effort" />
-        </joint>
-        <joint name="${external_axis_prefix}aico1_4_v2_joint2">
-          <command_interface name="position" />
-          <command_interface name="velocity" />
-          <command_interface name="effort" />
-          <state_interface name="position">
-            <param name="initial_value">0.0</param>
-          </state_interface>
-          <state_interface name="velocity" />
-          <state_interface name="effort" />
-        </joint>
-        <joint name="${external_axis_prefix}aico1_4_v2_joint_head">
-          <command_interface name="position" />
-          <command_interface name="velocity" />
-          <command_interface name="effort" />
-          <state_interface name="position">
-            <param name="initial_value">0.0</param>
-          </state_interface>
-          <state_interface name="velocity" />
-          <state_interface name="effort" />
-        </joint>
-      </xacro:if>
       <!-- 24 digital IO ports (16 on control box + 2 inside the wrist connector per wrist, max 4 wrists) -->
       <xacro:macro name="loop_gpio" params="idx">

File: urdf/flexiv.urdf.xacro (robot description, xacro)
@@ -1,9 +1,7 @@
 <?xml version="1.0" encoding="utf-8"?>
 <robot xmlns:xacro="http://www.ros.org/wiki/xacro" name="$(arg robot_type)">
-  <!-- 'robot_type' values: EnlightL, Rizon4, Rizon4s, Rizon4M, Rizon4R, Rizon10, Rizon10s -->
-  <xacro:arg name="rizon_type" default="Rizon4" />
-  <xacro:arg name="robot_type" default="$(arg rizon_type)" />
-  <!-- import model macros -->
-  <xacro:include filename="$(find flexiv_description)/urdf/common/rizon_robot.xacro" />
+  <!-- 'robot_type' values: EnlightL -->
+  <xacro:arg name="robot_type" default="EnlightL" />
+  <!-- import model macro -->
   <xacro:include filename="$(find flexiv_description)/urdf/common/enlight_robot.xacro" />
   <!-- parameters -->
@@ -29,87 +27,43 @@
   <xacro:arg name="mounting_file" default="$(find flexiv_description)/config/single_robot_mounting.yaml" />
   <xacro:property name="mounting" value="${xacro.load_yaml('$(arg mounting_file)')}" />
-  <xacro:if value="${'$(arg robot_type)' == 'EnlightL'}">
-    <xacro:if value="${'$(arg initial_positions_file)' == ''}">
-      <xacro:enlight_robot
-        robot_type="$(arg robot_type)"
-        robot_sn="$(arg robot_sn)"
-        joint_limits_parameters_file="$(arg joint_limits_parameters_file)"
-        kinematics_parameters_file="$(arg kinematics_parameters_file)"
-        inertia_parameters_file="$(arg inertia_parameters_file)"
-        visual_parameters_file="$(arg visual_parameters_file)"
-        arm_prefix="$(arg arm_prefix)"
-        load_gripper="$(arg load_gripper)"
-        gripper_name="$(arg gripper_name)"
-        load_mounted_ft_sensor="$(arg load_mounted_ft_sensor)"
-        ros2_control="$(arg ros2_control)"
-        rdk_control_mode="$(arg rdk_control_mode)"
-        use_fake_hardware="$(arg use_fake_hardware)"
-        fake_sensor_commands="$(arg fake_sensor_commands)"
-        initial_positions_file="$(find flexiv_description)/config/EnlightL/initial_positions.yaml"
-        base_rpy="${radians(mounting['orientation']['rx'])} ${radians(mounting['orientation']['ry'])} ${radians(mounting['orientation']['rz'])}">
-      </xacro:enlight_robot>
-    </xacro:if>
-    <xacro:unless value="${'$(arg initial_positions_file)' == ''}">
-      <xacro:enlight_robot
-        robot_type="$(arg robot_type)"
-        robot_sn="$(arg robot_sn)"
-        joint_limits_parameters_file="$(arg joint_limits_parameters_file)"
-        kinematics_parameters_file="$(arg kinematics_parameters_file)"
-        inertia_parameters_file="$(arg inertia_parameters_file)"
-        visual_parameters_file="$(arg visual_parameters_file)"
-        arm_prefix="$(arg arm_prefix)"
-        load_gripper="$(arg load_gripper)"
-        gripper_name="$(arg gripper_name)"
-        load_mounted_ft_sensor="$(arg load_mounted_ft_sensor)"
-        ros2_control="$(arg ros2_control)"
-        rdk_control_mode="$(arg rdk_control_mode)"
-        use_fake_hardware="$(arg use_fake_hardware)"
-        fake_sensor_commands="$(arg fake_sensor_commands)"
-        initial_positions_file="$(arg initial_positions_file)"
-        base_rpy="${radians(mounting['orientation']['rx'])} ${radians(mounting['orientation']['ry'])} ${radians(mounting['orientation']['rz'])}">
-      </xacro:enlight_robot>
-    </xacro:unless>
+  <xacro:if value="${'$(arg initial_positions_file)' == ''}">
+    <xacro:enlight_robot
+      robot_type="$(arg robot_type)"
+      robot_sn="$(arg robot_sn)"
+      joint_limits_parameters_file="$(arg joint_limits_parameters_file)"
+      kinematics_parameters_file="$(arg kinematics_parameters_file)"
+      inertia_parameters_file="$(arg inertia_parameters_file)"
+      visual_parameters_file="$(arg visual_parameters_file)"
+      arm_prefix="$(arg arm_prefix)"
+      load_gripper="$(arg load_gripper)"
+      gripper_name="$(arg gripper_name)"
+      load_mounted_ft_sensor="$(arg load_mounted_ft_sensor)"
+      ros2_control="$(arg ros2_control)"
+      rdk_control_mode="$(arg rdk_control_mode)"
+      use_fake_hardware="$(arg use_fake_hardware)"
+      fake_sensor_commands="$(arg fake_sensor_commands)"
+      initial_positions_file="$(find flexiv_description)/config/EnlightL/initial_positions.yaml"
+      base_rpy="${radians(mounting['orientation']['rx'])} ${radians(mounting['orientation']['ry'])} ${radians(mounting['orientation']['rz'])}">
+    </xacro:enlight_robot>
   </xacro:if>
-  <xacro:unless value="${'$(arg robot_type)' == 'EnlightL'}">
-    <xacro:if value="${'$(arg initial_positions_file)' == ''}">
-      <xacro:rizon_robot
-        rizon_type="$(arg robot_type)"
-        robot_sn="$(arg robot_sn)"
-        joint_limits_parameters_file="$(arg joint_limits_parameters_file)"
-        kinematics_parameters_file="$(arg kinematics_parameters_file)"
-        inertia_parameters_file="$(arg inertia_parameters_file)"
-        visual_parameters_file="$(arg visual_parameters_file)"
-        arm_prefix="$(arg arm_prefix)"
-        load_gripper="$(arg load_gripper)"
-        gripper_name="$(arg gripper_name)"
-        load_mounted_ft_sensor="$(arg load_mounted_ft_sensor)"
-        ros2_control="$(arg ros2_control)"
-        rdk_control_mode="$(arg rdk_control_mode)"
-        use_fake_hardware="$(arg use_fake_hardware)"
-        fake_sensor_commands="$(arg fake_sensor_commands)"
-        initial_positions_file="$(find flexiv_description)/config/initial_positions.yaml"
-        base_rpy="${radians(mounting['orientation']['rx'])} ${radians(mounting['orientation']['ry'])} ${radians(mounting['orientation']['rz'])}">
-      </xacro:rizon_robot>
-    </xacro:if>
-    <xacro:unless value="${'$(arg initial_positions_file)' == ''}">
-      <xacro:rizon_robot
-        rizon_type="$(arg robot_type)"
-        robot_sn="$(arg robot_sn)"
-        joint_limits_parameters_file="$(arg joint_limits_parameters_file)"
-        kinematics_parameters_file="$(arg kinematics_parameters_file)"
-        inertia_parameters_file="$(arg inertia_parameters_file)"
-        visual_parameters_file="$(arg visual_parameters_file)"
-        arm_prefix="$(arg arm_prefix)"
-        load_gripper="$(arg load_gripper)"
-        gripper_name="$(arg gripper_name)"
-        load_mounted_ft_sensor="$(arg load_mounted_ft_sensor)"
-        ros2_control="$(arg ros2_control)"
-        rdk_control_mode="$(arg rdk_control_mode)"
-        use_fake_hardware="$(arg use_fake_hardware)"
-        fake_sensor_commands="$(arg fake_sensor_commands)"
-        initial_positions_file="$(arg initial_positions_file)"
-        base_rpy="${radians(mounting['orientation']['rx'])} ${radians(mounting['orientation']['ry'])} ${radians(mounting['orientation']['rz'])}">
-      </xacro:rizon_robot>
-    </xacro:unless>
+  <xacro:unless value="${'$(arg initial_positions_file)' == ''}">
+    <xacro:enlight_robot
+      robot_type="$(arg robot_type)"
+      robot_sn="$(arg robot_sn)"
+      joint_limits_parameters_file="$(arg joint_limits_parameters_file)"
+      kinematics_parameters_file="$(arg kinematics_parameters_file)"
+      inertia_parameters_file="$(arg inertia_parameters_file)"
+      visual_parameters_file="$(arg visual_parameters_file)"
+      arm_prefix="$(arg arm_prefix)"
+      load_gripper="$(arg load_gripper)"
+      gripper_name="$(arg gripper_name)"
+      load_mounted_ft_sensor="$(arg load_mounted_ft_sensor)"
+      ros2_control="$(arg ros2_control)"
+      rdk_control_mode="$(arg rdk_control_mode)"
+      use_fake_hardware="$(arg use_fake_hardware)"
+      fake_sensor_commands="$(arg fake_sensor_commands)"
+      initial_positions_file="$(arg initial_positions_file)"
+      base_rpy="${radians(mounting['orientation']['rx'])} ${radians(mounting['orientation']['ry'])} ${radians(mounting['orientation']['rz'])}">
+    </xacro:enlight_robot>
   </xacro:unless>
 </robot>
