Commit message: fix: make load_mounted_ft_sensor functional again
Two defects made the mounted FT sensor impossible to load through
flexiv.urdf.xacro on this branch:

- enlight_robot.xacro unconditionally reassigned its own incoming param
  (<xacro:property name="load_mounted_ft_sensor" value="false"/>), so
  the caller's value was always discarded. Remove the line.
- enlight_arm.xacro resolved the sensor yamls from config/FT03-D1/, which
  does not exist; only config/FT03/ does. humble-v1's rizon_arm.xacro used
  config/FT03/ correctly, so the v2 rename was applied to the path but not
  to the directory. Point the paths back at config/FT03/.

The first defect masked the second, which is why neither surfaced.

Verified: robot_type:=Enlight-L and robot_type:=Rizon4 each emit 0
wrist-sensor elements by default and 12 with load_mounted_ft_sensor:=true.

File: urdf/common/enlight_arm.xacro (robot description, xacro)
@@ -21,7 +21,7 @@
       visual_parameters_file="${visual_parameters_file}"
       load_mounted_ft_sensor="${load_mounted_ft_sensor}"
-      sensor_kinematics_file="$(find flexiv_description)/config/FT03-D1/ft_sensor_kinematics.yaml"
-      sensor_inertia_file="$(find flexiv_description)/config/FT03-D1/ft_sensor_inertia.yaml"
-      sensor_visual_file="$(find flexiv_description)/config/FT03-D1/ft_sensor_visual.yaml"
+      sensor_kinematics_file="$(find flexiv_description)/config/FT03/ft_sensor_kinematics.yaml"
+      sensor_inertia_file="$(find flexiv_description)/config/FT03/ft_sensor_inertia.yaml"
+      sensor_visual_file="$(find flexiv_description)/config/FT03/ft_sensor_visual.yaml"
     />
     <xacro:if value="${create_base_joint}">

File: urdf/common/enlight_robot.xacro (robot description, xacro)
@@ -25,5 +25,4 @@
     <xacro:property name="prefix"
       value="${(arm_prefix + '_' + robot_sn + '_') if arm_prefix != '' and robot_sn != '' else (arm_prefix + robot_sn + '_') if (arm_prefix + robot_sn) != '' else ''}" />
-    <xacro:property name="load_mounted_ft_sensor" value="false" />
     <xacro:if value="${load_gripper and gripper_name=='Flexiv-GN01'}">
       <xacro:include filename="$(find flexiv_description)/urdf/common/grav_macro.xacro" />
