Commit message: Add material definition for flexiv_black

File: urdf/common/grav_macro.xacro (robot description, xacro)
@@ -328,8 +328,4 @@
       <child link="${prefix}grav_base_link" />
     </joint>
-    <!-- materials -->
-    <material name="flexiv_black">
-      <color rgba="0.22 0.22 0.22 1" />
-    </material>
   </xacro:macro>
 </robot>

File: urdf/flexiv.urdf.xacro (robot description, xacro)
@@ -6,4 +6,7 @@
        MICO-Ultra (2-DOF waist torso on mobile base + two Enlight-L arms). -->
   <xacro:arg name="robot_type" default="Enlight-L" />
+  <material name="flexiv_black">
+    <color rgba="0.22 0.22 0.22 1" />
+  </material>
   <!-- import model macro -->
   <xacro:include filename="$(find flexiv_description)/urdf/common/enlight_robot.xacro" />
