Commit message: Move Grav TCP to 0.18 m via base_to_tcp and drop the extra finger TCP frames

File: urdf/common/grav_macro.xacro (robot description, xacro)
@@ -185,6 +185,6 @@
       </collision>
     </link>
-    <!-- TCP links -->
-    <link name="${prefix}grav_tcp"><!-- open finger, used by RCA -->
+    <!-- TCP between the open finger tips -->
+    <link name="${prefix}grav_tcp">
       <inertial>
         <origin rpy="0 0 0" xyz="0 0 0" />
@@ -193,36 +193,9 @@
       </inertial>
     </link>
-    <link name="${prefix}closed_fingers_tcp">
-      <inertial>
-        <origin rpy="0 0 0" xyz="0 0 0" />
-        <mass value="0" />
-        <inertia ixx="0" ixy="0" ixz="0" iyy="0" iyz="0" izz="0" />
-      </inertial>
-    </link>
-    <link name="${prefix}left_finger_tcp">
-      <inertial>
-        <origin rpy="0 0 0" xyz="0 0 0" />
-        <mass value="0" />
-        <inertia ixx="0" ixy="0" ixz="0" iyy="0" iyz="0" izz="0" />
-      </inertial>
-    </link>
-    <link name="${prefix}right_finger_tcp">
-      <inertial>
-        <origin rpy="0 0 0" xyz="0 0 0" />
-        <mass value="0" />
-        <inertia ixx="0" ixy="0" ixz="0" iyy="0" iyz="0" izz="0" />
-      </inertial>
-    </link>
     <!-- JOINTS -->
-    <joint name="${prefix}open_fingers_tcp_joint" type="fixed">
-      <origin rpy="0 0 0" xyz="0 0 0.15" />
+    <joint name="${prefix}base_to_tcp" type="fixed">
+      <origin rpy="0 0 0" xyz="0 0 0.18" />
       <parent link="${prefix}grav_base_link" />
       <child link="${prefix}grav_tcp" />
-      <axis xyz="0 0 1" />
-    </joint>
-    <joint name="${prefix}closed_fingers_tcp_joint" type="fixed">
-      <origin rpy="0 0 0" xyz="0 0 0.20" />
-      <parent link="${prefix}grav_base_link" />
-      <child link="${prefix}closed_fingers_tcp" />
       <axis xyz="0 0 1" />
     </joint>
@@ -258,10 +231,4 @@
       <axis xyz="0 0 1" />
     </joint>
-    <joint name="${prefix}left_finger_tcp_joint" type="fixed">
-      <origin rpy="0 0 0" xyz="0 0.0135 0.036" />
-      <parent link="${prefix}left_finger_tip" />
-      <child link="${prefix}left_finger_tcp" />
-      <axis xyz="0 0 1" />
-    </joint>
     <!-- right finger joints -->
     <joint name="${prefix}right_outer_knuckle_joint" type="revolute">
@@ -293,10 +260,4 @@
       <parent link="${prefix}right_finger_mount" />
       <child link="${prefix}right_finger_tip" />
-      <axis xyz="0 0 1" />
-    </joint>
-    <joint name="${prefix}right_finger_tcp_joint" type="fixed">
-      <origin rpy="0 0 0" xyz="0 0.0135 0.036" />
-      <parent link="${prefix}right_finger_tip" />
-      <child link="${prefix}right_finger_tcp" />
       <axis xyz="0 0 1" />
     </joint>
