Commit message: feat: parameterize GPIO port count and external axis in single-robot control
Adds three optional params to flexiv_ros2_control, forwarded by
enlight_robot. All default to the current behavior, so Enlight-L and MICO
output is unchanged (verified: still 20 digital_output interfaces).

- num_gpio_ports (default 20) replaces the hardcoded loop bound. Digital IO
  is 16 control-box ports plus 2 per wrist connector, so Enlight-L and MICO
  have 20 but Rizon has 18. Without this the restored Rizon models would
  inherit two GPIO ports their hardware does not have.
- external_axis_type / external_axis_prefix re-enable the AICO1 external-axis
  joints, which humble-v1's rizon.ros2_control.xacro emitted and the v2
  rewrite dropped. AICO1 mounts a single arm on a positioner, so its axis
  joints belong to this single-robot interface, not the paired one.

The repeated external-axis joint blocks are collapsed into an ext_axis_joint
macro rather than restored as three verbatim copies.

File: urdf/common/enlight_robot.xacro (robot description, xacro)
@@ -22,4 +22,7 @@
     base_xyz:='0.0 0.0 0.0'
     base_rpy:='0.0 0.0 0.0'
+    num_gpio_ports:=20
+    external_axis_type:=''
+    external_axis_prefix:=''
     ">
     <xacro:property name="prefix"
@@ -48,4 +51,7 @@
         fake_sensor_commands="${fake_sensor_commands}"
         initial_positions_file="${initial_positions_file}"
+        num_gpio_ports="${num_gpio_ports}"
+        external_axis_type="${external_axis_type}"
+        external_axis_prefix="${external_axis_prefix}"
       />
     </xacro:if>

File: urdf/common/flexiv.ros2_control.xacro (robot description, xacro)
@@ -1,4 +1,7 @@
 <?xml version="1.0"?>
 <robot xmlns:xacro="http://www.ros.org/wiki/xacro">
+  <!-- Single-robot ros2_control: one robot_sn, one FlexivHardwareInterface.
+       For two robots paired on a platform (Rizon dual, AICO2) see
+       rizon_dual.ros2_control.xacro instead. -->
   <xacro:macro name="flexiv_ros2_control"
     params="
@@ -9,4 +12,7 @@
     fake_sensor_commands:=false
     initial_positions_file
+    num_gpio_ports:=20
+    external_axis_type:=''
+    external_axis_prefix:=''
     ">
     <xacro:property name="initial_positions" value="${xacro.load_yaml(initial_positions_file)['initial_positions']}"/>
@@ -23,4 +29,7 @@
           <param name="prefix">${prefix}</param>
           <param name="rdk_control_mode">${rdk_control_mode}</param>
+          <xacro:unless value="${external_axis_type == ''}">
+            <param name="external_axis_type">${external_axis_type}</param>
+          </xacro:unless>
         </xacro:unless>
       </hardware>
@@ -95,9 +104,33 @@
         <state_interface name="effort" />
       </joint>
-      <!-- 20 digital IO ports (16 on control box + 2 in each wrist connector, max 2 wrists). -->
+      <!-- External axis joints. AICO1 mounts a single arm on a positioner, so
+           the axis joints join this robot's interface rather than a paired one. -->
+      <xacro:macro name="ext_axis_joint" params="name">
+        <joint name="${external_axis_prefix}${name}">
+          <command_interface name="position" />
+          <command_interface name="velocity" />
+          <command_interface name="effort" />
+          <state_interface name="position">
+            <param name="initial_value">0.0</param>
+          </state_interface>
+          <state_interface name="velocity" />
+          <state_interface name="effort" />
+        </joint>
+      </xacro:macro>
+      <xacro:if value="${external_axis_type == 'aico1_4_v1'}">
+        <!-- joint1 is not actuated on this variant. -->
+        <xacro:ext_axis_joint name="aico1_4_v1_joint2" />
+      </xacro:if>
+      <xacro:if value="${external_axis_type == 'aico1_4_v2'}">
+        <xacro:ext_axis_joint name="aico1_4_v2_joint1" />
+        <xacro:ext_axis_joint name="aico1_4_v2_joint2" />
+        <xacro:ext_axis_joint name="aico1_4_v2_joint_head" />
+      </xacro:if>
+      <!-- Digital IO ports: 16 on the control box plus 2 in each wrist connector.
+           Enlight-L and MICO have two wrist connectors (20); Rizon has one (18). -->
       <xacro:macro name="loop_gpio" params="idx">
         <command_interface name="digital_output_${idx}" />
         <state_interface name="digital_input_${idx}" />
-        <xacro:if value="${idx &lt; 19}">
+        <xacro:if value="${idx &lt; num_gpio_ports - 1}">
           <xacro:loop_gpio idx="${idx+1}" />
         </xacro:if>

Commit message: fix: derive arm prefixes from one shared macro (#28)
MICO failed to build with an empty robot_sn. mico_core.xacro named the arm
attachment joint's child link 'left_${robot_sn}_base_link', which becomes
'left__base_link' when robot_sn is empty, while enlight_robot.xacro only
inserts the separating underscore when both arm_prefix and robot_sn are
non-empty and so creates 'left_base_link'. check_urdf then failed with
'child link [left__base_link] ... not found'.

The conditional formula existed in exactly one place, enlight_robot.xacro,
while six other sites hardcoded 'left_${robot_sn}_'. Rather than patch the
one reported site, move the formula into flexiv_common.xacro as
compute_arm_prefix, which exposes the result as 'computed_arm_prefix' via
scope=parent, matching how read_model_data already publishes its values.
Every site now derives prefixes from it, so the two forms cannot diverge
again.

This fixes three further instances of the same defect found while checking
the report:

- MICO-Plus and MICO-Ultra, identical to the reported MICO-Core failure.
- AICO2-4-V1/4-V2/10-V1, whose external axis adapter joints reference the
  arm base links, broken with an empty or one-sided pair of serial numbers.
- A silent variant in Enlight-LL and Rizon-Dual: the tree parsed fine
  because both arms build their own base joints, but the generated
  ros2_control block referenced 'left__joint1' while the URDF declared
  'left_joint1'. That surfaces as a controller-manager failure at runtime
  rather than a parse error, so check_urdf alone did not catch it.

Callers capture the result with lazy_eval=false, otherwise the left and
right captures both resolve to whichever call ran last.

Verified across 32 combinations (every robot type with empty, full and
one-sided serial numbers, plus custom arm and external axis prefixes): all
produce a valid tree and no ros2_control joint reference without a matching
URDF joint. Output for non-empty serial numbers is byte-identical to before
this change for all nine representative models, so existing users see no
difference.

Torso and GPIO names still interpolate robot_sn directly ('${robot_sn}_torso_',
'${robot_sn}_gpio'). With an empty serial number those read '_torso_' and
'_gpio', which is cosmetic rather than broken because the producing and
consuming sites share the one expression. Left alone to keep this change
scoped.

File: urdf/common/enlight_robot.xacro (robot description, xacro)
@@ -26,6 +26,7 @@
     external_axis_prefix:=''
     ">
-    <xacro:property name="prefix"
-      value="${(arm_prefix + '_' + robot_sn + '_') if arm_prefix != '' and robot_sn != '' else (arm_prefix + robot_sn + '_') if (arm_prefix + robot_sn) != '' else ''}" />
+    <xacro:include filename="$(find flexiv_description)/urdf/common/flexiv_common.xacro" />
+    <xacro:compute_arm_prefix arm_prefix="${arm_prefix}" robot_sn="${robot_sn}" />
+    <xacro:property name="prefix" value="${computed_arm_prefix}" />
     <xacro:if value="${load_gripper and gripper_name=='Flexiv-GN01'}">
       <xacro:include filename="$(find flexiv_description)/urdf/common/grav_macro.xacro" />

File: urdf/common/flexiv_common.xacro (robot description, xacro)
@@ -1,4 +1,16 @@
 <?xml version="1.0"?>
 <robot xmlns:xacro="http://wiki.ros.org/xacro">
+  <!--
+    Compute an arm's joint/link name prefix and expose it to the caller as
+    'computed_arm_prefix'.
+    This is the single source of truth for the prefix.
+    arm_prefix: 'left', 'right' or '' (user-supplied prefixes also allowed)
+    robot_sn:   robot serial number, may be empty
+  -->
+  <xacro:macro name="compute_arm_prefix" params="arm_prefix:='' robot_sn:=''">
+    <xacro:property name="computed_arm_prefix"
+      value="${(arm_prefix + '_' + robot_sn + '_') if arm_prefix != '' and robot_sn != '' else (arm_prefix + robot_sn + '_') if (arm_prefix + robot_sn) != '' else ''}"
+      scope="parent" />
+  </xacro:macro>
   <!--
     Extract visual parameters from the config file

File: urdf/common/mico_core.xacro (robot description, xacro)
@@ -29,4 +29,10 @@
     <xacro:property name="arm_cfg" value="$(find flexiv_description)/config/Enlight-L" />
     <xacro:property name="torso_prefix" value="${robot_sn}_torso_" />
+    <!-- Must match the prefixes enlight_robot derives, including when robot_sn is
+         empty. lazy_eval is off so each capture resolves before the next call. -->
+    <xacro:compute_arm_prefix arm_prefix="left" robot_sn="${robot_sn}" />
+    <xacro:property name="prefix_left" value="${computed_arm_prefix}" lazy_eval="false" />
+    <xacro:compute_arm_prefix arm_prefix="right" robot_sn="${robot_sn}" />
+    <xacro:property name="prefix_right" value="${computed_arm_prefix}" lazy_eval="false" />
     <xacro:read_model_data
       joint_limits_parameters_file="${torso_joint_limits_file}"
@@ -117,10 +123,10 @@
     <joint name="${torso_prefix}left_flange_to_left_arm" type="fixed">
       <parent link="${torso_prefix}left_flange" />
-      <child link="left_${robot_sn}_base_link" />
+      <child link="${prefix_left}base_link" />
       <origin xyz="0 0 0" rpy="0 0 0" />
     </joint>
     <joint name="${torso_prefix}right_flange_to_right_arm" type="fixed">
       <parent link="${torso_prefix}right_flange" />
-      <child link="right_${robot_sn}_base_link" />
+      <child link="${prefix_right}base_link" />
       <origin xyz="0 0 0" rpy="0 0 0" />
     </joint>
@@ -128,6 +134,6 @@
     <xacro:if value="${ros2_control}">
       <xacro:flexiv_dual_ros2_control
-        prefix_left="left_${robot_sn}_"
-        prefix_right="right_${robot_sn}_"
+        prefix_left="${prefix_left}"
+        prefix_right="${prefix_right}"
         robot_sn="${robot_sn}"
         rdk_control_mode="${rdk_control_mode}"

File: urdf/common/mico_plus.xacro (robot description, xacro)
@@ -29,4 +29,10 @@
     <xacro:property name="arm_cfg" value="$(find flexiv_description)/config/Enlight-L" />
     <xacro:property name="torso_prefix" value="${robot_sn}_torso_" />
+    <!-- Must match the prefixes enlight_robot derives, including when robot_sn is
+         empty. lazy_eval is off so each capture resolves before the next call. -->
+    <xacro:compute_arm_prefix arm_prefix="left" robot_sn="${robot_sn}" />
+    <xacro:property name="prefix_left" value="${computed_arm_prefix}" lazy_eval="false" />
+    <xacro:compute_arm_prefix arm_prefix="right" robot_sn="${robot_sn}" />
+    <xacro:property name="prefix_right" value="${computed_arm_prefix}" lazy_eval="false" />
     <xacro:read_model_data
       joint_limits_parameters_file="${torso_joint_limits_file}"
@@ -146,10 +152,10 @@
     <joint name="${torso_prefix}left_flange_to_left_arm" type="fixed">
       <parent link="${torso_prefix}left_flange" />
-      <child link="left_${robot_sn}_base_link" />
+      <child link="${prefix_left}base_link" />
       <origin xyz="0 0 0" rpy="0 0 0" />
     </joint>
     <joint name="${torso_prefix}right_flange_to_right_arm" type="fixed">
       <parent link="${torso_prefix}right_flange" />
-      <child link="right_${robot_sn}_base_link" />
+      <child link="${prefix_right}base_link" />
       <origin xyz="0 0 0" rpy="0 0 0" />
     </joint>
@@ -157,6 +163,6 @@
     <xacro:if value="${ros2_control}">
       <xacro:flexiv_mico_ros2_control
-        prefix_left="left_${robot_sn}_"
-        prefix_right="right_${robot_sn}_"
+        prefix_left="${prefix_left}"
+        prefix_right="${prefix_right}"
         robot_sn="${robot_sn}"
         rdk_control_mode="${rdk_control_mode}"

File: urdf/common/mico_ultra.xacro (robot description, xacro)
@@ -30,4 +30,10 @@
     <xacro:property name="arm_cfg" value="$(find flexiv_description)/config/Enlight-L" />
     <xacro:property name="torso_prefix" value="${robot_sn}_torso_" />
+    <!-- Must match the prefixes enlight_robot derives, including when robot_sn is
+         empty. lazy_eval is off so each capture resolves before the next call. -->
+    <xacro:compute_arm_prefix arm_prefix="left" robot_sn="${robot_sn}" />
+    <xacro:property name="prefix_left" value="${computed_arm_prefix}" lazy_eval="false" />
+    <xacro:compute_arm_prefix arm_prefix="right" robot_sn="${robot_sn}" />
+    <xacro:property name="prefix_right" value="${computed_arm_prefix}" lazy_eval="false" />
     <xacro:read_model_data
       joint_limits_parameters_file="${torso_joint_limits_file}"
@@ -146,10 +152,10 @@
     <joint name="${torso_prefix}left_flange_to_left_arm" type="fixed">
       <parent link="${torso_prefix}left_flange" />
-      <child link="left_${robot_sn}_base_link" />
+      <child link="${prefix_left}base_link" />
       <origin xyz="0 0 0" rpy="0 0 0" />
     </joint>
     <joint name="${torso_prefix}right_flange_to_right_arm" type="fixed">
       <parent link="${torso_prefix}right_flange" />
-      <child link="right_${robot_sn}_base_link" />
+      <child link="${prefix_right}base_link" />
       <origin xyz="0 0 0" rpy="0 0 0" />
     </joint>
@@ -157,6 +163,6 @@
     <xacro:if value="${ros2_control}">
       <xacro:flexiv_mico_ros2_control
-        prefix_left="left_${robot_sn}_"
-        prefix_right="right_${robot_sn}_"
+        prefix_left="${prefix_left}"
+        prefix_right="${prefix_right}"
         robot_sn="${robot_sn}"
         rdk_control_mode="${rdk_control_mode}"

File: urdf/flexiv.urdf.xacro (robot description, xacro)
@@ -21,4 +21,5 @@
   </material>
   <!-- import model macro -->
+  <xacro:include filename="$(find flexiv_description)/urdf/common/flexiv_common.xacro" />
   <xacro:include filename="$(find flexiv_description)/urdf/common/enlight_robot.xacro" />
   <!-- parameters -->
@@ -164,9 +165,15 @@
       base_rpy="${radians(right_pose['rx'])} ${radians(right_pose['ry'])} ${radians(right_pose['rz'])}">
     </xacro:enlight_robot>
-    <!-- Single unified ros2_control for both arms (one robot_sn, prefix_left/prefix_right). -->
+    <!-- Single unified ros2_control for both arms (one robot_sn, prefix_left/prefix_right).
+         Prefixes come from compute_arm_prefix so they match the arms' own links even
+         when robot_sn is empty. -->
+    <xacro:compute_arm_prefix arm_prefix="left" robot_sn="$(arg robot_sn)" />
+    <xacro:property name="ll_prefix_left" value="${computed_arm_prefix}" lazy_eval="false" />
+    <xacro:compute_arm_prefix arm_prefix="right" robot_sn="$(arg robot_sn)" />
+    <xacro:property name="ll_prefix_right" value="${computed_arm_prefix}" lazy_eval="false" />
     <xacro:if value="$(arg ros2_control)">
       <xacro:flexiv_dual_ros2_control
-        prefix_left="left_$(arg robot_sn)_"
-        prefix_right="right_$(arg robot_sn)_"
+        prefix_left="${ll_prefix_left}"
+        prefix_right="${ll_prefix_right}"
         robot_sn="$(arg robot_sn)"
         rdk_control_mode="$(arg rdk_control_mode)"
@@ -242,7 +249,7 @@
       <origin xyz="0 0 0" rpy="0 0 0" />
     </joint>
-    <!-- enlight_robot derives the arm prefix as 'arm_prefix_robot_sn_'. -->
-    <xacro:property name="aico1_arm_prefix"
-      value="${('$(arg arm_prefix)' + '_' + '$(arg robot_sn)' + '_') if '$(arg arm_prefix)' != '' and '$(arg robot_sn)' != '' else ('$(arg arm_prefix)' + '$(arg robot_sn)' + '_') if ('$(arg arm_prefix)' + '$(arg robot_sn)') != '' else ''}" />
+    <!-- Must match the prefix enlight_robot derives for this arm. -->
+    <xacro:compute_arm_prefix arm_prefix="$(arg arm_prefix)" robot_sn="$(arg robot_sn)" />
+    <xacro:property name="aico1_arm_prefix" value="${computed_arm_prefix}" lazy_eval="false" />
     <xacro:if value="${robot_type_str == 'AICO1-4-V1'}">
       <xacro:aico1_4_v1 prefix="$(arg external_axis_prefix)"
@@ -303,6 +310,11 @@
       </xacro:unless>
     </xacro:if>
-    <xacro:property name="prefix_left" value="left_$(arg robot_sn_left)_" />
-    <xacro:property name="prefix_right" value="right_$(arg robot_sn_right)_" />
+    <!-- Must match the prefixes enlight_robot derives, including when either serial
+         number is empty. lazy_eval is off so each capture resolves before the next
+         call. -->
+    <xacro:compute_arm_prefix arm_prefix="left" robot_sn="$(arg robot_sn_left)" />
+    <xacro:property name="prefix_left" value="${computed_arm_prefix}" lazy_eval="false" />
+    <xacro:compute_arm_prefix arm_prefix="right" robot_sn="$(arg robot_sn_right)" />
+    <xacro:property name="prefix_right" value="${computed_arm_prefix}" lazy_eval="false" />
     <xacro:property name="init_left" value="${cfg}/${arm_left}/initial_positions.yaml" />
     <xacro:property name="init_right" value="${cfg}/${arm_right}/initial_positions.yaml" />
