Commit message: fix: apply arm prefix naming rule to torso and GPIO names

File: urdf/common/flexiv_dual.ros2_control.xacro (robot description, xacro)
@@ -19,4 +19,9 @@
     initial_positions_file_right
     ">
+    <xacro:include filename="$(find flexiv_description)/urdf/common/flexiv_common.xacro" />
+    <!-- Same omit-separator rule as the arm prefixes, so these names match the ones
+         the model files generate even when robot_sn is empty. -->
+    <xacro:compute_arm_prefix robot_sn="${robot_sn}" />
+    <xacro:property name="sn_prefix" value="${computed_arm_prefix}" lazy_eval="false" />
     <xacro:property name="initial_positions_left"
       value="${xacro.load_yaml(initial_positions_file_left)['initial_positions']}" />
@@ -58,5 +63,6 @@
       <xacro:dual_arm_joints arm_prefix="${prefix_right}" initial_positions="${initial_positions_right}" />
       <!-- Single GPIO block for the whole robot. The unified hardware interface names GPIO
-           interfaces "${robot_sn}_gpio" regardless of arm count. -->
+           interfaces "<robot_sn>_gpio" (or "gpio" when robot_sn is empty) regardless of
+           arm count. -->
       <xacro:macro name="loop_gpio" params="idx">
         <command_interface name="digital_output_${idx}" />
@@ -66,5 +72,5 @@
         </xacro:if>
       </xacro:macro>
-      <gpio name="${robot_sn}_gpio">
+      <gpio name="${sn_prefix}gpio">
         <xacro:loop_gpio idx="0" />
       </gpio>

File: urdf/common/flexiv_mico.ros2_control.xacro (robot description, xacro)
@@ -3,7 +3,7 @@
   <!--
     MICO-Plus / MICO-Ultra ros2_control: mirrors flexiv_dual_ros2_control but additionally emits
-    the 2 torso revolute joints (${robot_sn}_torso_joint1/2). The torso joint prefix
-    intentionally differs from left_/right_ so the hardware interface classifies them as
-    external-axis joints.
+    the 2 torso revolute joints, named "<robot_sn>_torso_joint1/2" (or "torso_joint1/2"
+    when robot_sn is empty). The torso joint prefix intentionally differs from
+    left_/right_ so the hardware interface classifies them as external-axis joints.
   -->
   <xacro:macro name="flexiv_mico_ros2_control"
@@ -19,4 +19,9 @@
     torso_initial_positions_file
     ">
+    <xacro:include filename="$(find flexiv_description)/urdf/common/flexiv_common.xacro" />
+    <!-- Same omit-separator rule as the arm prefixes, so these names match the ones
+         the model files generate even when robot_sn is empty. -->
+    <xacro:compute_arm_prefix robot_sn="${robot_sn}" />
+    <xacro:property name="sn_prefix" value="${computed_arm_prefix}" lazy_eval="false" />
     <xacro:property name="initial_positions_left"
       value="${xacro.load_yaml(initial_positions_file_left)['initial_positions']}" />
@@ -60,5 +65,5 @@
       <xacro:mico_arm_joints arm_prefix="${prefix_right}" initial_positions="${initial_positions_right}" />
       <!-- Torso joints: classified as external-axis joints by the hardware interface. -->
-      <joint name="${robot_sn}_torso_joint1">
+      <joint name="${sn_prefix}torso_joint1">
         <command_interface name="position" />
         <command_interface name="velocity" />
@@ -70,5 +75,5 @@
         <state_interface name="effort" />
       </joint>
-      <joint name="${robot_sn}_torso_joint2">
+      <joint name="${sn_prefix}torso_joint2">
         <command_interface name="position" />
         <command_interface name="velocity" />
@@ -88,5 +93,5 @@
         </xacro:if>
       </xacro:macro>
-      <gpio name="${robot_sn}_gpio">
+      <gpio name="${sn_prefix}gpio">
         <xacro:mico_loop_gpio idx="0" />
       </gpio>

File: urdf/common/mico_core.xacro (robot description, xacro)
@@ -3,5 +3,6 @@
   <!--
     MICO-Core: fixed torso (no actuated torso joints) with two Enlight-L arms.
-    Arm joints: left_${robot_sn}_joint1..7, right_${robot_sn}_joint1..7.
+    Arm joints: left_<robot_sn>_joint1..7, right_<robot_sn>_joint1..7.
+    An empty robot_sn drops the separating underscore, e.g. 'torso_joint1', 'left_joint1'.
     ros2_control: reuses flexiv_dual_ros2_control (no torso joints to add).
   -->
@@ -28,7 +29,11 @@
     ">
     <xacro:property name="arm_cfg" value="$(find flexiv_description)/config/Enlight-L" />
-    <xacro:property name="torso_prefix" value="${robot_sn}_torso_" />
-    <!-- Must match the prefixes enlight_robot derives, including when robot_sn is
-         empty. lazy_eval is off so each capture resolves before the next call. -->
+    <!-- All prefixes follow the same rule as the arms: the separating underscore
+         only appears when the part it separates is non-empty, so an empty robot_sn
+         gives 'torso_base_link' rather than '_torso_base_link'. lazy_eval is off so
+         each capture resolves before the next call. -->
+    <xacro:compute_arm_prefix robot_sn="${robot_sn}" />
+    <xacro:property name="sn_prefix" value="${computed_arm_prefix}" lazy_eval="false" />
+    <xacro:property name="torso_prefix" value="${sn_prefix}torso_" lazy_eval="false" />
     <xacro:compute_arm_prefix arm_prefix="left" robot_sn="${robot_sn}" />
     <xacro:property name="prefix_left" value="${computed_arm_prefix}" lazy_eval="false" />

File: urdf/common/mico_plus.xacro (robot description, xacro)
@@ -3,6 +3,7 @@
   <!--
     MICO-Plus: 2-DOF torso (yaw + pitch) with two Enlight-L arms.
-    Torso joints: ${robot_sn}_torso_joint1 (yaw), ${robot_sn}_torso_joint2 (pitch).
-    Arm joints:   left_${robot_sn}_joint1..7, right_${robot_sn}_joint1..7.
+    Torso joints: <robot_sn>_torso_joint1 (yaw), <robot_sn>_torso_joint2 (pitch).
+    Arm joints:   left_<robot_sn>_joint1..7, right_<robot_sn>_joint1..7.
+    An empty robot_sn drops the separating underscore, e.g. 'torso_joint1', 'left_joint1'.
   -->
   <xacro:include filename="$(find flexiv_description)/urdf/common/flexiv_common.xacro" />
@@ -28,7 +29,11 @@
     ">
     <xacro:property name="arm_cfg" value="$(find flexiv_description)/config/Enlight-L" />
-    <xacro:property name="torso_prefix" value="${robot_sn}_torso_" />
-    <!-- Must match the prefixes enlight_robot derives, including when robot_sn is
-         empty. lazy_eval is off so each capture resolves before the next call. -->
+    <!-- All prefixes follow the same rule as the arms: the separating underscore
+         only appears when the part it separates is non-empty, so an empty robot_sn
+         gives 'torso_base_link' rather than '_torso_base_link'. lazy_eval is off so
+         each capture resolves before the next call. -->
+    <xacro:compute_arm_prefix robot_sn="${robot_sn}" />
+    <xacro:property name="sn_prefix" value="${computed_arm_prefix}" lazy_eval="false" />
+    <xacro:property name="torso_prefix" value="${sn_prefix}torso_" lazy_eval="false" />
     <xacro:compute_arm_prefix arm_prefix="left" robot_sn="${robot_sn}" />
     <xacro:property name="prefix_left" value="${computed_arm_prefix}" lazy_eval="false" />

File: urdf/common/mico_ultra.xacro (robot description, xacro)
@@ -4,6 +4,7 @@
     MICO-Ultra: 2-DOF torso (waist yaw + pitch) with two Enlight-L arms, mounted on a mobile base.
     base_link is the mobile-base root (empty link, no mesh present).
-    Torso joints: ${robot_sn}_torso_joint1 (waist yaw), ${robot_sn}_torso_joint2 (pitch).
-    Arm joints:   left_${robot_sn}_joint1..7, right_${robot_sn}_joint1..7.
+    Torso joints: <robot_sn>_torso_joint1 (waist yaw), <robot_sn>_torso_joint2 (pitch).
+    Arm joints:   left_<robot_sn>_joint1..7, right_<robot_sn>_joint1..7.
+    An empty robot_sn drops the separating underscore, e.g. 'torso_joint1', 'left_joint1'.
   -->
   <xacro:include filename="$(find flexiv_description)/urdf/common/flexiv_common.xacro" />
@@ -29,7 +30,11 @@
     ">
     <xacro:property name="arm_cfg" value="$(find flexiv_description)/config/Enlight-L" />
-    <xacro:property name="torso_prefix" value="${robot_sn}_torso_" />
-    <!-- Must match the prefixes enlight_robot derives, including when robot_sn is
-         empty. lazy_eval is off so each capture resolves before the next call. -->
+    <!-- All prefixes follow the same rule as the arms: the separating underscore
+         only appears when the part it separates is non-empty, so an empty robot_sn
+         gives 'torso_base_link' rather than '_torso_base_link'. lazy_eval is off so
+         each capture resolves before the next call. -->
+    <xacro:compute_arm_prefix robot_sn="${robot_sn}" />
+    <xacro:property name="sn_prefix" value="${computed_arm_prefix}" lazy_eval="false" />
+    <xacro:property name="torso_prefix" value="${sn_prefix}torso_" lazy_eval="false" />
     <xacro:compute_arm_prefix arm_prefix="left" robot_sn="${robot_sn}" />
     <xacro:property name="prefix_left" value="${computed_arm_prefix}" lazy_eval="false" />
