Commit message: feat: rename to flexiv_arm and flexiv_robot macros for robot model configuration

File: urdf/common/flexiv_arm.xacro (robot description, xacro)
@@ -2,5 +2,5 @@
 <robot xmlns:xacro="http://wiki.ros.org/xacro">
   <xacro:include filename="$(find flexiv_description)/urdf/common/flexiv_common.xacro" />
-  <xacro:macro name="enlight_arm"
+  <xacro:macro name="flexiv_arm"
     params="
     prefix
@@ -36,5 +36,5 @@
       <child link="${prefix}link1" />
       <xacro:get_kinematics name="joint1" />
-      <axis xyz="0 0 1" />
+      <xacro:get_joint_axis name="joint1" />
       <xacro:get_joint_limits name="joint1" />
     </joint>
@@ -43,5 +43,5 @@
       <child link="${prefix}link2" />
       <xacro:get_kinematics name="joint2" />
-      <axis xyz="0 0 1" />
+      <xacro:get_joint_axis name="joint2" />
       <xacro:get_joint_limits name="joint2" />
     </joint>
@@ -50,5 +50,5 @@
       <child link="${prefix}link3" />
       <xacro:get_kinematics name="joint3" />
-      <axis xyz="0 0 1" />
+      <xacro:get_joint_axis name="joint3" />
       <xacro:get_joint_limits name="joint3" />
     </joint>
@@ -57,5 +57,5 @@
       <child link="${prefix}link4" />
       <xacro:get_kinematics name="joint4" />
-      <axis xyz="0 0 1" />
+      <xacro:get_joint_axis name="joint4" />
       <xacro:get_joint_limits name="joint4" />
     </joint>
@@ -64,5 +64,5 @@
       <child link="${prefix}link5" />
       <xacro:get_kinematics name="joint5" />
-      <axis xyz="0 0 1" />
+      <xacro:get_joint_axis name="joint5" />
       <xacro:get_joint_limits name="joint5" />
     </joint>
@@ -71,5 +71,5 @@
       <child link="${prefix}link6" />
       <xacro:get_kinematics name="joint6" />
-      <axis xyz="0 0 1" />
+      <xacro:get_joint_axis name="joint6" />
       <xacro:get_joint_limits name="joint6" />
     </joint>
@@ -78,5 +78,5 @@
       <child link="${prefix}link7" />
       <xacro:get_kinematics name="joint7" />
-      <axis xyz="0 0 1" />
+      <xacro:get_joint_axis name="joint7" />
       <xacro:get_joint_limits name="joint7" />
     </joint>

File: urdf/common/flexiv_common.xacro (robot description, xacro)
@@ -95,4 +95,12 @@
   </xacro:macro>
   <!--
+    Extract the joint rotation axis from the config file.
+    name: name of the joint
+  -->
+  <xacro:macro name="get_joint_axis" params="name">
+    <xacro:property name="joint_kinematics" value="${sec_kinematics[name]}" lazy_eval="false" />
+    <axis xyz="${joint_kinematics['axis'] if 'axis' in joint_kinematics else '0 0 1'}" />
+  </xacro:macro>
+  <!--
     Extract inertia parameters from the config file
     name: name of the link

File: urdf/common/flexiv_robot.xacro (robot description, xacro)
@@ -1,5 +1,5 @@
 <?xml version="1.0"?>
 <robot xmlns:xacro="http://wiki.ros.org/xacro">
-  <xacro:macro name="enlight_robot"
+  <xacro:macro name="flexiv_robot"
     params="
     robot_type
@@ -13,16 +13,8 @@
     gripper_name:='Flexiv-GN01'
     load_mounted_ft_sensor:=false
-    ros2_control:=false
-    rdk_control_mode:='joint_position'
-    use_fake_hardware:=false
-    fake_sensor_commands:=false
     add_world_link:=true
     create_base_joint:=true
-    initial_positions_file:='$(find flexiv_description)/config/Enlight-L/initial_positions.yaml'
     base_xyz:='0.0 0.0 0.0'
     base_rpy:='0.0 0.0 0.0'
-    num_gpio_ports:=20
-    external_axis_type:=''
-    external_axis_prefix:=''
     ">
     <xacro:include filename="$(find flexiv_description)/urdf/common/flexiv_common.xacro" />
@@ -33,6 +25,6 @@
       <xacro:flexiv_GN01 prefix="${prefix}" mesh_prefix_path="package://flexiv_description/" />
     </xacro:if>
-    <xacro:include filename="$(find flexiv_description)/urdf/common/enlight_arm.xacro" />
-    <xacro:enlight_arm prefix="${prefix}"
+    <xacro:include filename="$(find flexiv_description)/urdf/common/flexiv_arm.xacro" />
+    <xacro:flexiv_arm prefix="${prefix}"
       load_mounted_ft_sensor="${load_mounted_ft_sensor}"
       joint_limits_parameters_file="${joint_limits_parameters_file}"
@@ -45,16 +37,4 @@
       base_rpy="${base_rpy}"
     />
-    <xacro:if value="${ros2_control}">
-      <xacro:include filename="$(find flexiv_description)/urdf/common/flexiv.ros2_control.xacro" />
-      <xacro:flexiv_ros2_control prefix="${prefix}" robot_sn="${robot_sn}"
-        rdk_control_mode="${rdk_control_mode}"
-        use_fake_hardware="${use_fake_hardware}"
-        fake_sensor_commands="${fake_sensor_commands}"
-        initial_positions_file="${initial_positions_file}"
-        num_gpio_ports="${num_gpio_ports}"
-        external_axis_type="${external_axis_type}"
-        external_axis_prefix="${external_axis_prefix}"
-      />
-    </xacro:if>
   </xacro:macro>
 </robot>

File: urdf/flexiv.urdf.xacro (robot description, xacro)
@@ -2,18 +2,17 @@
 <robot xmlns:xacro="http://www.ros.org/wiki/xacro" name="$(arg robot_type)">
   <!-- Single entry point for every Flexiv robot model. 'robot_type' values:
-       Single arm on a mount (one robot_sn):
-         Enlight-L, Rizon4, Rizon4s, Rizon4M, Rizon4R, Rizon10, Rizon10s
-       One robot with two arms (one robot_sn):
-         Enlight-LL   dual arm on world
-         MICO-Core    fixed torso + two Enlight-L arms
-         MICO-Plus    2-DOF pan-tilt torso + two Enlight-L arms
-         MICO-Ultra   2-DOF waist torso on mobile base + two Enlight-L arms
-       Single arm on an external axis (one robot_sn, use 'arm_type' to pick the arm):
-         AICO1-4-V1, AICO1-4-V2
-       Two paired robots (robot_sn_left + robot_sn_right, 'arm_type_left/right'):
-         Rizon-Dual   two arms on a shared mount, no external axis
-         AICO2-4-V1, AICO2-4-V2, AICO2-10-V1
-       Which of these a given software release actually supports is decided by
-       RDK and RCA. This package is a resource depot and hosts all of them. -->
+    Single arm on a mount (one robot_sn):
+      Enlight-L, Rizon4, Rizon4s, Rizon4M, Rizon4R, Rizon10, Rizon10s
+    One robot with two arms (one robot_sn):
+      Enlight-LL   dual arm on world
+      MICO-Core    fixed torso + two Enlight-L arms
+      MICO-Plus    2-DOF pan-tilt torso + two Enlight-L arms
+      MICO-Ultra   2-DOF waist torso on mobile base + two Enlight-L arms
+    Single arm on an external axis (one robot_sn, use 'arm_type' to pick the arm):
+      AICO1-4-V1, AICO1-4-V2
+    Two paired robots (robot_sn_left + robot_sn_right, 'arm_type_left/right'):
+      Rizon-Dual   two arms on a shared mount, no external axis
+      AICO2-4-V1, AICO2-4-V2, AICO2-10-V1
+  -->
   <xacro:arg name="robot_type" default="Enlight-L" />
   <material name="flexiv_black">
@@ -22,5 +21,5 @@
   <!-- import model macro -->
   <xacro:include filename="$(find flexiv_description)/urdf/common/flexiv_common.xacro" />
-  <xacro:include filename="$(find flexiv_description)/urdf/common/enlight_robot.xacro" />
+  <xacro:include filename="$(find flexiv_description)/urdf/common/flexiv_robot.xacro" />
   <!-- parameters -->
   <xacro:arg name="arm_prefix" default="" />
@@ -37,10 +36,4 @@
   <xacro:arg name="gripper_name" default="Flexiv-GN01" />
   <xacro:arg name="load_mounted_ft_sensor" default="false" />
-  <!-- ros2_control related parameters -->
-  <xacro:arg name="ros2_control" default="false" />
-  <xacro:arg name="rdk_control_mode" default="joint_position" />
-  <xacro:arg name="use_fake_hardware" default="false" />
-  <xacro:arg name="fake_sensor_commands" default="false" />
-  <xacro:arg name="initial_positions_file" default="" />
   <xacro:arg name="mounting_file" default="$(find flexiv_description)/config/single_robot_mounting.yaml" />
   <xacro:arg name="dual_mounting_file" default="$(find flexiv_description)/config/dual_robot_mounting.yaml" />
@@ -48,5 +41,5 @@
   <!-- External axis (AICO) parameters -->
   <xacro:arg name="external_axis_prefix" default="" />
-  <!-- Arm carried by an external axis. Empty means 'pick the default for this axis'. -->
+  <!-- Arm carried by an external axis. -->
   <xacro:arg name="arm_type" default="" />
   <!-- Paired-robot parameters. Only read by Rizon-Dual and AICO2 configurations. -->
@@ -87,12 +80,5 @@
   <xacro:if value="${is_single}">
     <xacro:property name="mounting" value="${xacro.load_yaml('$(arg mounting_file)')}" />
-    <xacro:if value="${'$(arg initial_positions_file)' == ''}">
-      <xacro:property name="resolved_initial_positions_file"
-        value="$(find flexiv_description)/config/$(arg robot_type)/initial_positions.yaml" />
-    </xacro:if>
-    <xacro:unless value="${'$(arg initial_positions_file)' == ''}">
-      <xacro:property name="resolved_initial_positions_file" value="$(arg initial_positions_file)" />
-    </xacro:unless>
-    <xacro:enlight_robot
+    <xacro:flexiv_robot
       robot_type="$(arg robot_type)"
       robot_sn="$(arg robot_sn)"
@@ -105,16 +91,9 @@
       gripper_name="$(arg gripper_name)"
       load_mounted_ft_sensor="$(arg load_mounted_ft_sensor)"
-      ros2_control="$(arg ros2_control)"
-      rdk_control_mode="$(arg rdk_control_mode)"
-      use_fake_hardware="$(arg use_fake_hardware)"
-      fake_sensor_commands="$(arg fake_sensor_commands)"
-      initial_positions_file="${resolved_initial_positions_file}"
-      num_gpio_ports="${18 if robot_type_str.startswith('Rizon') else 20}"
       base_rpy="${radians(mounting['orientation']['rx'])} ${radians(mounting['orientation']['ry'])} ${radians(mounting['orientation']['rz'])}">
-    </xacro:enlight_robot>
+    </xacro:flexiv_robot>
   </xacro:if>
   <!-- ============================== DUAL ARM (Enlight-LL) ============================== -->
   <xacro:if value="${is_enlight_ll}">
-    <xacro:include filename="$(find flexiv_description)/urdf/common/flexiv_dual.ros2_control.xacro" />
     <xacro:property name="dual_mounting" value="${xacro.load_yaml('$(arg dual_mounting_file)')}" />
     <xacro:property name="left_pose" value="${dual_mounting['positions']['left']}" />
@@ -122,7 +101,6 @@
     <!-- Each arm of a dual-arm product is an Enlight-L: reuse its config + meshes for both arms. -->
     <xacro:property name="arm_cfg" value="$(find flexiv_description)/config/Enlight-L" />
-    <xacro:property name="arm_init_positions" value="${arm_cfg}/initial_positions.yaml" />
-    <!-- Left arm: owns the shared world link + its base joint. ros2_control handled below. -->
-    <xacro:enlight_robot
+    <!-- Left arm: owns the shared world link + its base joint. -->
+    <xacro:flexiv_robot
       robot_type="Enlight-L"
       robot_sn="$(arg robot_sn)"
@@ -135,15 +113,11 @@
       gripper_name="$(arg gripper_name)"
       load_mounted_ft_sensor="$(arg load_mounted_ft_sensor)"
-      ros2_control="false"
-      use_fake_hardware="$(arg use_fake_hardware)"
-      fake_sensor_commands="$(arg fake_sensor_commands)"
-      initial_positions_file="${arm_init_positions}"
       add_world_link="true"
       create_base_joint="true"
       base_xyz="${left_pose['x']} ${left_pose['y']} ${left_pose['z']}"
       base_rpy="${radians(left_pose['rx'])} ${radians(left_pose['ry'])} ${radians(left_pose['rz'])}">
-    </xacro:enlight_robot>
+    </xacro:flexiv_robot>
     <!-- Right arm: reuses the world link created by the left arm. -->
-    <xacro:enlight_robot
+    <xacro:flexiv_robot
       robot_type="Enlight-L"
       robot_sn="$(arg robot_sn)"
@@ -156,31 +130,13 @@
       gripper_name="$(arg gripper_name)"
       load_mounted_ft_sensor="$(arg load_mounted_ft_sensor)"
-      ros2_control="false"
-      use_fake_hardware="$(arg use_fake_hardware)"
-      fake_sensor_commands="$(arg fake_sensor_commands)"
-      initial_positions_file="${arm_init_positions}"
       add_world_link="false"
       create_base_joint="true"
       base_xyz="${right_pose['x']} ${right_pose['y']} ${right_pose['z']}"
       base_rpy="${radians(right_pose['rx'])} ${radians(right_pose['ry'])} ${radians(right_pose['rz'])}">
-    </xacro:enlight_robot>
-    <!-- Single unified ros2_control for both arms (one robot_sn, prefix_left/prefix_right).
-         Prefixes come from compute_arm_prefix so they match the arms' own links even
-         when robot_sn is empty. -->
+    </xacro:flexiv_robot>
     <xacro:compute_arm_prefix arm_prefix="left" robot_sn="$(arg robot_sn)" />
     <xacro:property name="ll_prefix_left" value="${computed_arm_prefix}" lazy_eval="false" />
     <xacro:compute_arm_prefix arm_prefix="right" robot_sn="$(arg robot_sn)" />
     <xacro:property name="ll_prefix_right" value="${computed_arm_prefix}" lazy_eval="false" />
-    <xacro:if value="$(arg ros2_control)">
-      <xacro:flexiv_dual_ros2_control
-        prefix_left="${ll_prefix_left}"
-        prefix_right="${ll_prefix_right}"
-        robot_sn="$(arg robot_sn)"
-        rdk_control_mode="$(arg rdk_control_mode)"
-        use_fake_hardware="$(arg use_fake_hardware)"
-        fake_sensor_commands="$(arg fake_sensor_commands)"
-        initial_positions_file_left="${arm_init_positions}"
-        initial_positions_file_right="${arm_init_positions}" />
-    </xacro:if>
   </xacro:if>
   <!-- ============================== MICO-Core ============================== -->
@@ -193,10 +149,5 @@
       gripper_name="$(arg gripper_name)"
       load_mounted_ft_sensor="$(arg load_mounted_ft_sensor)"
-      ros2_control="$(arg ros2_control)"
-      rdk_control_mode="$(arg rdk_control_mode)"
-      use_fake_hardware="$(arg use_fake_hardware)"
-      fake_sensor_commands="$(arg fake_sensor_commands)"
-      arm_init_positions_file="${arm_cfg}/initial_positions.yaml"
-      torso_init_positions_file="$(find flexiv_description)/config/MICO-Core/torso_initial_positions.yaml" />
+      />
   </xacro:if>
   <!-- ============================== MICO-Plus ============================== -->
@@ -209,10 +160,5 @@
       gripper_name="$(arg gripper_name)"
       load_mounted_ft_sensor="$(arg load_mounted_ft_sensor)"
-      ros2_control="$(arg ros2_control)"
-      rdk_control_mode="$(arg rdk_control_mode)"
-      use_fake_hardware="$(arg use_fake_hardware)"
-      fake_sensor_commands="$(arg fake_sensor_commands)"
-      arm_init_positions_file="${arm_cfg}/initial_positions.yaml"
-      torso_init_positions_file="$(find flexiv_description)/config/MICO-Plus/torso_initial_positions.yaml" />
+      />
   </xacro:if>
   <!-- ============================== MICO-Ultra ============================== -->
@@ -225,10 +171,5 @@
       gripper_name="$(arg gripper_name)"
       load_mounted_ft_sensor="$(arg load_mounted_ft_sensor)"
-      ros2_control="$(arg ros2_control)"
-      rdk_control_mode="$(arg rdk_control_mode)"
-      use_fake_hardware="$(arg use_fake_hardware)"
-      fake_sensor_commands="$(arg fake_sensor_commands)"
-      arm_init_positions_file="${arm_cfg}/initial_positions.yaml"
-      torso_init_positions_file="$(find flexiv_description)/config/MICO-Ultra/torso_initial_positions.yaml" />
+      />
   </xacro:if>
   <!-- ================= AICO1: single arm on a 2-DOF external axis ================= -->
@@ -249,5 +190,5 @@
       <origin xyz="0 0 0" rpy="0 0 0" />
     </joint>
-    <!-- Must match the prefix enlight_robot derives for this arm. -->
+    <!-- Must match the prefix flexiv_robot derives for this arm. -->
     <xacro:compute_arm_prefix arm_prefix="$(arg arm_prefix)" robot_sn="$(arg robot_sn)" />
     <xacro:property name="aico1_arm_prefix" value="${computed_arm_prefix}" lazy_eval="false" />
@@ -262,5 +203,5 @@
         mesh_prefix_path="package://flexiv_description/" />
     </xacro:if>
-    <xacro:enlight_robot
+    <xacro:flexiv_robot
       robot_type="${aico1_arm}"
       robot_sn="$(arg robot_sn)"
@@ -273,21 +214,11 @@
       gripper_name="$(arg gripper_name)"
       load_mounted_ft_sensor="$(arg load_mounted_ft_sensor)"
-      ros2_control="$(arg ros2_control)"
-      rdk_control_mode="$(arg rdk_control_mode)"
-      use_fake_hardware="$(arg use_fake_hardware)"
-      fake_sensor_commands="$(arg fake_sensor_commands)"
-      initial_positions_file="${cfg}/${aico1_arm}/initial_positions.yaml"
-      num_gpio_ports="${18 if aico1_arm.startswith('Rizon') else 20}"
-      external_axis_type="${external_axis_type}"
-      external_axis_prefix="$(arg external_axis_prefix)"
       add_world_link="false"
       create_base_joint="false" />
   </xacro:if>
   <!-- ========== PAIRED ROBOTS: Rizon-Dual and AICO2 (two serial numbers) ==========
-       Distinct from Enlight-LL and MICO above: those are one robot with two arms on
-       a single robot_sn, these are two robots driven together, so they need
-       FlexivDualHardwareInterface via rizon_dual.ros2_control.xacro. -->
+       Two robots driven together, as opposed to Enlight-LL and MICO above which are
+       one robot with two arms on a single robot_sn. -->
   <xacro:if value="${is_paired}">
-    <xacro:include filename="$(find flexiv_description)/urdf/common/rizon_dual.ros2_control.xacro" />
     <!-- AICO2-10-V1 carries two Rizon10; the -4- variants carry a Rizon4 / Rizon4R
          mirrored pair, which is also the default for a plain Rizon-Dual. -->
@@ -310,5 +241,5 @@
       </xacro:unless>
     </xacro:if>
-    <!-- Must match the prefixes enlight_robot derives, including when either serial
+    <!-- Must match the prefixes flexiv_robot derives, including when either serial
          number is empty. lazy_eval is off so each capture resolves before the next
          call. -->
@@ -317,6 +248,4 @@
     <xacro:compute_arm_prefix arm_prefix="right" robot_sn="$(arg robot_sn_right)" />
     <xacro:property name="prefix_right" value="${computed_arm_prefix}" lazy_eval="false" />
-    <xacro:property name="init_left" value="${cfg}/${arm_left}/initial_positions.yaml" />
-    <xacro:property name="init_right" value="${cfg}/${arm_right}/initial_positions.yaml" />
     <link name="world" />
     <!-- AICO2: the external axis carries both arms, so neither creates a base joint. -->
@@ -366,5 +295,5 @@
       <xacro:property name="paired_base_joint" value="true" />
     </xacro:if>
-    <xacro:enlight_robot
+    <xacro:flexiv_robot
       robot_type="${arm_left}"
       robot_sn="$(arg robot_sn_left)"
@@ -377,11 +306,9 @@
       gripper_name="$(arg gripper_name_left)"
       load_mounted_ft_sensor="$(arg load_mounted_ft_sensor_left)"
-      ros2_control="false"
-      initial_positions_file="${init_left}"
       add_world_link="false"
       create_base_joint="${paired_base_joint}"
       base_xyz="${paired_left_xyz}"
       base_rpy="${paired_left_rpy}" />
-    <xacro:enlight_robot
+    <xacro:flexiv_robot
       robot_type="${arm_right}"
       robot_sn="$(arg robot_sn_right)"
@@ -394,6 +321,4 @@
       gripper_name="$(arg gripper_name_right)"
       load_mounted_ft_sensor="$(arg load_mounted_ft_sensor_right)"
-      ros2_control="false"
-      initial_positions_file="${init_right}"
       add_world_link="false"
       create_base_joint="${paired_base_joint}"
@@ -401,18 +326,4 @@
       base_rpy="${paired_right_rpy}" />
     <!-- One interface spanning both robots plus any external axis joints. -->
-    <xacro:if value="$(arg ros2_control)">
-      <xacro:rizon_dual_ros2_control
-        prefix_left="${prefix_left}"
-        prefix_right="${prefix_right}"
-        robot_sn_left="$(arg robot_sn_left)"
-        robot_sn_right="$(arg robot_sn_right)"
-        rdk_control_mode="$(arg rdk_control_mode)"
-        use_fake_hardware="$(arg use_fake_hardware)"
-        fake_sensor_commands="$(arg fake_sensor_commands)"
-        initial_positions_file_left="${init_left}"
-        initial_positions_file_right="${init_right}"
-        external_axis_type="${external_axis_type}"
-        external_axis_prefix="$(arg external_axis_prefix)" />
-    </xacro:if>
   </xacro:if>
 </robot>
