Commit message: Replace gripper_name with gripper_type and add Grav Enhanced gripper types

File: urdf/common/flexiv_robot.xacro (robot description, xacro)
@@ -11,5 +11,5 @@
     arm_prefix:=''
     load_gripper:=false
-    gripper_name:='Flexiv-GN01'
+    gripper_type:='Grav'
     load_mounted_ft_sensor:=false
     add_world_link:=true
@@ -26,7 +26,17 @@
       ${xacro.fatal('load_mounted_ft_sensor is only supported by Rizon4, Rizon4R, Rizon10 and Rizon10R. robot_type \'' + robot_type + '\' does not support a mounted FT sensor.')}
     </xacro:if>
-    <xacro:if value="${load_gripper and gripper_name=='Flexiv-GN01'}">
+    <xacro:property name="gripper_types"
+      value="${xacro.load_yaml('$(find flexiv_description)/config/gripper_types.yaml')['gripper_types']}" />
+    <xacro:if value="${load_gripper and gripper_type not in gripper_types}">
+      ${xacro.fatal('Invalid gripper_type \'' + gripper_type + '\'. Available: ' + ', '.join(gripper_types) + '.')}
+    </xacro:if>
+    <xacro:if value="${load_gripper and gripper_type=='Grav'}">
       <xacro:include filename="$(find flexiv_description)/urdf/common/grav_macro.xacro" />
-      <xacro:flexiv_GN01 prefix="${prefix}" mesh_prefix_path="package://flexiv_description/" />
+      <xacro:GN01 prefix="${prefix}" mesh_prefix_path="package://flexiv_description/" />
+    </xacro:if>
+    <xacro:if value="${load_gripper and gripper_type in ['Grav-Enhanced', 'Grav-Enhanced-A']}">
+      <xacro:include filename="$(find flexiv_description)/urdf/common/grav_enhanced_macro.xacro" />
+      <xacro:EG prefix="${prefix}" mesh_prefix_path="package://flexiv_description/"
+        mode="${'EG-P' if gripper_type == 'Grav-Enhanced' else 'EG-A'}" />
     </xacro:if>
     <xacro:include filename="$(find flexiv_description)/urdf/common/flexiv_arm.xacro" />

File: urdf/common/grav_macro.xacro (robot description, xacro)
@@ -1,5 +1,5 @@
 <?xml version="1.0"?>
 <robot xmlns:xacro="http://wiki.ros.org/xacro">
-  <xacro:macro name="flexiv_GN01" params="prefix mesh_prefix_path">
+  <xacro:macro name="GN01" params="prefix mesh_prefix_path">
     <!-- base link -->
     <link name="${prefix}grav_base_link">

File: urdf/common/mico_core.xacro (robot description, xacro)
@@ -12,5 +12,5 @@
     robot_sn
     load_gripper:=false
-    gripper_name:='Flexiv-GN01'
+    gripper_type:='Grav'
     load_mounted_ft_sensor:=false
     torso_joint_limits_file:='$(find flexiv_description)/config/MICO-Core/joint_limits.yaml'
@@ -92,5 +92,5 @@
       arm_prefix="left"
       load_gripper="${load_gripper}"
-      gripper_name="${gripper_name}"
+      gripper_type="${gripper_type}"
       load_mounted_ft_sensor="${load_mounted_ft_sensor}"
       add_world_link="false"
@@ -108,5 +108,5 @@
       arm_prefix="right"
       load_gripper="${load_gripper}"
-      gripper_name="${gripper_name}"
+      gripper_type="${gripper_type}"
       load_mounted_ft_sensor="${load_mounted_ft_sensor}"
       add_world_link="false"

File: urdf/common/mico_plus.xacro (robot description, xacro)
@@ -13,5 +13,5 @@
     robot_sn
     load_gripper:=false
-    gripper_name:='Flexiv-GN01'
+    gripper_type:='Grav'
     load_mounted_ft_sensor:=false
     torso_joint_limits_file:='$(find flexiv_description)/config/MICO-Plus/joint_limits.yaml'
@@ -122,5 +122,5 @@
       arm_prefix="left"
       load_gripper="${load_gripper}"
-      gripper_name="${gripper_name}"
+      gripper_type="${gripper_type}"
       load_mounted_ft_sensor="${load_mounted_ft_sensor}"
       add_world_link="false"
@@ -138,5 +138,5 @@
       arm_prefix="right"
       load_gripper="${load_gripper}"
-      gripper_name="${gripper_name}"
+      gripper_type="${gripper_type}"
       load_mounted_ft_sensor="${load_mounted_ft_sensor}"
       add_world_link="false"

File: urdf/common/mico_ultra.xacro (robot description, xacro)
@@ -14,5 +14,5 @@
     robot_sn
     load_gripper:=false
-    gripper_name:='Flexiv-GN01'
+    gripper_type:='Grav'
     load_mounted_ft_sensor:=false
     torso_joint_limits_file:='$(find flexiv_description)/config/MICO-Ultra/joint_limits.yaml'
@@ -122,5 +122,5 @@
       arm_prefix="left"
       load_gripper="${load_gripper}"
-      gripper_name="${gripper_name}"
+      gripper_type="${gripper_type}"
       load_mounted_ft_sensor="${load_mounted_ft_sensor}"
       add_world_link="false"
@@ -138,5 +138,5 @@
       arm_prefix="right"
       load_gripper="${load_gripper}"
-      gripper_name="${gripper_name}"
+      gripper_type="${gripper_type}"
       load_mounted_ft_sensor="${load_mounted_ft_sensor}"
       add_world_link="false"

File: urdf/flexiv.urdf.xacro (robot description, xacro)
@@ -35,5 +35,5 @@
     default="$(find flexiv_description)/config/$(arg robot_type)/visual_parameters.yaml" />
   <xacro:arg name="load_gripper" default="false" />
-  <xacro:arg name="gripper_name" default="Flexiv-GN01" />
+  <xacro:arg name="gripper_type" default="Grav" />
   <xacro:arg name="load_mounted_ft_sensor" default="false" />
   <xacro:arg name="mounting_file" default="$(find flexiv_description)/config/single_robot_mounting.yaml" />
@@ -51,6 +51,6 @@
   <xacro:arg name="load_gripper_left" default="false" />
   <xacro:arg name="load_gripper_right" default="false" />
-  <xacro:arg name="gripper_name_left" default="Flexiv-GN01" />
-  <xacro:arg name="gripper_name_right" default="Flexiv-GN01" />
+  <xacro:arg name="gripper_type_left" default="Grav" />
+  <xacro:arg name="gripper_type_right" default="Grav" />
   <xacro:arg name="load_mounted_ft_sensor_left" default="false" />
   <xacro:arg name="load_mounted_ft_sensor_right" default="false" />
@@ -98,5 +98,5 @@
       arm_prefix="$(arg arm_prefix)"
       load_gripper="$(arg load_gripper)"
-      gripper_name="$(arg gripper_name)"
+      gripper_type="$(arg gripper_type)"
       load_mounted_ft_sensor="$(arg load_mounted_ft_sensor)"
       base_rpy="${radians(mounting['orientation']['rx'])} ${radians(mounting['orientation']['ry'])} ${radians(mounting['orientation']['rz'])}">
@@ -125,5 +125,5 @@
       arm_prefix="left"
       load_gripper="$(arg load_gripper)"
-      gripper_name="$(arg gripper_name)"
+      gripper_type="$(arg gripper_type)"
       load_mounted_ft_sensor="$(arg load_mounted_ft_sensor)"
       add_world_link="true"
@@ -143,5 +143,5 @@
       arm_prefix="right"
       load_gripper="$(arg load_gripper)"
-      gripper_name="$(arg gripper_name)"
+      gripper_type="$(arg gripper_type)"
       load_mounted_ft_sensor="$(arg load_mounted_ft_sensor)"
       add_world_link="false"
@@ -166,5 +166,5 @@
       kinematics_parameters_file="${mico_core_kin}"
       load_gripper="$(arg load_gripper)"
-      gripper_name="$(arg gripper_name)"
+      gripper_type="$(arg gripper_type)"
       load_mounted_ft_sensor="$(arg load_mounted_ft_sensor)"
       />
@@ -181,5 +181,5 @@
       kinematics_parameters_file="${mico_plus_kin}"
       load_gripper="$(arg load_gripper)"
-      gripper_name="$(arg gripper_name)"
+      gripper_type="$(arg gripper_type)"
       load_mounted_ft_sensor="$(arg load_mounted_ft_sensor)"
       />
@@ -196,5 +196,5 @@
       kinematics_parameters_file="${mico_ultra_kin}"
       load_gripper="$(arg load_gripper)"
-      gripper_name="$(arg gripper_name)"
+      gripper_type="$(arg gripper_type)"
       load_mounted_ft_sensor="$(arg load_mounted_ft_sensor)"
       />
@@ -242,5 +242,5 @@
       arm_prefix="$(arg arm_prefix)"
       load_gripper="$(arg load_gripper)"
-      gripper_name="$(arg gripper_name)"
+      gripper_type="$(arg gripper_type)"
       load_mounted_ft_sensor="$(arg load_mounted_ft_sensor)"
       add_world_link="false"
@@ -336,5 +336,5 @@
       arm_prefix="left"
       load_gripper="$(arg load_gripper_left)"
-      gripper_name="$(arg gripper_name_left)"
+      gripper_type="$(arg gripper_type_left)"
       load_mounted_ft_sensor="$(arg load_mounted_ft_sensor_left)"
       add_world_link="false"
@@ -351,5 +351,5 @@
       arm_prefix="right"
       load_gripper="$(arg load_gripper_right)"
-      gripper_name="$(arg gripper_name_right)"
+      gripper_type="$(arg gripper_type_right)"
       load_mounted_ft_sensor="$(arg load_mounted_ft_sensor_right)"
       add_world_link="false"
