Commit message: Task/Merge humble-v1 and humble-v2 branches → humble (#30)

File: urdf/common/flexiv_common.xacro (robot description, xacro)
@@ -1,4 +1,16 @@
 <?xml version="1.0"?>
 <robot xmlns:xacro="http://wiki.ros.org/xacro">
+  <!--
+    Compute an arm's joint/link name prefix and expose it to the caller as
+    'computed_arm_prefix'.
+    This is the single source of truth for the prefix.
+    arm_prefix: 'left', 'right' or '' (user-supplied prefixes also allowed)
+    robot_sn:   robot serial number, may be empty
+  -->
+  <xacro:macro name="compute_arm_prefix" params="arm_prefix:='' robot_sn:=''">
+    <xacro:property name="computed_arm_prefix"
+      value="${(arm_prefix + '_' + robot_sn + '_') if arm_prefix != '' and robot_sn != '' else (arm_prefix + robot_sn + '_') if (arm_prefix + robot_sn) != '' else ''}"
+      scope="parent" />
+  </xacro:macro>
   <!--
     Extract visual parameters from the config file
@@ -81,4 +93,12 @@
     <origin xyz="${kinematics['x']} ${kinematics['y']} ${kinematics['z']}"
       rpy="${kinematics['roll']} ${kinematics['pitch']} ${kinematics['yaw']}" />
+  </xacro:macro>
+  <!--
+    Extract the joint rotation axis from the config file.
+    name: name of the joint
+  -->
+  <xacro:macro name="get_joint_axis" params="name">
+    <xacro:property name="joint_kinematics" value="${sec_kinematics[name]}" lazy_eval="false" />
+    <axis xyz="${joint_kinematics['axis'] if 'axis' in joint_kinematics else '0 0 1'}" />
   </xacro:macro>
   <!--

File: urdf/common/mico_core.xacro (robot description, xacro)
@@ -3,10 +3,9 @@
   <!--
     MICO-Core: fixed torso (no actuated torso joints) with two Enlight-L arms.
-    Arm joints: left_${robot_sn}_joint1..7, right_${robot_sn}_joint1..7.
-    ros2_control: reuses flexiv_dual_ros2_control (no torso joints to add).
+    Arm joints: left_<robot_sn>_joint1..7, right_<robot_sn>_joint1..7.
+    An empty robot_sn drops the separating underscore, e.g. 'torso_joint1', 'left_joint1'.
   -->
   <xacro:include filename="$(find flexiv_description)/urdf/common/flexiv_common.xacro" />
-  <xacro:include filename="$(find flexiv_description)/urdf/common/enlight_robot.xacro" />
-  <xacro:include filename="$(find flexiv_description)/urdf/common/flexiv_dual.ros2_control.xacro" />
+  <xacro:include filename="$(find flexiv_description)/urdf/common/flexiv_robot.xacro" />
   <xacro:macro name="mico_core"
     params="
@@ -15,11 +14,4 @@
     gripper_name:='Flexiv-GN01'
     load_mounted_ft_sensor:=false
-    ros2_control:=false
-    rdk_control_mode:='joint_position'
-    use_fake_hardware:=false
-    fake_sensor_commands:=false
-    arm_init_positions_file
-    right_arm_init_positions_file:='$(find flexiv_description)/config/Enlight-L/initial_positions_mirrored.yaml'
-    torso_init_positions_file:=''
     torso_joint_limits_file:='$(find flexiv_description)/config/MICO-Core/joint_limits.yaml'
     torso_kinematics_file:='$(find flexiv_description)/config/MICO-Core/default_kinematics.yaml'
@@ -28,5 +20,15 @@
     ">
     <xacro:property name="arm_cfg" value="$(find flexiv_description)/config/Enlight-L" />
-    <xacro:property name="torso_prefix" value="${robot_sn}_torso_" />
+    <!-- All prefixes follow the same rule as the arms: the separating underscore
+         only appears when the part it separates is non-empty, so an empty robot_sn
+         gives 'torso_base_link' rather than '_torso_base_link'. lazy_eval is off so
+         each capture resolves before the next call. -->
+    <xacro:compute_arm_prefix robot_sn="${robot_sn}" />
+    <xacro:property name="sn_prefix" value="${computed_arm_prefix}" lazy_eval="false" />
+    <xacro:property name="torso_prefix" value="${sn_prefix}torso_" lazy_eval="false" />
+    <xacro:compute_arm_prefix arm_prefix="left" robot_sn="${robot_sn}" />
+    <xacro:property name="prefix_left" value="${computed_arm_prefix}" lazy_eval="false" />
+    <xacro:compute_arm_prefix arm_prefix="right" robot_sn="${robot_sn}" />
+    <xacro:property name="prefix_right" value="${computed_arm_prefix}" lazy_eval="false" />
     <xacro:read_model_data
       joint_limits_parameters_file="${torso_joint_limits_file}"
@@ -77,5 +79,5 @@
     </joint>
     <!-- Left arm (Enlight-L): no world link, no base joint (we attach it below) -->
-    <xacro:enlight_robot
+    <xacro:flexiv_robot
       robot_type="Enlight-L"
       robot_sn="${robot_sn}"
@@ -88,13 +90,9 @@
       gripper_name="${gripper_name}"
       load_mounted_ft_sensor="${load_mounted_ft_sensor}"
-      ros2_control="false"
-      use_fake_hardware="${use_fake_hardware}"
-      fake_sensor_commands="${fake_sensor_commands}"
-      initial_positions_file="${arm_init_positions_file}"
       add_world_link="false"
       create_base_joint="false"
     />
     <!-- Right arm (Enlight-L): no world link, no base joint -->
-    <xacro:enlight_robot
+    <xacro:flexiv_robot
       robot_type="Enlight-L"
       robot_sn="${robot_sn}"
@@ -107,8 +105,4 @@
       gripper_name="${gripper_name}"
       load_mounted_ft_sensor="${load_mounted_ft_sensor}"
-      ros2_control="false"
-      use_fake_hardware="${use_fake_hardware}"
-      fake_sensor_commands="${fake_sensor_commands}"
-      initial_positions_file="${right_arm_init_positions_file}"
       add_world_link="false"
       create_base_joint="false"
@@ -117,24 +111,12 @@
     <joint name="${torso_prefix}left_flange_to_left_arm" type="fixed">
       <parent link="${torso_prefix}left_flange" />
-      <child link="left_${robot_sn}_base_link" />
+      <child link="${prefix_left}base_link" />
       <origin xyz="0 0 0" rpy="0 0 0" />
     </joint>
     <joint name="${torso_prefix}right_flange_to_right_arm" type="fixed">
       <parent link="${torso_prefix}right_flange" />
-      <child link="right_${robot_sn}_base_link" />
+      <child link="${prefix_right}base_link" />
       <origin xyz="0 0 0" rpy="0 0 0" />
     </joint>
-    <!-- ros2_control: MICO-Core has no torso joints, reuse dual ros2_control directly -->
-    <xacro:if value="${ros2_control}">
-      <xacro:flexiv_dual_ros2_control
-        prefix_left="left_${robot_sn}_"
-        prefix_right="right_${robot_sn}_"
-        robot_sn="${robot_sn}"
-        rdk_control_mode="${rdk_control_mode}"
-        use_fake_hardware="${use_fake_hardware}"
-        fake_sensor_commands="${fake_sensor_commands}"
-        initial_positions_file_left="${arm_init_positions_file}"
-        initial_positions_file_right="${right_arm_init_positions_file}" />
-    </xacro:if>
   </xacro:macro>
 </robot>

File: urdf/common/mico_plus.xacro (robot description, xacro)
@@ -3,10 +3,10 @@
   <!--
     MICO-Plus: 2-DOF torso (yaw + pitch) with two Enlight-L arms.
-    Torso joints: ${robot_sn}_torso_joint1 (yaw), ${robot_sn}_torso_joint2 (pitch).
-    Arm joints:   left_${robot_sn}_joint1..7, right_${robot_sn}_joint1..7.
+    Torso joints: <robot_sn>_torso_joint1 (yaw), <robot_sn>_torso_joint2 (pitch).
+    Arm joints:   left_<robot_sn>_joint1..7, right_<robot_sn>_joint1..7.
+    An empty robot_sn drops the separating underscore, e.g. 'torso_joint1', 'left_joint1'.
   -->
   <xacro:include filename="$(find flexiv_description)/urdf/common/flexiv_common.xacro" />
-  <xacro:include filename="$(find flexiv_description)/urdf/common/enlight_robot.xacro" />
-  <xacro:include filename="$(find flexiv_description)/urdf/common/flexiv_mico.ros2_control.xacro" />
+  <xacro:include filename="$(find flexiv_description)/urdf/common/flexiv_robot.xacro" />
   <xacro:macro name="mico_plus"
     params="
@@ -15,11 +15,4 @@
     gripper_name:='Flexiv-GN01'
     load_mounted_ft_sensor:=false
-    ros2_control:=false
-    rdk_control_mode:='joint_position'
-    use_fake_hardware:=false
-    fake_sensor_commands:=false
-    arm_init_positions_file
-    right_arm_init_positions_file:='$(find flexiv_description)/config/Enlight-L/initial_positions_mirrored.yaml'
-    torso_init_positions_file:=''
     torso_joint_limits_file:='$(find flexiv_description)/config/MICO-Plus/joint_limits.yaml'
     torso_kinematics_file:='$(find flexiv_description)/config/MICO-Plus/default_kinematics.yaml'
@@ -28,5 +21,15 @@
     ">
     <xacro:property name="arm_cfg" value="$(find flexiv_description)/config/Enlight-L" />
-    <xacro:property name="torso_prefix" value="${robot_sn}_torso_" />
+    <!-- All prefixes follow the same rule as the arms: the separating underscore
+         only appears when the part it separates is non-empty, so an empty robot_sn
+         gives 'torso_base_link' rather than '_torso_base_link'. lazy_eval is off so
+         each capture resolves before the next call. -->
+    <xacro:compute_arm_prefix robot_sn="${robot_sn}" />
+    <xacro:property name="sn_prefix" value="${computed_arm_prefix}" lazy_eval="false" />
+    <xacro:property name="torso_prefix" value="${sn_prefix}torso_" lazy_eval="false" />
+    <xacro:compute_arm_prefix arm_prefix="left" robot_sn="${robot_sn}" />
+    <xacro:property name="prefix_left" value="${computed_arm_prefix}" lazy_eval="false" />
+    <xacro:compute_arm_prefix arm_prefix="right" robot_sn="${robot_sn}" />
+    <xacro:property name="prefix_right" value="${computed_arm_prefix}" lazy_eval="false" />
     <xacro:read_model_data
       joint_limits_parameters_file="${torso_joint_limits_file}"
@@ -106,5 +109,5 @@
     </joint>
     <!-- Left arm (Enlight-L): no world link, no base joint -->
-    <xacro:enlight_robot
+    <xacro:flexiv_robot
       robot_type="Enlight-L"
       robot_sn="${robot_sn}"
@@ -117,13 +120,9 @@
       gripper_name="${gripper_name}"
       load_mounted_ft_sensor="${load_mounted_ft_sensor}"
-      ros2_control="false"
-      use_fake_hardware="${use_fake_hardware}"
-      fake_sensor_commands="${fake_sensor_commands}"
-      initial_positions_file="${arm_init_positions_file}"
       add_world_link="false"
       create_base_joint="false"
     />
     <!-- Right arm (Enlight-L): no world link, no base joint -->
-    <xacro:enlight_robot
+    <xacro:flexiv_robot
       robot_type="Enlight-L"
       robot_sn="${robot_sn}"
@@ -136,8 +135,4 @@
       gripper_name="${gripper_name}"
       load_mounted_ft_sensor="${load_mounted_ft_sensor}"
-      ros2_control="false"
-      use_fake_hardware="${use_fake_hardware}"
-      fake_sensor_commands="${fake_sensor_commands}"
-      initial_positions_file="${right_arm_init_positions_file}"
       add_world_link="false"
       create_base_joint="false"
@@ -146,25 +141,12 @@
     <joint name="${torso_prefix}left_flange_to_left_arm" type="fixed">
       <parent link="${torso_prefix}left_flange" />
-      <child link="left_${robot_sn}_base_link" />
+      <child link="${prefix_left}base_link" />
       <origin xyz="0 0 0" rpy="0 0 0" />
     </joint>
     <joint name="${torso_prefix}right_flange_to_right_arm" type="fixed">
       <parent link="${torso_prefix}right_flange" />
-      <child link="right_${robot_sn}_base_link" />
+      <child link="${prefix_right}base_link" />
       <origin xyz="0 0 0" rpy="0 0 0" />
     </joint>
-    <!-- ros2_control: MICO-Plus uses flexiv_mico_ros2_control (includes torso joints) -->
-    <xacro:if value="${ros2_control}">
-      <xacro:flexiv_mico_ros2_control
-        prefix_left="left_${robot_sn}_"
-        prefix_right="right_${robot_sn}_"
-        robot_sn="${robot_sn}"
-        rdk_control_mode="${rdk_control_mode}"
-        use_fake_hardware="${use_fake_hardware}"
-        fake_sensor_commands="${fake_sensor_commands}"
-        initial_positions_file_left="${arm_init_positions_file}"
-        initial_positions_file_right="${right_arm_init_positions_file}"
-        torso_initial_positions_file="${torso_init_positions_file}" />
-    </xacro:if>
   </xacro:macro>
 </robot>

File: urdf/common/mico_ultra.xacro (robot description, xacro)
@@ -4,10 +4,10 @@
     MICO-Ultra: 2-DOF torso (waist yaw + pitch) with two Enlight-L arms, mounted on a mobile base.
     base_link is the mobile-base root (empty link, no mesh present).
-    Torso joints: ${robot_sn}_torso_joint1 (waist yaw), ${robot_sn}_torso_joint2 (pitch).
-    Arm joints:   left_${robot_sn}_joint1..7, right_${robot_sn}_joint1..7.
+    Torso joints: <robot_sn>_torso_joint1 (waist yaw), <robot_sn>_torso_joint2 (pitch).
+    Arm joints:   left_<robot_sn>_joint1..7, right_<robot_sn>_joint1..7.
+    An empty robot_sn drops the separating underscore, e.g. 'torso_joint1', 'left_joint1'.
   -->
   <xacro:include filename="$(find flexiv_description)/urdf/common/flexiv_common.xacro" />
-  <xacro:include filename="$(find flexiv_description)/urdf/common/enlight_robot.xacro" />
-  <xacro:include filename="$(find flexiv_description)/urdf/common/flexiv_mico.ros2_control.xacro" />
+  <xacro:include filename="$(find flexiv_description)/urdf/common/flexiv_robot.xacro" />
   <xacro:macro name="mico_ultra"
     params="
@@ -16,11 +16,4 @@
     gripper_name:='Flexiv-GN01'
     load_mounted_ft_sensor:=false
-    ros2_control:=false
-    rdk_control_mode:='joint_position'
-    use_fake_hardware:=false
-    fake_sensor_commands:=false
-    arm_init_positions_file
-    right_arm_init_positions_file:='$(find flexiv_description)/config/Enlight-L/initial_positions_mirrored.yaml'
-    torso_init_positions_file:=''
     torso_joint_limits_file:='$(find flexiv_description)/config/MICO-Ultra/joint_limits.yaml'
     torso_kinematics_file:='$(find flexiv_description)/config/MICO-Ultra/default_kinematics.yaml'
@@ -29,5 +22,15 @@
     ">
     <xacro:property name="arm_cfg" value="$(find flexiv_description)/config/Enlight-L" />
-    <xacro:property name="torso_prefix" value="${robot_sn}_torso_" />
+    <!-- All prefixes follow the same rule as the arms: the separating underscore
+         only appears when the part it separates is non-empty, so an empty robot_sn
+         gives 'torso_base_link' rather than '_torso_base_link'. lazy_eval is off so
+         each capture resolves before the next call. -->
+    <xacro:compute_arm_prefix robot_sn="${robot_sn}" />
+    <xacro:property name="sn_prefix" value="${computed_arm_prefix}" lazy_eval="false" />
+    <xacro:property name="torso_prefix" value="${sn_prefix}torso_" lazy_eval="false" />
+    <xacro:compute_arm_prefix arm_prefix="left" robot_sn="${robot_sn}" />
+    <xacro:property name="prefix_left" value="${computed_arm_prefix}" lazy_eval="false" />
+    <xacro:compute_arm_prefix arm_prefix="right" robot_sn="${robot_sn}" />
+    <xacro:property name="prefix_right" value="${computed_arm_prefix}" lazy_eval="false" />
     <xacro:read_model_data
       joint_limits_parameters_file="${torso_joint_limits_file}"
@@ -106,5 +109,5 @@
     </joint>
     <!-- Left arm (Enlight-L): no world link, no base joint -->
-    <xacro:enlight_robot
+    <xacro:flexiv_robot
       robot_type="Enlight-L"
       robot_sn="${robot_sn}"
@@ -117,13 +120,9 @@
       gripper_name="${gripper_name}"
       load_mounted_ft_sensor="${load_mounted_ft_sensor}"
-      ros2_control="false"
-      use_fake_hardware="${use_fake_hardware}"
-      fake_sensor_commands="${fake_sensor_commands}"
-      initial_positions_file="${arm_init_positions_file}"
       add_world_link="false"
       create_base_joint="false"
     />
     <!-- Right arm (Enlight-L): no world link, no base joint -->
-    <xacro:enlight_robot
+    <xacro:flexiv_robot
       robot_type="Enlight-L"
       robot_sn="${robot_sn}"
@@ -136,8 +135,4 @@
       gripper_name="${gripper_name}"
       load_mounted_ft_sensor="${load_mounted_ft_sensor}"
-      ros2_control="false"
-      use_fake_hardware="${use_fake_hardware}"
-      fake_sensor_commands="${fake_sensor_commands}"
-      initial_positions_file="${right_arm_init_positions_file}"
       add_world_link="false"
       create_base_joint="false"
@@ -146,25 +141,12 @@
     <joint name="${torso_prefix}left_flange_to_left_arm" type="fixed">
       <parent link="${torso_prefix}left_flange" />
-      <child link="left_${robot_sn}_base_link" />
+      <child link="${prefix_left}base_link" />
       <origin xyz="0 0 0" rpy="0 0 0" />
     </joint>
     <joint name="${torso_prefix}right_flange_to_right_arm" type="fixed">
       <parent link="${torso_prefix}right_flange" />
-      <child link="right_${robot_sn}_base_link" />
+      <child link="${prefix_right}base_link" />
       <origin xyz="0 0 0" rpy="0 0 0" />
     </joint>
-    <!-- ros2_control: MICO-Ultra uses flexiv_mico_ros2_control (includes torso joints) -->
-    <xacro:if value="${ros2_control}">
-      <xacro:flexiv_mico_ros2_control
-        prefix_left="left_${robot_sn}_"
-        prefix_right="right_${robot_sn}_"
-        robot_sn="${robot_sn}"
-        rdk_control_mode="${rdk_control_mode}"
-        use_fake_hardware="${use_fake_hardware}"
-        fake_sensor_commands="${fake_sensor_commands}"
-        initial_positions_file_left="${arm_init_positions_file}"
-        initial_positions_file_right="${right_arm_init_positions_file}"
-        torso_initial_positions_file="${torso_init_positions_file}" />
-    </xacro:if>
   </xacro:macro>
 </robot>
