Commit message: Add kinematics configuration for dual-arm robots and update URDF references

File: urdf/common/flexiv_common.xacro (robot description, xacro)
@@ -126,12 +126,17 @@
     sensor_inertia_file: path to the sensor inertia parameters YAML file
     sensor_visual_file: path to the sensor visual parameters YAML file
+    kinematics_section: section of the kinematics YAML holding this chain, empty for the whole map
   -->
   <xacro:macro name="read_model_data"
-    params="joint_limits_parameters_file kinematics_parameters_file inertia_parameters_file visual_parameters_file load_mounted_ft_sensor:=false sensor_kinematics_file:='' sensor_inertia_file:='' sensor_visual_file:=''">
+    params="joint_limits_parameters_file kinematics_parameters_file inertia_parameters_file visual_parameters_file load_mounted_ft_sensor:=false sensor_kinematics_file:='' sensor_inertia_file:='' sensor_visual_file:='' kinematics_section:=''">
     <!-- Read YAML files -->
     <xacro:property name="config_joint_limits_parameters"
       value="${xacro.load_yaml(joint_limits_parameters_file)}" />
-    <xacro:property name="config_kinematics_parameters"
-      value="${xacro.load_yaml(kinematics_parameters_file)}" />
+    <!-- One robot instance is one kinematics file. Products that carry more than one chain
+         name a section per chain; a single arm leaves the section empty and uses the whole map. -->
+    <xacro:property name="config_kinematics_all"
+      value="${xacro.load_yaml(kinematics_parameters_file)['kinematics']}" />
+    <xacro:property name="kinematics_entries"
+      value="${config_kinematics_all if kinematics_section == '' else config_kinematics_all[kinematics_section]}" />
     <xacro:property name="config_inertia_parameters"
       value="${xacro.load_yaml(inertia_parameters_file)}" />
@@ -148,5 +153,5 @@
       <!-- Merge dictionaries -->
       <xacro:property name="sec_kinematics"
-        value="${dict(config_kinematics_parameters['kinematics'], **config_sensor_kinematics['kinematics'])}"
+        value="${dict(kinematics_entries, **config_sensor_kinematics['kinematics'])}"
         scope="parent" />
       <xacro:property name="sec_inertia_parameters"
@@ -158,6 +163,5 @@
     </xacro:if>
     <xacro:unless value="${load_mounted_ft_sensor}">
-      <xacro:property name="sec_kinematics"
-        value="${config_kinematics_parameters['kinematics']}" scope="parent" />
+      <xacro:property name="sec_kinematics" value="${kinematics_entries}" scope="parent" />
       <xacro:property name="sec_inertia_parameters"
         value="${config_inertia_parameters['inertia_parameters']}" scope="parent" />

File: urdf/common/flexiv_robot.xacro (robot description, xacro)
@@ -17,4 +17,5 @@
     base_xyz:='0.0 0.0 0.0'
     base_rpy:='0.0 0.0 0.0'
+    kinematics_section:=''
     ">
     <xacro:include filename="$(find flexiv_description)/urdf/common/flexiv_common.xacro" />
@@ -34,4 +35,5 @@
       joint_limits_parameters_file="${joint_limits_parameters_file}"
       kinematics_parameters_file="${kinematics_parameters_file}"
+      kinematics_section="${kinematics_section}"
       inertia_parameters_file="${inertia_parameters_file}"
       visual_parameters_file="${visual_parameters_file}"

File: urdf/common/mico_core.xacro (robot description, xacro)
@@ -20,4 +20,7 @@
     ">
     <xacro:property name="arm_cfg" value="$(find flexiv_description)/config/Enlight-L" />
+    <!-- Kinematics are per-robot and live in this product's own file, one section per arm.
+         The rest of arm_cfg is model spec shared with a standalone Enlight-L. -->
+    <xacro:property name="arm_kinematics_file" value="${torso_kinematics_file}" />
     <!-- All prefixes follow the same rule as the arms: the separating underscore
          only appears when the part it separates is non-empty, so an empty robot_sn
@@ -34,4 +37,5 @@
       joint_limits_parameters_file="${torso_joint_limits_file}"
       kinematics_parameters_file="${torso_kinematics_file}"
+      kinematics_section="EXT_AXIS"
       inertia_parameters_file="${torso_inertia_file}"
       visual_parameters_file="${torso_visual_file}" />
@@ -83,5 +87,6 @@
       robot_sn="${robot_sn}"
       joint_limits_parameters_file="${arm_cfg}/joint_limits.yaml"
-      kinematics_parameters_file="${arm_cfg}/default_kinematics.yaml"
+      kinematics_parameters_file="${arm_kinematics_file}"
+      kinematics_section="ARM_1"
       inertia_parameters_file="${arm_cfg}/inertia_parameters.yaml"
       visual_parameters_file="${arm_cfg}/visual_parameters.yaml"
@@ -98,5 +103,6 @@
       robot_sn="${robot_sn}"
       joint_limits_parameters_file="${arm_cfg}/joint_limits.yaml"
-      kinematics_parameters_file="${arm_cfg}/default_kinematics.yaml"
+      kinematics_parameters_file="${arm_kinematics_file}"
+      kinematics_section="ARM_2"
       inertia_parameters_file="${arm_cfg}/inertia_parameters.yaml"
       visual_parameters_file="${arm_cfg}/visual_parameters.yaml"

File: urdf/common/mico_plus.xacro (robot description, xacro)
@@ -21,4 +21,7 @@
     ">
     <xacro:property name="arm_cfg" value="$(find flexiv_description)/config/Enlight-L" />
+    <!-- Kinematics are per-robot and live in this product's own file, one section per arm.
+         The rest of arm_cfg is model spec shared with a standalone Enlight-L. -->
+    <xacro:property name="arm_kinematics_file" value="${torso_kinematics_file}" />
     <!-- All prefixes follow the same rule as the arms: the separating underscore
          only appears when the part it separates is non-empty, so an empty robot_sn
@@ -35,4 +38,5 @@
       joint_limits_parameters_file="${torso_joint_limits_file}"
       kinematics_parameters_file="${torso_kinematics_file}"
+      kinematics_section="EXT_AXIS"
       inertia_parameters_file="${torso_inertia_file}"
       visual_parameters_file="${torso_visual_file}" />
@@ -113,5 +117,6 @@
       robot_sn="${robot_sn}"
       joint_limits_parameters_file="${arm_cfg}/joint_limits.yaml"
-      kinematics_parameters_file="${arm_cfg}/default_kinematics.yaml"
+      kinematics_parameters_file="${arm_kinematics_file}"
+      kinematics_section="ARM_1"
       inertia_parameters_file="${arm_cfg}/inertia_parameters.yaml"
       visual_parameters_file="${arm_cfg}/visual_parameters.yaml"
@@ -128,5 +133,6 @@
       robot_sn="${robot_sn}"
       joint_limits_parameters_file="${arm_cfg}/joint_limits.yaml"
-      kinematics_parameters_file="${arm_cfg}/default_kinematics.yaml"
+      kinematics_parameters_file="${arm_kinematics_file}"
+      kinematics_section="ARM_2"
       inertia_parameters_file="${arm_cfg}/inertia_parameters.yaml"
       visual_parameters_file="${arm_cfg}/visual_parameters.yaml"

File: urdf/common/mico_ultra.xacro (robot description, xacro)
@@ -22,4 +22,7 @@
     ">
     <xacro:property name="arm_cfg" value="$(find flexiv_description)/config/Enlight-L" />
+    <!-- Kinematics are per-robot and live in this product's own file, one section per arm.
+         The rest of arm_cfg is model spec shared with a standalone Enlight-L. -->
+    <xacro:property name="arm_kinematics_file" value="${torso_kinematics_file}" />
     <!-- All prefixes follow the same rule as the arms: the separating underscore
          only appears when the part it separates is non-empty, so an empty robot_sn
@@ -36,4 +39,5 @@
       joint_limits_parameters_file="${torso_joint_limits_file}"
       kinematics_parameters_file="${torso_kinematics_file}"
+      kinematics_section="EXT_AXIS"
       inertia_parameters_file="${torso_inertia_file}"
       visual_parameters_file="${torso_visual_file}" />
@@ -113,5 +117,6 @@
       robot_sn="${robot_sn}"
       joint_limits_parameters_file="${arm_cfg}/joint_limits.yaml"
-      kinematics_parameters_file="${arm_cfg}/default_kinematics.yaml"
+      kinematics_parameters_file="${arm_kinematics_file}"
+      kinematics_section="ARM_1"
       inertia_parameters_file="${arm_cfg}/inertia_parameters.yaml"
       visual_parameters_file="${arm_cfg}/visual_parameters.yaml"
@@ -128,5 +133,6 @@
       robot_sn="${robot_sn}"
       joint_limits_parameters_file="${arm_cfg}/joint_limits.yaml"
-      kinematics_parameters_file="${arm_cfg}/default_kinematics.yaml"
+      kinematics_parameters_file="${arm_kinematics_file}"
+      kinematics_section="ARM_2"
       inertia_parameters_file="${arm_cfg}/inertia_parameters.yaml"
       visual_parameters_file="${arm_cfg}/visual_parameters.yaml"

File: urdf/flexiv.urdf.xacro (robot description, xacro)
@@ -107,4 +107,7 @@
     <!-- Each arm of a dual-arm product is an Enlight-L: reuse its config + meshes for both arms. -->
     <xacro:property name="arm_cfg" value="$(find flexiv_description)/config/Enlight-L" />
+    <!-- Kinematics are per-robot and live in this product's own file, one section per arm. -->
+    <xacro:property name="ll_kinematics_file"
+      value="$(find flexiv_description)/config/Enlight-LL/default_kinematics.yaml" />
     <!-- Left arm: owns the shared world link + its base joint. -->
     <xacro:flexiv_robot
@@ -112,5 +115,6 @@
       robot_sn="$(arg robot_sn)"
       joint_limits_parameters_file="${arm_cfg}/joint_limits.yaml"
-      kinematics_parameters_file="${arm_cfg}/default_kinematics.yaml"
+      kinematics_parameters_file="${ll_kinematics_file}"
+      kinematics_section="ARM_1"
       inertia_parameters_file="${arm_cfg}/inertia_parameters.yaml"
       visual_parameters_file="${arm_cfg}/visual_parameters.yaml"
@@ -129,5 +133,6 @@
       robot_sn="$(arg robot_sn)"
       joint_limits_parameters_file="${arm_cfg}/joint_limits.yaml"
-      kinematics_parameters_file="${arm_cfg}/default_kinematics.yaml"
+      kinematics_parameters_file="${ll_kinematics_file}"
+      kinematics_section="ARM_2"
       inertia_parameters_file="${arm_cfg}/inertia_parameters.yaml"
       visual_parameters_file="${arm_cfg}/visual_parameters.yaml"

Commit message: Emit the inertial element from get_inertias so arm links carry mass and inertia

File: urdf/common/flexiv_common.xacro (robot description, xacro)
@@ -108,11 +108,13 @@
   <xacro:macro name="get_inertias" params="name">
     <xacro:property name="inertias" value="${sec_inertia_parameters[name]}" lazy_eval="false" />
-    <origin xyz="${inertias['origin']['x']} ${inertias['origin']['y']} ${inertias['origin']['z']}"
-      rpy="${inertias['origin']['roll']} ${inertias['origin']['pitch']} ${inertias['origin']['yaw']}" />
-    <mass value="${inertias['mass']}" />
-    <inertia ixx="${inertias['inertia']['ixx']}" ixy="${inertias['inertia']['ixy']}"
-      ixz="${inertias['inertia']['ixz']}" iyy="${inertias['inertia']['iyy']}"
-      iyz="${inertias['inertia']['iyz']}"
-      izz="${inertias['inertia']['izz']}" />
+    <inertial>
+      <origin xyz="${inertias['origin']['x']} ${inertias['origin']['y']} ${inertias['origin']['z']}"
+        rpy="${inertias['origin']['roll']} ${inertias['origin']['pitch']} ${inertias['origin']['yaw']}" />
+      <mass value="${inertias['mass']}" />
+      <inertia ixx="${inertias['inertia']['ixx']}" ixy="${inertias['inertia']['ixy']}"
+        ixz="${inertias['inertia']['ixz']}" iyy="${inertias['inertia']['iyy']}"
+        iyz="${inertias['inertia']['iyz']}"
+        izz="${inertias['inertia']['izz']}" />
+    </inertial>
   </xacro:macro>
   <!--

File: urdf/common/mico_core.xacro (robot description, xacro)
@@ -48,7 +48,5 @@
     <!-- Torso: MICO-Core base_link (fixed, no revolute joints) -->
     <link name="${torso_prefix}base_link">
-      <inertial>
-        <xacro:get_inertias name="base_link" />
-      </inertial>
+      <xacro:get_inertias name="base_link" />
       <xacro:get_visuals name="base_link" />
       <xacro:get_collisions name="base_link" />

File: urdf/common/mico_plus.xacro (robot description, xacro)
@@ -49,21 +49,15 @@
     <!-- Torso links -->
     <link name="${torso_prefix}base_link">
-      <inertial>
-        <xacro:get_inertias name="base_link" />
-      </inertial>
+      <xacro:get_inertias name="base_link" />
       <xacro:get_visuals name="base_link" />
       <xacro:get_collisions name="base_link" />
     </link>
     <link name="${torso_prefix}link1">
-      <inertial>
-        <xacro:get_inertias name="link1" />
-      </inertial>
+      <xacro:get_inertias name="link1" />
       <xacro:get_visuals name="link1" />
       <xacro:get_collisions name="link1" />
     </link>
     <link name="${torso_prefix}link2">
-      <inertial>
-        <xacro:get_inertias name="link2" />
-      </inertial>
+      <xacro:get_inertias name="link2" />
       <xacro:get_visuals name="link2" />
       <xacro:get_collisions name="link2" />

File: urdf/common/mico_ultra.xacro (robot description, xacro)
@@ -50,20 +50,14 @@
     <!-- Mobile base root: empty link -->
     <link name="${torso_prefix}base_link">
-      <inertial>
-        <xacro:get_inertias name="base_link" />
-      </inertial>
+      <xacro:get_inertias name="base_link" />
     </link>
     <!-- Torso links -->
     <link name="${torso_prefix}link1">
-      <inertial>
-        <xacro:get_inertias name="link1" />
-      </inertial>
+      <xacro:get_inertias name="link1" />
       <xacro:get_visuals name="link1" />
       <xacro:get_collisions name="link1" />
     </link>
     <link name="${torso_prefix}link2">
-      <inertial>
-        <xacro:get_inertias name="link2" />
-      </inertial>
+      <xacro:get_inertias name="link2" />
       <xacro:get_visuals name="link2" />
       <xacro:get_collisions name="link2" />
