Commit message: Fix hardcoded kinematics param file path

File: urdf/common/mico_core.xacro (robot description, xacro)
@@ -15,12 +15,11 @@
     load_mounted_ft_sensor:=false
     torso_joint_limits_file:='$(find flexiv_description)/config/MICO-Core/joint_limits.yaml'
-    torso_kinematics_file:='$(find flexiv_description)/config/MICO-Core/default_kinematics.yaml'
+    kinematics_parameters_file:='$(find flexiv_description)/config/MICO-Core/default_kinematics.yaml'
     torso_inertia_file:='$(find flexiv_description)/config/MICO-Core/inertia_parameters.yaml'
     torso_visual_file:='$(find flexiv_description)/config/MICO-Core/visual_parameters.yaml'
     ">
     <xacro:property name="arm_cfg" value="$(find flexiv_description)/config/Enlight-L" />
-    <!-- Kinematics are per-robot and live in this product's own file, one section per arm.
-         The rest of arm_cfg is model spec shared with a standalone Enlight-L. -->
-    <xacro:property name="arm_kinematics_file" value="${torso_kinematics_file}" />
+    <!-- Kinematics are per-robot and live in this product's own file, one section per
+         chain. The rest of arm_cfg is model spec shared with a standalone Enlight-L. -->
     <!-- All prefixes follow the same rule as the arms: the separating underscore
          only appears when the part it separates is non-empty, so an empty robot_sn
@@ -36,5 +35,5 @@
     <xacro:read_model_data
       joint_limits_parameters_file="${torso_joint_limits_file}"
-      kinematics_parameters_file="${torso_kinematics_file}"
+      kinematics_parameters_file="${kinematics_parameters_file}"
       kinematics_section="EXT_AXIS"
       inertia_parameters_file="${torso_inertia_file}"
@@ -87,5 +86,5 @@
       robot_sn="${robot_sn}"
       joint_limits_parameters_file="${arm_cfg}/joint_limits.yaml"
-      kinematics_parameters_file="${arm_kinematics_file}"
+      kinematics_parameters_file="${kinematics_parameters_file}"
       kinematics_section="ARM_1"
       inertia_parameters_file="${arm_cfg}/inertia_parameters.yaml"
@@ -103,5 +102,5 @@
       robot_sn="${robot_sn}"
       joint_limits_parameters_file="${arm_cfg}/joint_limits.yaml"
-      kinematics_parameters_file="${arm_kinematics_file}"
+      kinematics_parameters_file="${kinematics_parameters_file}"
       kinematics_section="ARM_2"
       inertia_parameters_file="${arm_cfg}/inertia_parameters.yaml"

File: urdf/common/mico_plus.xacro (robot description, xacro)
@@ -16,12 +16,11 @@
     load_mounted_ft_sensor:=false
     torso_joint_limits_file:='$(find flexiv_description)/config/MICO-Plus/joint_limits.yaml'
-    torso_kinematics_file:='$(find flexiv_description)/config/MICO-Plus/default_kinematics.yaml'
+    kinematics_parameters_file:='$(find flexiv_description)/config/MICO-Plus/default_kinematics.yaml'
     torso_inertia_file:='$(find flexiv_description)/config/MICO-Plus/inertia_parameters.yaml'
     torso_visual_file:='$(find flexiv_description)/config/MICO-Plus/visual_parameters.yaml'
     ">
     <xacro:property name="arm_cfg" value="$(find flexiv_description)/config/Enlight-L" />
-    <!-- Kinematics are per-robot and live in this product's own file, one section per arm.
-         The rest of arm_cfg is model spec shared with a standalone Enlight-L. -->
-    <xacro:property name="arm_kinematics_file" value="${torso_kinematics_file}" />
+    <!-- Kinematics are per-robot and live in this product's own file, one section per
+         chain. The rest of arm_cfg is model spec shared with a standalone Enlight-L. -->
     <!-- All prefixes follow the same rule as the arms: the separating underscore
          only appears when the part it separates is non-empty, so an empty robot_sn
@@ -37,5 +36,5 @@
     <xacro:read_model_data
       joint_limits_parameters_file="${torso_joint_limits_file}"
-      kinematics_parameters_file="${torso_kinematics_file}"
+      kinematics_parameters_file="${kinematics_parameters_file}"
       kinematics_section="EXT_AXIS"
       inertia_parameters_file="${torso_inertia_file}"
@@ -117,5 +116,5 @@
       robot_sn="${robot_sn}"
       joint_limits_parameters_file="${arm_cfg}/joint_limits.yaml"
-      kinematics_parameters_file="${arm_kinematics_file}"
+      kinematics_parameters_file="${kinematics_parameters_file}"
       kinematics_section="ARM_1"
       inertia_parameters_file="${arm_cfg}/inertia_parameters.yaml"
@@ -133,5 +132,5 @@
       robot_sn="${robot_sn}"
       joint_limits_parameters_file="${arm_cfg}/joint_limits.yaml"
-      kinematics_parameters_file="${arm_kinematics_file}"
+      kinematics_parameters_file="${kinematics_parameters_file}"
       kinematics_section="ARM_2"
       inertia_parameters_file="${arm_cfg}/inertia_parameters.yaml"

File: urdf/common/mico_ultra.xacro (robot description, xacro)
@@ -17,12 +17,11 @@
     load_mounted_ft_sensor:=false
     torso_joint_limits_file:='$(find flexiv_description)/config/MICO-Ultra/joint_limits.yaml'
-    torso_kinematics_file:='$(find flexiv_description)/config/MICO-Ultra/default_kinematics.yaml'
+    kinematics_parameters_file:='$(find flexiv_description)/config/MICO-Ultra/default_kinematics.yaml'
     torso_inertia_file:='$(find flexiv_description)/config/MICO-Ultra/inertia_parameters.yaml'
     torso_visual_file:='$(find flexiv_description)/config/MICO-Ultra/visual_parameters.yaml'
     ">
     <xacro:property name="arm_cfg" value="$(find flexiv_description)/config/Enlight-L" />
-    <!-- Kinematics are per-robot and live in this product's own file, one section per arm.
-         The rest of arm_cfg is model spec shared with a standalone Enlight-L. -->
-    <xacro:property name="arm_kinematics_file" value="${torso_kinematics_file}" />
+    <!-- Kinematics are per-robot and live in this product's own file, one section per
+         chain. The rest of arm_cfg is model spec shared with a standalone Enlight-L. -->
     <!-- All prefixes follow the same rule as the arms: the separating underscore
          only appears when the part it separates is non-empty, so an empty robot_sn
@@ -38,5 +37,5 @@
     <xacro:read_model_data
       joint_limits_parameters_file="${torso_joint_limits_file}"
-      kinematics_parameters_file="${torso_kinematics_file}"
+      kinematics_parameters_file="${kinematics_parameters_file}"
       kinematics_section="EXT_AXIS"
       inertia_parameters_file="${torso_inertia_file}"
@@ -117,5 +116,5 @@
       robot_sn="${robot_sn}"
       joint_limits_parameters_file="${arm_cfg}/joint_limits.yaml"
-      kinematics_parameters_file="${arm_kinematics_file}"
+      kinematics_parameters_file="${kinematics_parameters_file}"
       kinematics_section="ARM_1"
       inertia_parameters_file="${arm_cfg}/inertia_parameters.yaml"
@@ -133,5 +132,5 @@
       robot_sn="${robot_sn}"
       joint_limits_parameters_file="${arm_cfg}/joint_limits.yaml"
-      kinematics_parameters_file="${arm_kinematics_file}"
+      kinematics_parameters_file="${kinematics_parameters_file}"
       kinematics_section="ARM_2"
       inertia_parameters_file="${arm_cfg}/inertia_parameters.yaml"

File: urdf/flexiv.urdf.xacro (robot description, xacro)
@@ -109,5 +109,6 @@
     <!-- Kinematics are per-robot and live in this product's own file, one section per arm. -->
     <xacro:property name="ll_kinematics_file"
-      value="$(find flexiv_description)/config/Enlight-LL/default_kinematics.yaml" />
+      value="${'$(arg kinematics_parameters_file)' if '$(arg kinematics_parameters_file)' != ''
+               else cfg + '/Enlight-LL/default_kinematics.yaml'}" />
     <!-- Left arm: owns the shared world link + its base joint. -->
     <xacro:flexiv_robot
@@ -155,6 +156,10 @@
     <xacro:include filename="$(find flexiv_description)/urdf/common/mico_core.xacro" />
     <xacro:property name="arm_cfg" value="$(find flexiv_description)/config/Enlight-L" />
+    <xacro:property name="mico_core_kin"
+      value="${'$(arg kinematics_parameters_file)' if '$(arg kinematics_parameters_file)' != ''
+               else cfg + '/MICO-Core/default_kinematics.yaml'}" />
     <xacro:mico_core
       robot_sn="$(arg robot_sn)"
+      kinematics_parameters_file="${mico_core_kin}"
       load_gripper="$(arg load_gripper)"
       gripper_name="$(arg gripper_name)"
@@ -166,6 +171,10 @@
     <xacro:include filename="$(find flexiv_description)/urdf/common/mico_plus.xacro" />
     <xacro:property name="arm_cfg" value="$(find flexiv_description)/config/Enlight-L" />
+    <xacro:property name="mico_plus_kin"
+      value="${'$(arg kinematics_parameters_file)' if '$(arg kinematics_parameters_file)' != ''
+               else cfg + '/MICO-Plus/default_kinematics.yaml'}" />
     <xacro:mico_plus
       robot_sn="$(arg robot_sn)"
+      kinematics_parameters_file="${mico_plus_kin}"
       load_gripper="$(arg load_gripper)"
       gripper_name="$(arg gripper_name)"
@@ -177,6 +186,10 @@
     <xacro:include filename="$(find flexiv_description)/urdf/common/mico_ultra.xacro" />
     <xacro:property name="arm_cfg" value="$(find flexiv_description)/config/Enlight-L" />
+    <xacro:property name="mico_ultra_kin"
+      value="${'$(arg kinematics_parameters_file)' if '$(arg kinematics_parameters_file)' != ''
+               else cfg + '/MICO-Ultra/default_kinematics.yaml'}" />
     <xacro:mico_ultra
       robot_sn="$(arg robot_sn)"
+      kinematics_parameters_file="${mico_ultra_kin}"
       load_gripper="$(arg load_gripper)"
       gripper_name="$(arg gripper_name)"

Commit message: Update MICO-Core/Plus/Ultra meshes, kinematics, inertia and torso limits

File: urdf/common/mico_core.xacro (robot description, xacro)
@@ -52,4 +52,14 @@
       <xacro:get_collisions name="base_link" />
     </link>
+    <link name="${torso_prefix}neck_link">
+      <xacro:get_inertias name="neck_link" />
+      <xacro:get_visuals name="neck_link" />
+      <xacro:get_collisions name="neck_link" />
+    </link>
+    <link name="${torso_prefix}head_link">
+      <xacro:get_inertias name="head_link" />
+      <xacro:get_visuals name="head_link" />
+      <xacro:get_collisions name="head_link" />
+    </link>
     <!-- Torso flange links (massless) -->
     <link name="${torso_prefix}left_flange">
@@ -78,4 +88,15 @@
       <parent link="${torso_prefix}base_link" />
       <child link="${torso_prefix}right_flange" />
+    </joint>
+    <!-- Fixed neck and head -->
+    <joint name="${torso_prefix}neck_joint" type="fixed">
+      <xacro:get_kinematics name="neck_joint" />
+      <parent link="${torso_prefix}base_link" />
+      <child link="${torso_prefix}neck_link" />
+    </joint>
+    <joint name="${torso_prefix}head_joint" type="fixed">
+      <xacro:get_kinematics name="head_joint" />
+      <parent link="${torso_prefix}neck_link" />
+      <child link="${torso_prefix}head_link" />
     </joint>
     <!-- Left arm (Enlight-L): no world link, no base joint (we attach it below) -->

File: urdf/common/mico_plus.xacro (robot description, xacro)
@@ -63,4 +63,14 @@
       <xacro:get_collisions name="link2" />
     </link>
+    <link name="${torso_prefix}neck_link">
+      <xacro:get_inertias name="neck_link" />
+      <xacro:get_visuals name="neck_link" />
+      <xacro:get_collisions name="neck_link" />
+    </link>
+    <link name="${torso_prefix}head_link">
+      <xacro:get_inertias name="head_link" />
+      <xacro:get_visuals name="head_link" />
+      <xacro:get_collisions name="head_link" />
+    </link>
     <!-- Torso flange links (massless) -->
     <link name="${torso_prefix}left_flange">
@@ -104,4 +114,15 @@
       <parent link="${torso_prefix}link2" />
       <child link="${torso_prefix}right_flange" />
+    </joint>
+    <!-- Fixed neck and head -->
+    <joint name="${torso_prefix}neck_joint" type="fixed">
+      <xacro:get_kinematics name="neck_joint" />
+      <parent link="${torso_prefix}link2" />
+      <child link="${torso_prefix}neck_link" />
+    </joint>
+    <joint name="${torso_prefix}head_joint" type="fixed">
+      <xacro:get_kinematics name="head_joint" />
+      <parent link="${torso_prefix}neck_link" />
+      <child link="${torso_prefix}head_link" />
     </joint>
     <!-- Left arm (Enlight-L): no world link, no base joint -->

File: urdf/common/mico_ultra.xacro (robot description, xacro)
@@ -3,5 +3,4 @@
   <!--
     MICO-Ultra: 2-DOF torso (waist yaw + pitch) with two Enlight-L arms, mounted on a mobile base.
-    base_link is the mobile-base root (empty link, no mesh present).
     Torso joints: <robot_sn>_torso_joint1 (waist yaw), <robot_sn>_torso_joint2 (pitch).
     Arm joints:   left_<robot_sn>_joint1..7, right_<robot_sn>_joint1..7.
@@ -41,5 +40,5 @@
       inertia_parameters_file="${torso_inertia_file}"
       visual_parameters_file="${torso_visual_file}" />
-    <!-- World link and fixed joint to torso base (mobile base root: empty link, no mesh) -->
+    <!-- World link and fixed joint to torso base -->
     <link name="world" />
     <joint name="${torso_prefix}world_joint" type="fixed">
@@ -48,7 +47,9 @@
       <origin xyz="0 0 0" rpy="0 0 0" />
     </joint>
-    <!-- Mobile base root: empty link -->
+    <!-- Mobile base -->
     <link name="${torso_prefix}base_link">
       <xacro:get_inertias name="base_link" />
+      <xacro:get_visuals name="base_link" />
+      <xacro:get_collisions name="base_link" />
     </link>
     <!-- Torso links -->
@@ -62,4 +63,14 @@
       <xacro:get_visuals name="link2" />
       <xacro:get_collisions name="link2" />
+    </link>
+    <link name="${torso_prefix}neck_link">
+      <xacro:get_inertias name="neck_link" />
+      <xacro:get_visuals name="neck_link" />
+      <xacro:get_collisions name="neck_link" />
+    </link>
+    <link name="${torso_prefix}head_link">
+      <xacro:get_inertias name="head_link" />
+      <xacro:get_visuals name="head_link" />
+      <xacro:get_collisions name="head_link" />
     </link>
     <!-- Torso flange links (massless) -->
@@ -104,4 +115,15 @@
       <parent link="${torso_prefix}link2" />
       <child link="${torso_prefix}right_flange" />
+    </joint>
+    <!-- Fixed neck and head -->
+    <joint name="${torso_prefix}neck_joint" type="fixed">
+      <xacro:get_kinematics name="neck_joint" />
+      <parent link="${torso_prefix}link2" />
+      <child link="${torso_prefix}neck_link" />
+    </joint>
+    <joint name="${torso_prefix}head_joint" type="fixed">
+      <xacro:get_kinematics name="head_joint" />
+      <parent link="${torso_prefix}neck_link" />
+      <child link="${torso_prefix}head_link" />
     </joint>
     <!-- Left arm (Enlight-L): no world link, no base joint -->
