Commit message: Add single robot mounting configuration and integrate into Rizon URDF

File: urdf/rizon.urdf.xacro (robot description, xacro)
@@ -25,4 +25,6 @@
   <xacro:arg name="fake_sensor_commands" default="false" />
   <xacro:arg name="initial_positions_file" default="$(find flexiv_description)/config/initial_positions.yaml" />
+  <xacro:arg name="mounting_file" default="$(find flexiv_description)/config/single_robot_mounting.yaml" />
+  <xacro:property name="mounting" value="${xacro.load_yaml('$(arg mounting_file)')}" />
   <xacro:rizon_robot
     rizon_type="$(arg rizon_type)"
@@ -40,5 +42,6 @@
     use_fake_hardware="$(arg use_fake_hardware)"
     fake_sensor_commands="$(arg fake_sensor_commands)"
-    initial_positions_file="$(arg initial_positions_file)">
+    initial_positions_file="$(arg initial_positions_file)"
+    base_rpy="${radians(mounting['mounting']['rx'])} ${radians(mounting['mounting']['ry'])} ${radians(mounting['mounting']['rz'])}">
   </xacro:rizon_robot>
 </robot>

Commit message: Feature/Add robot mounting config yaml (#7)

File: urdf/rizon.urdf.xacro (robot description, xacro)
@@ -25,4 +25,6 @@
   <xacro:arg name="fake_sensor_commands" default="false" />
   <xacro:arg name="initial_positions_file" default="$(find flexiv_description)/config/initial_positions.yaml" />
+  <xacro:arg name="mounting_file" default="$(find flexiv_description)/config/single_robot_mounting.yaml" />
+  <xacro:property name="mounting" value="${xacro.load_yaml('$(arg mounting_file)')}" />
   <xacro:rizon_robot
     rizon_type="$(arg rizon_type)"
@@ -40,5 +42,6 @@
     use_fake_hardware="$(arg use_fake_hardware)"
     fake_sensor_commands="$(arg fake_sensor_commands)"
-    initial_positions_file="$(arg initial_positions_file)">
+    initial_positions_file="$(arg initial_positions_file)"
+    base_rpy="${radians(mounting['orientation']['rx'])} ${radians(mounting['orientation']['ry'])} ${radians(mounting['orientation']['rz'])}">
   </xacro:rizon_robot>
 </robot>

File: urdf/rizon_dual.urdf.xacro (robot description, xacro)
@@ -18,5 +18,5 @@
   <xacro:arg name="initial_positions_file_left" default="$(find flexiv_description)/config/left_initial_positions.yaml" />
   <xacro:arg name="initial_positions_file_right" default="$(find flexiv_description)/config/right_initial_positions.yaml" />
-  <xacro:arg name="translations_file" default="$(find flexiv_description)/config/dual_arm_translations.yaml" />
+  <xacro:arg name="mounting_file" default="$(find flexiv_description)/config/dual_arm_mounting.yaml" />
   <xacro:include filename="$(find flexiv_description)/urdf/common/rizon_robot.xacro" />
   <xacro:include filename="$(find flexiv_description)/urdf/common/rizon_dual.ros2_control.xacro" />
@@ -24,5 +24,5 @@
   <xacro:property name="prefix_left" value="left_$(arg robot_sn_left)_" />
   <xacro:property name="prefix_right" value="right_$(arg robot_sn_right)_" />
-  <xacro:property name="translations" value="${xacro.load_yaml('$(arg translations_file)')}" />
+  <xacro:property name="mounting" value="${xacro.load_yaml('$(arg mounting_file)')}" />
   <link name="world" />
   <!-- Left Robot -->
@@ -40,6 +40,6 @@
     ros2_control="false"
     add_world_link="false"
-    base_xyz="${translations['translations']['left']['x']} ${translations['translations']['left']['y']} ${translations['translations']['left']['z']}"
-    base_rpy="0 0 0"
+    base_xyz="${mounting['positions']['left']['x']} ${mounting['positions']['left']['y']} ${mounting['positions']['left']['z']}"
+    base_rpy="${radians(mounting['positions']['left']['rx'])} ${radians(mounting['positions']['left']['ry'])} ${radians(mounting['positions']['left']['rz'])}"
   />
   <!-- Right Robot -->
@@ -57,6 +57,6 @@
     ros2_control="false"
     add_world_link="false"
-    base_xyz="${translations['translations']['right']['x']} ${translations['translations']['right']['y']} ${translations['translations']['right']['z']}"
-    base_rpy="0 0 0"
+    base_xyz="${mounting['positions']['right']['x']} ${mounting['positions']['right']['y']} ${mounting['positions']['right']['z']}"
+    base_rpy="${radians(mounting['positions']['right']['rx'])} ${radians(mounting['positions']['right']['ry'])} ${radians(mounting['positions']['right']['rz'])}"
   />
   <!-- Dual ROS 2 Control -->
@@ -72,10 +72,10 @@
       initial_positions_file_left="$(arg initial_positions_file_left)"
       initial_positions_file_right="$(arg initial_positions_file_right)"
-      translation_left_x="${translations['translations']['left']['x']}"
-      translation_left_y="${translations['translations']['left']['y']}"
-      translation_left_z="${translations['translations']['left']['z']}"
-      translation_right_x="${translations['translations']['right']['x']}"
-      translation_right_y="${translations['translations']['right']['y']}"
-      translation_right_z="${translations['translations']['right']['z']}"
+      translation_left_x="${mounting['positions']['left']['x']}"
+      translation_left_y="${mounting['positions']['left']['y']}"
+      translation_left_z="${mounting['positions']['left']['z']}"
+      translation_right_x="${mounting['positions']['right']['x']}"
+      translation_right_y="${mounting['positions']['right']['y']}"
+      translation_right_z="${mounting['positions']['right']['z']}"
     />
   </xacro:if>
