Commit message: Add AICO2-4-V2 mesh and update URDF

File: urdf/aico2.urdf.xacro (robot description, xacro)
@@ -36,4 +36,5 @@
     default="$(find flexiv_description)/config/right_initial_positions.yaml" />
   <xacro:include filename="$(find flexiv_description)/urdf/common/aico2_4_v1.xacro" />
+  <xacro:include filename="$(find flexiv_description)/urdf/common/aico2_4_v2.xacro" />
   <xacro:include filename="$(find flexiv_description)/urdf/common/aico2_10_v1.xacro" />
   <xacro:include filename="$(find flexiv_description)/urdf/common/rizon_robot.xacro" />
@@ -57,4 +58,15 @@
       <parent link="world" />
       <child link="$(arg external_axis_prefix)aico2_4_v1_base_link" />
+      <origin xyz="0 0 0" rpy="0 0 0" />
+    </joint>
+  </xacro:if>
+  <xacro:if value="${'$(arg external_axis_type)' == 'aico2_4_v2'}">
+    <xacro:aico2_4_v2 prefix="$(arg external_axis_prefix)"
+      left_arm_prefix="${calculated_left_arm_prefix}"
+      right_arm_prefix="${calculated_right_arm_prefix}"
+      mesh_prefix_path="package://flexiv_description/" />
+    <joint name="world_to_platform" type="fixed">
+      <parent link="world" />
+      <child link="$(arg external_axis_prefix)aico2_4_v2_base_link" />
       <origin xyz="0 0 0" rpy="0 0 0" />
     </joint>

File: urdf/common/aico2_10_v1.xacro (robot description, xacro)
@@ -8,5 +8,5 @@
       <child link="${prefix}aico2_10_v1_link1" />
       <axis xyz="0 0 1" />
-      <limit lower="-1.57" upper="1.57" effort="1000" velocity="1" />
+      <limit lower="-1.57" upper="1.57" effort="1000" velocity="1.047" />
     </joint>
     <joint name="${prefix}aico2_10_v1_joint2" type="revolute">
@@ -15,5 +15,5 @@
       <child link="${prefix}aico2_10_v1_link2" />
       <axis xyz="0 1 0" />
-      <limit lower="0" upper="1.57" effort="1900" velocity="1" />
+      <limit lower="0" upper="1.57" effort="1900" velocity="1.047" />
     </joint>
     <joint name="${prefix}aico2_10_v1_left_arm_adapter" type="fixed">

File: urdf/common/aico2_4_v1.xacro (robot description, xacro)
@@ -15,5 +15,5 @@
       <child link="${prefix}aico2_4_v1_link2" />
       <axis xyz="0 1 0" />
-      <limit lower="0" upper="1.57" effort="365" velocity="1" />
+      <limit lower="0" upper="1.57" effort="1000" velocity="1.05" />
     </joint>
     <joint name="${prefix}aico2_4_v1_left_arm_adapter" type="fixed">

File: urdf/common/rizon_dual.ros2_control.xacro (robot description, xacro)
@@ -88,4 +88,26 @@
         </joint>
       </xacro:if>
+      <xacro:if value="${external_axis_type == 'aico2_4_v2'}">
+        <joint name="${external_axis_prefix}aico2_4_v2_joint1">
+          <command_interface name="position" />
+          <command_interface name="velocity" />
+          <command_interface name="effort" />
+          <state_interface name="position">
+            <param name="initial_value">0.0</param>
+          </state_interface>
+          <state_interface name="velocity" />
+          <state_interface name="effort" />
+        </joint>
+        <joint name="${external_axis_prefix}aico2_4_v2_joint2">
+          <command_interface name="position" />
+          <command_interface name="velocity" />
+          <command_interface name="effort" />
+          <state_interface name="position">
+            <param name="initial_value">0.0</param>
+          </state_interface>
+          <state_interface name="velocity" />
+          <state_interface name="effort" />
+        </joint>
+      </xacro:if>
       <xacro:if value="${external_axis_type == 'aico2_10_v1'}">
         <joint name="${external_axis_prefix}aico2_10_v1_joint1">

Commit message: Task/Update AICO series model names (#14)

File: urdf/aico2.urdf.xacro (robot description, xacro)
@@ -1,5 +1,5 @@
 <?xml version="1.0" encoding="utf-8"?>
 <robot xmlns:xacro="http://www.ros.org/wiki/xacro" name="aico2">
-  <xacro:arg name="external_axis_type" default="aico2_platform_x1" />
+  <xacro:arg name="external_axis_type" default="aico2_4_v1" />
   <xacro:arg name="external_axis_prefix" default="" />
   <xacro:arg name="rizon_type" default="Rizon4" />
@@ -10,6 +10,6 @@
     <xacro:property name="rizon_type_left" value="Rizon4" />
     <xacro:property name="rizon_type_right" value="Rizon4R" />
-    <xacro:if value="${'$(arg external_axis_type)' != 'aico2_platform_x1'}">
-      ${xacro.warning('AICO2 with Rizon4 configuration only supports aico2_platform_x1 external axis. You selected $(arg external_axis_type).')}
+    <xacro:if value="${'$(arg external_axis_type)' != 'aico2_4_v1' and '$(arg external_axis_type)' != 'aico2_4_v2'}">
+      ${xacro.warning('AICO2 with Rizon4 configuration only supports AICO2-4-V1 or AICO2-4-V2 external axis. You selected $(arg external_axis_type).')}
     </xacro:if>
   </xacro:if>
@@ -17,6 +17,6 @@
     <xacro:property name="rizon_type_left" value="Rizon10" />
     <xacro:property name="rizon_type_right" value="Rizon10" />
-    <xacro:if value="${'$(arg external_axis_type)' != 'aico2_platform_x2'}">
-      ${xacro.warning('AICO2 with Rizon10 configuration only supports aico2_platform_x2 external axis. You selected $(arg external_axis_type).')}
+    <xacro:if value="${'$(arg external_axis_type)' != 'aico2_10_v1'}">
+      ${xacro.warning('AICO2 with Rizon10 configuration only supports AICO2-10-V1 external axis. You selected $(arg external_axis_type).')}
     </xacro:if>
   </xacro:if>
@@ -35,6 +35,7 @@
   <xacro:arg name="initial_positions_file_right"
     default="$(find flexiv_description)/config/right_initial_positions.yaml" />
-  <xacro:include filename="$(find flexiv_description)/urdf/common/aico2_platform_x1.xacro" />
-  <xacro:include filename="$(find flexiv_description)/urdf/common/aico2_platform_x2.xacro" />
+  <xacro:include filename="$(find flexiv_description)/urdf/common/aico2_4_v1.xacro" />
+  <xacro:include filename="$(find flexiv_description)/urdf/common/aico2_4_v2.xacro" />
+  <xacro:include filename="$(find flexiv_description)/urdf/common/aico2_10_v1.xacro" />
   <xacro:include filename="$(find flexiv_description)/urdf/common/rizon_robot.xacro" />
   <xacro:include filename="$(find flexiv_description)/urdf/common/rizon_dual.ros2_control.xacro" />
@@ -49,6 +50,6 @@
   <!-- Instantiate External Axis -->
   <link name="world" />
-  <xacro:if value="${'$(arg external_axis_type)' == 'aico2_platform_x1'}">
-    <xacro:aico2_platform_x1 prefix="$(arg external_axis_prefix)"
+  <xacro:if value="${'$(arg external_axis_type)' == 'aico2_4_v1'}">
+    <xacro:aico2_4_v1 prefix="$(arg external_axis_prefix)"
       left_arm_prefix="${calculated_left_arm_prefix}"
       right_arm_prefix="${calculated_right_arm_prefix}"
@@ -56,10 +57,10 @@
     <joint name="world_to_platform" type="fixed">
       <parent link="world" />
-      <child link="$(arg external_axis_prefix)aico2_x1_base_link" />
+      <child link="$(arg external_axis_prefix)aico2_4_v1_base_link" />
       <origin xyz="0 0 0" rpy="0 0 0" />
     </joint>
   </xacro:if>
-  <xacro:if value="${'$(arg external_axis_type)' == 'aico2_platform_x2'}">
-    <xacro:aico2_platform_x2 prefix="$(arg external_axis_prefix)"
+  <xacro:if value="${'$(arg external_axis_type)' == 'aico2_4_v2'}">
+    <xacro:aico2_4_v2 prefix="$(arg external_axis_prefix)"
       left_arm_prefix="${calculated_left_arm_prefix}"
       right_arm_prefix="${calculated_right_arm_prefix}"
@@ -67,5 +68,16 @@
     <joint name="world_to_platform" type="fixed">
       <parent link="world" />
-      <child link="$(arg external_axis_prefix)aico2_x2_base_link" />
+      <child link="$(arg external_axis_prefix)aico2_4_v2_base_link" />
+      <origin xyz="0 0 0" rpy="0 0 0" />
+    </joint>
+  </xacro:if>
+  <xacro:if value="${'$(arg external_axis_type)' == 'aico2_10_v1'}">
+    <xacro:aico2_10_v1 prefix="$(arg external_axis_prefix)"
+      left_arm_prefix="${calculated_left_arm_prefix}"
+      right_arm_prefix="${calculated_right_arm_prefix}"
+      mesh_prefix_path="package://flexiv_description/" />
+    <joint name="world_to_platform" type="fixed">
+      <parent link="world" />
+      <child link="$(arg external_axis_prefix)aico2_10_v1_base_link" />
       <origin xyz="0 0 0" rpy="0 0 0" />
     </joint>

File: urdf/common/aico2_10_v1.xacro (robot description, xacro)
@@ -1,33 +1,33 @@
 <?xml version="1.0" encoding="utf-8"?>
 <robot xmlns:xacro="http://wiki.ros.org/xacro">
-  <xacro:macro name="aico2_platform_x2"
+  <xacro:macro name="aico2_10_v1"
     params="prefix left_arm_prefix right_arm_prefix mesh_prefix_path">
-    <joint name="${prefix}aico2_x2_joint1" type="revolute">
+    <joint name="${prefix}aico2_10_v1_joint1" type="revolute">
       <origin xyz="0 0 0.804" rpy="0 0 0" />
-      <parent link="${prefix}aico2_x2_base_link" />
-      <child link="${prefix}aico2_x2_link1" />
+      <parent link="${prefix}aico2_10_v1_base_link" />
+      <child link="${prefix}aico2_10_v1_link1" />
       <axis xyz="0 0 1" />
-      <limit lower="-1.57" upper="1.57" effort="1000" velocity="1" />
+      <limit lower="-1.57" upper="1.57" effort="1000" velocity="1.047" />
     </joint>
-    <joint name="${prefix}aico2_x2_joint2" type="revolute">
+    <joint name="${prefix}aico2_10_v1_joint2" type="revolute">
       <origin xyz="0 0 0.116" rpy="0 0 0" />
-      <parent link="${prefix}aico2_x2_link1" />
-      <child link="${prefix}aico2_x2_link2" />
+      <parent link="${prefix}aico2_10_v1_link1" />
+      <child link="${prefix}aico2_10_v1_link2" />
       <axis xyz="0 1 0" />
-      <limit lower="0" upper="1.57" effort="1900" velocity="1" />
+      <limit lower="0" upper="1.57" effort="1900" velocity="1.047" />
     </joint>
-    <joint name="${prefix}aico2_x2_left_arm_adapter" type="fixed">
+    <joint name="${prefix}aico2_10_v1_left_arm_adapter" type="fixed">
       <origin xyz="0 -0.0375 0.33" rpy="-1.5708 1.5708 0" />
-      <parent link="${prefix}aico2_x2_link2" />
+      <parent link="${prefix}aico2_10_v1_link2" />
       <child link="${left_arm_prefix}base_link" />
       <axis xyz="0 0 0" />
     </joint>
-    <joint name="${prefix}aico2_x2_right_arm_adapter" type="fixed">
+    <joint name="${prefix}aico2_10_v1_right_arm_adapter" type="fixed">
       <origin xyz="0 0.0375 0.33" rpy="1.5708 -1.5708 0" />
-      <parent link="${prefix}aico2_x2_link2" />
+      <parent link="${prefix}aico2_10_v1_link2" />
       <child link="${right_arm_prefix}base_link" />
       <axis xyz="0 0 0" />
     </joint>
-    <link name="${prefix}aico2_x2_base_link">
+    <link name="${prefix}aico2_10_v1_base_link">
       <inertial>
         <origin xyz="-0.006 -0.00638 0.157" rpy="0 0 0" />
@@ -38,5 +38,5 @@
         <origin xyz="0 0 0" rpy="0 0 0" />
         <geometry>
-          <mesh filename="${mesh_prefix_path}meshes/AICO2-X2/visual/base_link.obj" />
+          <mesh filename="${mesh_prefix_path}meshes/AICO2-10-V1/visual/base_link.obj" />
         </geometry>
         <material name="">
@@ -47,9 +47,9 @@
         <origin xyz="0 0 0" rpy="0 0 0" />
         <geometry>
-          <mesh filename="${mesh_prefix_path}meshes/AICO2-X2/collision/base_link.stl" />
+          <mesh filename="${mesh_prefix_path}meshes/AICO2-10-V1/collision/base_link.stl" />
         </geometry>
       </collision>
     </link>
-    <link name="${prefix}aico2_x2_link1">
+    <link name="${prefix}aico2_10_v1_link1">
       <inertial>
         <origin xyz="-0.00685 -0.00021 -0.073" rpy="0 0 0" />
@@ -60,5 +60,5 @@
         <origin xyz="0 0 0" rpy="0 0 0" />
         <geometry>
-          <mesh filename="${mesh_prefix_path}meshes/AICO2-X2/visual/link1.obj" />
+          <mesh filename="${mesh_prefix_path}meshes/AICO2-10-V1/visual/link1.obj" />
         </geometry>
         <material name="">
@@ -69,9 +69,9 @@
         <origin xyz="0 0 0" rpy="0 0 0" />
         <geometry>
-          <mesh filename="${mesh_prefix_path}meshes/AICO2-X2/collision/link1.stl" />
+          <mesh filename="${mesh_prefix_path}meshes/AICO2-10-V1/collision/link1.stl" />
         </geometry>
       </collision>
     </link>
-    <link name="${prefix}aico2_x2_link2">
+    <link name="${prefix}aico2_10_v1_link2">
       <inertial>
         <origin xyz="0.00217 3E-05 0.3" rpy="0 0 0" />
@@ -82,5 +82,5 @@
         <origin xyz="0 0 0" rpy="0 0 0" />
         <geometry>
-          <mesh filename="${mesh_prefix_path}meshes/AICO2-X2/visual/link2.obj" />
+          <mesh filename="${mesh_prefix_path}meshes/AICO2-10-V1/visual/link2.obj" />
         </geometry>
         <material name="">
@@ -91,5 +91,5 @@
         <origin xyz="0 0 0" rpy="0 0 0" />
         <geometry>
-          <mesh filename="${mesh_prefix_path}meshes/AICO2-X2/collision/link2.stl" />
+          <mesh filename="${mesh_prefix_path}meshes/AICO2-10-V1/collision/link2.stl" />
         </geometry>
       </collision>

File: urdf/common/aico2_4_v1.xacro (robot description, xacro)
@@ -1,33 +1,33 @@
 <?xml version="1.0" encoding="utf-8"?>
 <robot xmlns:xacro="http://wiki.ros.org/xacro">
-  <xacro:macro name="aico2_platform_x1"
+  <xacro:macro name="aico2_4_v1"
     params="prefix left_arm_prefix right_arm_prefix mesh_prefix_path">
-    <joint name="${prefix}aico2_x1_joint1" type="revolute">
+    <joint name="${prefix}aico2_4_v1_joint1" type="revolute">
       <origin xyz="0 0 0.307" rpy="0 0 0" />
-      <parent link="${prefix}aico2_x1_base_link" />
-      <child link="${prefix}aico2_x1_link1" />
+      <parent link="${prefix}aico2_4_v1_base_link" />
+      <child link="${prefix}aico2_4_v1_link1" />
       <axis xyz="0 0 1" />
       <limit lower="-1.57" upper="1.57" effort="400" velocity="1.05" />
     </joint>
-    <joint name="${prefix}aico2_x1_joint2" type="revolute">
+    <joint name="${prefix}aico2_4_v1_joint2" type="revolute">
       <origin xyz="0.025 0 0" rpy="0 0 0" />
-      <parent link="${prefix}aico2_x1_link1" />
-      <child link="${prefix}aico2_x1_link2" />
+      <parent link="${prefix}aico2_4_v1_link1" />
+      <child link="${prefix}aico2_4_v1_link2" />
       <axis xyz="0 1 0" />
-      <limit lower="0" upper="1.57" effort="365" velocity="1" />
+      <limit lower="0" upper="1.57" effort="1000" velocity="1.05" />
     </joint>
-    <joint name="${prefix}aico2_x1_left_arm_adapter" type="fixed">
+    <joint name="${prefix}aico2_4_v1_left_arm_adapter" type="fixed">
       <origin xyz="0 -0.035 0.2885" rpy="-1.5708 0 0" />
-      <parent link="${prefix}aico2_x1_link2" />
+      <parent link="${prefix}aico2_4_v1_link2" />
       <child link="${left_arm_prefix}base_link" />
       <axis xyz="0 0 0" />
     </joint>
-    <joint name="${prefix}aico2_x1_right_arm_adapter" type="fixed">
+    <joint name="${prefix}aico2_4_v1_right_arm_adapter" type="fixed">
       <origin xyz="0 0.035 0.2885" rpy="1.5708 0 0" />
-      <parent link="${prefix}aico2_x1_link2" />
+      <parent link="${prefix}aico2_4_v1_link2" />
       <child link="${right_arm_prefix}base_link" />
       <axis xyz="0 0 0" />
     </joint>
-    <link name="${prefix}aico2_x1_base_link">
+    <link name="${prefix}aico2_4_v1_base_link">
       <inertial>
         <origin xyz="0.0052 -0.0154 0.258" rpy="0 0 0" />
@@ -38,5 +38,5 @@
         <origin xyz="0 0 0" rpy="0 0 1.5708" />
         <geometry>
-          <mesh filename="${mesh_prefix_path}meshes/AICO2-X1/visual/base_link.obj"
+          <mesh filename="${mesh_prefix_path}meshes/AICO2-4-V1/visual/base_link.obj"
             scale="0.001 0.001 0.001" />
         </geometry>
@@ -48,9 +48,9 @@
         <origin xyz="0 0 0" rpy="0 0 0" />
         <geometry>
-          <mesh filename="${mesh_prefix_path}meshes/AICO2-X1/collision/base_link.stl" />
+          <mesh filename="${mesh_prefix_path}meshes/AICO2-4-V1/collision/base_link.stl" />
         </geometry>
       </collision>
     </link>
-    <link name="${prefix}aico2_x1_link1">
+    <link name="${prefix}aico2_4_v1_link1">
       <inertial>
         <origin xyz="0.0484 -6.38E-05 -0.134" rpy="0 0 0" />
@@ -61,5 +61,5 @@
         <origin xyz="0 0 0" rpy="0 0 1.5708" />
         <geometry>
-          <mesh filename="${mesh_prefix_path}meshes/AICO2-X1/visual/link1.obj" />
+          <mesh filename="${mesh_prefix_path}meshes/AICO2-4-V1/visual/link1.obj" />
         </geometry>
         <material name="">
@@ -70,9 +70,9 @@
         <origin xyz="0 0 0" rpy="0 0 0" />
         <geometry>
-          <mesh filename="${mesh_prefix_path}meshes/AICO2-X1/collision/link1.stl" />
+          <mesh filename="${mesh_prefix_path}meshes/AICO2-4-V1/collision/link1.stl" />
         </geometry>
       </collision>
     </link>
-    <link name="${prefix}aico2_x1_link2">
+    <link name="${prefix}aico2_4_v1_link2">
       <inertial>
         <origin xyz="-0.0155 0.00056 0.25" rpy="0 0 0" />
@@ -83,5 +83,5 @@
         <origin xyz="0 0 0" rpy="0 0 1.5708" />
         <geometry>
-          <mesh filename="${mesh_prefix_path}meshes/AICO2-X1/visual/link2.obj" />
+          <mesh filename="${mesh_prefix_path}meshes/AICO2-4-V1/visual/link2.obj" />
         </geometry>
         <material name="">
@@ -92,5 +92,5 @@
         <origin xyz="0 0 0" rpy="0 0 0" />
         <geometry>
-          <mesh filename="${mesh_prefix_path}meshes/AICO2-X1/collision/link2.stl" />
+          <mesh filename="${mesh_prefix_path}meshes/AICO2-4-V1/collision/link2.stl" />
         </geometry>
       </collision>

File: urdf/common/rizon_dual.ros2_control.xacro (robot description, xacro)
@@ -66,6 +66,6 @@
       <xacro:configure_joint joint_name="${prefix_left}joint7" initial_pos="${initial_positions_left['joint7']}" />
       <!-- External axis joints -->
-      <xacro:if value="${external_axis_type == 'aico2_platform_x1'}">
-        <joint name="${external_axis_prefix}aico2_x1_joint1">
+      <xacro:if value="${external_axis_type == 'aico2_4_v1'}">
+        <joint name="${external_axis_prefix}aico2_4_v1_joint1">
           <command_interface name="position" />
           <command_interface name="velocity" />
@@ -77,5 +77,5 @@
           <state_interface name="effort" />
         </joint>
-        <joint name="${external_axis_prefix}aico2_x1_joint2">
+        <joint name="${external_axis_prefix}aico2_4_v1_joint2">
           <command_interface name="position" />
           <command_interface name="velocity" />
@@ -88,6 +88,6 @@
         </joint>
       </xacro:if>
-      <xacro:if value="${external_axis_type == 'aico2_platform_x2'}">
-        <joint name="${external_axis_prefix}aico2_x2_joint1">
+      <xacro:if value="${external_axis_type == 'aico2_4_v2'}">
+        <joint name="${external_axis_prefix}aico2_4_v2_joint1">
           <command_interface name="position" />
           <command_interface name="velocity" />
@@ -99,5 +99,27 @@
           <state_interface name="effort" />
         </joint>
-        <joint name="${external_axis_prefix}aico2_x2_joint2">
+        <joint name="${external_axis_prefix}aico2_4_v2_joint2">
+          <command_interface name="position" />
+          <command_interface name="velocity" />
+          <command_interface name="effort" />
+          <state_interface name="position">
+            <param name="initial_value">0.0</param>
+          </state_interface>
+          <state_interface name="velocity" />
+          <state_interface name="effort" />
+        </joint>
+      </xacro:if>
+      <xacro:if value="${external_axis_type == 'aico2_10_v1'}">
+        <joint name="${external_axis_prefix}aico2_10_v1_joint1">
+          <command_interface name="position" />
+          <command_interface name="velocity" />
+          <command_interface name="effort" />
+          <state_interface name="position">
+            <param name="initial_value">0.0</param>
+          </state_interface>
+          <state_interface name="velocity" />
+          <state_interface name="effort" />
+        </joint>
+        <joint name="${external_axis_prefix}aico2_10_v1_joint2">
           <command_interface name="position" />
           <command_interface name="velocity" />
