Commit message: Refactor robot serial number handling for dual-arm configuration in URDF and launch files

File: urdf/aico2.urdf.xacro (robot description, xacro)
@@ -4,6 +4,5 @@
   <xacro:arg name="external_axis_prefix" default="" />
   <xacro:arg name="rizon_type" default="Rizon4" />
-  <xacro:arg name="robot_sn_left" default="" />
-  <xacro:arg name="robot_sn_right" default="" />
+  <xacro:arg name="robot_sn" default="" />
   <!-- Determine Rizon left and right types based on rizon_type -->
   <xacro:if value="${'$(arg rizon_type)' == 'Rizon4'}">
@@ -45,7 +44,7 @@
   <!-- Calculate the actual prefixes rizon_robot will use -->
   <xacro:property name="calculated_left_arm_prefix"
-    value="${(left_arm_prefix_arg + '_' + '$(arg robot_sn_left)' + '_') if left_arm_prefix_arg != '' and '$(arg robot_sn_left)' != '' else (left_arm_prefix_arg + '$(arg robot_sn_left)' + '_') if (left_arm_prefix_arg + '$(arg robot_sn_left)') != '' else ''}" />
+    value="${(left_arm_prefix_arg + '_' + '$(arg robot_sn)' + '_') if left_arm_prefix_arg != '' and '$(arg robot_sn)' != '' else (left_arm_prefix_arg + '$(arg robot_sn)' + '_') if (left_arm_prefix_arg + '$(arg robot_sn)') != '' else ''}" />
   <xacro:property name="calculated_right_arm_prefix"
-    value="${(right_arm_prefix_arg + '_' + '$(arg robot_sn_right)' + '_') if right_arm_prefix_arg != '' and '$(arg robot_sn_right)' != '' else (right_arm_prefix_arg + '$(arg robot_sn_right)' + '_') if (right_arm_prefix_arg + '$(arg robot_sn_right)') != '' else ''}" />
+    value="${(right_arm_prefix_arg + '_' + '$(arg robot_sn)' + '_') if right_arm_prefix_arg != '' and '$(arg robot_sn)' != '' else (right_arm_prefix_arg + '$(arg robot_sn)' + '_') if (right_arm_prefix_arg + '$(arg robot_sn)') != '' else ''}" />
   <!-- Instantiate External Axis -->
   <link name="world" />
@@ -86,5 +85,5 @@
   <xacro:rizon_robot
     rizon_type="${rizon_type_left}"
-    robot_sn="$(arg robot_sn_left)"
+    robot_sn="$(arg robot_sn)"
     joint_limits_parameters_file="$(find flexiv_description)/config/${rizon_type_left}/joint_limits.yaml"
     kinematics_parameters_file="$(find flexiv_description)/config/${rizon_type_left}/default_kinematics.yaml"
@@ -102,5 +101,5 @@
   <xacro:rizon_robot
     rizon_type="${rizon_type_right}"
-    robot_sn="$(arg robot_sn_right)"
+    robot_sn="$(arg robot_sn)"
     joint_limits_parameters_file="$(find flexiv_description)/config/${rizon_type_right}/joint_limits.yaml"
     kinematics_parameters_file="$(find flexiv_description)/config/${rizon_type_right}/default_kinematics.yaml"
@@ -120,6 +119,5 @@
       prefix_left="${calculated_left_arm_prefix}"
       prefix_right="${calculated_right_arm_prefix}"
-      robot_sn_left="$(arg robot_sn_left)"
-      robot_sn_right="$(arg robot_sn_right)"
+      robot_sn="$(arg robot_sn)"
       rdk_control_mode="$(arg rdk_control_mode)"
       use_fake_hardware="$(arg use_fake_hardware)"

File: urdf/common/rizon.ros2_control.xacro (robot description, xacro)
@@ -142,42 +142,14 @@
         </joint>
       </xacro:if>
-      <!-- 18 digital IO ports (16 on control box + 2 inside the wrist connector) -->
+      <!-- 24 digital IO ports (16 on control box + 2 inside the wrist connector per wrist, max 4 wrists) -->
+      <xacro:macro name="loop_gpio" params="idx">
+        <command_interface name="digital_output_${idx}" />
+        <state_interface name="digital_input_${idx}" />
+        <xacro:if value="${idx &lt; 23}">
+          <xacro:loop_gpio idx="${idx+1}" />
+        </xacro:if>
+      </xacro:macro>
       <gpio name="${prefix}gpio">
-        <command_interface name="digital_output_0" />
-        <command_interface name="digital_output_1" />
-        <command_interface name="digital_output_2" />
-        <command_interface name="digital_output_3" />
-        <command_interface name="digital_output_4" />
-        <command_interface name="digital_output_5" />
-        <command_interface name="digital_output_6" />
-        <command_interface name="digital_output_7" />
-        <command_interface name="digital_output_8" />
-        <command_interface name="digital_output_9" />
-        <command_interface name="digital_output_10" />
-        <command_interface name="digital_output_11" />
-        <command_interface name="digital_output_12" />
-        <command_interface name="digital_output_13" />
-        <command_interface name="digital_output_14" />
-        <command_interface name="digital_output_15" />
-        <command_interface name="digital_output_16" />
-        <command_interface name="digital_output_17" />
-        <state_interface name="digital_input_0" />
-        <state_interface name="digital_input_1" />
-        <state_interface name="digital_input_2" />
-        <state_interface name="digital_input_3" />
-        <state_interface name="digital_input_4" />
-        <state_interface name="digital_input_5" />
-        <state_interface name="digital_input_6" />
-        <state_interface name="digital_input_7" />
-        <state_interface name="digital_input_8" />
-        <state_interface name="digital_input_9" />
-        <state_interface name="digital_input_10" />
-        <state_interface name="digital_input_11" />
-        <state_interface name="digital_input_12" />
-        <state_interface name="digital_input_13" />
-        <state_interface name="digital_input_14" />
-        <state_interface name="digital_input_15" />
-        <state_interface name="digital_input_16" />
-        <state_interface name="digital_input_17" />
+        <xacro:loop_gpio idx="0" />
       </gpio>
     </ros2_control>

File: urdf/common/rizon_dual.ros2_control.xacro (robot description, xacro)
@@ -5,6 +5,5 @@
     prefix_left
     prefix_right
-    robot_sn_left
-    robot_sn_right
+    robot_sn
     rdk_control_mode:='joint_position'
     use_fake_hardware:=false
@@ -23,5 +22,24 @@
     <xacro:property name="initial_positions_left" value="${xacro.load_yaml(initial_positions_file_left)['initial_positions']}"/>
     <xacro:property name="initial_positions_right" value="${xacro.load_yaml(initial_positions_file_right)['initial_positions']}"/>
-    <ros2_control name="FlexivDualHardwareInterface" type="system">
+    <xacro:macro name="configure_joint" params="joint_name initial_pos">
+      <joint name="${joint_name}">
+        <command_interface name="position" />
+        <command_interface name="velocity" />
+        <command_interface name="effort" />
+        <state_interface name="position">
+          <param name="initial_value">${initial_pos}</param>
+        </state_interface>
+        <state_interface name="velocity" />
+        <state_interface name="effort" />
+      </joint>
+    </xacro:macro>
+    <xacro:macro name="loop_gpio" params="idx">
+      <command_interface name="digital_output_${idx}" />
+      <state_interface name="digital_input_${idx}" />
+      <xacro:if value="${idx &lt; 23}">
+        <xacro:loop_gpio idx="${idx+1}" />
+      </xacro:if>
+    </xacro:macro>
+    <ros2_control name="FlexivHardwareInterface" type="system">
       <hardware>
         <xacro:if value="${use_fake_hardware}">
@@ -31,38 +49,11 @@
         </xacro:if>
         <xacro:unless value="${use_fake_hardware}">
-          <plugin>flexiv_hardware/FlexivDualHardwareInterface</plugin>
-          <param name="robot_sn_left">${robot_sn_left}</param>
-          <param name="robot_sn_right">${robot_sn_right}</param>
+          <plugin>flexiv_hardware/FlexivHardwareInterface</plugin>
+          <param name="robot_sn">${robot_sn}</param>
           <param name="prefix_left">${prefix_left}</param>
           <param name="prefix_right">${prefix_right}</param>
           <param name="rdk_control_mode">${rdk_control_mode}</param>
-          <param name="external_axis_type">${external_axis_type}</param>
-          <param name="translation_left_x">${translation_left_x}</param>
-          <param name="translation_left_y">${translation_left_y}</param>
-          <param name="translation_left_z">${translation_left_z}</param>
-          <param name="translation_right_x">${translation_right_x}</param>
-          <param name="translation_right_y">${translation_right_y}</param>
-          <param name="translation_right_z">${translation_right_z}</param>
         </xacro:unless>
       </hardware>
-      <xacro:macro name="configure_joint" params="joint_name initial_pos">
-        <joint name="${joint_name}">
-          <command_interface name="position" />
-          <command_interface name="velocity" />
-          <command_interface name="effort" />
-          <state_interface name="position">
-            <param name="initial_value">${initial_pos}</param>
-          </state_interface>
-          <state_interface name="velocity" />
-          <state_interface name="effort" />
-        </joint>
-      </xacro:macro>
-      <xacro:configure_joint joint_name="${prefix_left}joint1" initial_pos="${initial_positions_left['joint1']}" />
-      <xacro:configure_joint joint_name="${prefix_left}joint2" initial_pos="${initial_positions_left['joint2']}" />
-      <xacro:configure_joint joint_name="${prefix_left}joint3" initial_pos="${initial_positions_left['joint3']}" />
-      <xacro:configure_joint joint_name="${prefix_left}joint4" initial_pos="${initial_positions_left['joint4']}" />
-      <xacro:configure_joint joint_name="${prefix_left}joint5" initial_pos="${initial_positions_left['joint5']}" />
-      <xacro:configure_joint joint_name="${prefix_left}joint6" initial_pos="${initial_positions_left['joint6']}" />
-      <xacro:configure_joint joint_name="${prefix_left}joint7" initial_pos="${initial_positions_left['joint7']}" />
       <!-- External axis joints -->
       <xacro:if value="${external_axis_type == 'aico2_4_v1'}">
@@ -132,4 +123,11 @@
         </joint>
       </xacro:if>
+      <xacro:configure_joint joint_name="${prefix_left}joint1" initial_pos="${initial_positions_left['joint1']}" />
+      <xacro:configure_joint joint_name="${prefix_left}joint2" initial_pos="${initial_positions_left['joint2']}" />
+      <xacro:configure_joint joint_name="${prefix_left}joint3" initial_pos="${initial_positions_left['joint3']}" />
+      <xacro:configure_joint joint_name="${prefix_left}joint4" initial_pos="${initial_positions_left['joint4']}" />
+      <xacro:configure_joint joint_name="${prefix_left}joint5" initial_pos="${initial_positions_left['joint5']}" />
+      <xacro:configure_joint joint_name="${prefix_left}joint6" initial_pos="${initial_positions_left['joint6']}" />
+      <xacro:configure_joint joint_name="${prefix_left}joint7" initial_pos="${initial_positions_left['joint7']}" />
       <xacro:configure_joint joint_name="${prefix_right}joint1" initial_pos="${initial_positions_right['joint1']}" />
       <xacro:configure_joint joint_name="${prefix_right}joint2" initial_pos="${initial_positions_right['joint2']}" />
@@ -139,16 +137,5 @@
       <xacro:configure_joint joint_name="${prefix_right}joint6" initial_pos="${initial_positions_right['joint6']}" />
       <xacro:configure_joint joint_name="${prefix_right}joint7" initial_pos="${initial_positions_right['joint7']}" />
-      <!-- 18 digital IO ports per robot -->
-      <xacro:macro name="loop_gpio" params="idx">
-        <command_interface name="digital_output_${idx}" />
-        <state_interface name="digital_input_${idx}" />
-        <xacro:if value="${idx &lt; 17}">
-          <xacro:loop_gpio idx="${idx+1}" />
-        </xacro:if>
-      </xacro:macro>
-      <gpio name="${prefix_left}gpio">
-        <xacro:loop_gpio idx="0" />
-      </gpio>
-      <gpio name="${prefix_right}gpio">
+      <gpio name="${robot_sn}_gpio">
         <xacro:loop_gpio idx="0" />
       </gpio>

File: urdf/rizon_dual.urdf.xacro (robot description, xacro)
@@ -1,6 +1,5 @@
 <?xml version="1.0" encoding="utf-8"?>
 <robot xmlns:xacro="http://www.ros.org/wiki/xacro" name="rizon_dual">
-  <xacro:arg name="robot_sn_left" default="" />
-  <xacro:arg name="robot_sn_right" default="" />
+  <xacro:arg name="robot_sn" default="" />
   <xacro:arg name="rizon_type_left" default="Rizon4" />
   <xacro:arg name="rizon_type_right" default="Rizon4R" />
@@ -22,6 +21,6 @@
   <xacro:include filename="$(find flexiv_description)/urdf/common/rizon_dual.ros2_control.xacro" />
   <!-- Define prefixes -->
-  <xacro:property name="prefix_left" value="left_$(arg robot_sn_left)_" />
-  <xacro:property name="prefix_right" value="right_$(arg robot_sn_right)_" />
+  <xacro:property name="prefix_left" value="left_$(arg robot_sn)_" />
+  <xacro:property name="prefix_right" value="right_$(arg robot_sn)_" />
   <xacro:property name="mounting" value="${xacro.load_yaml('$(arg mounting_file)')}" />
   <link name="world" />
@@ -29,5 +28,5 @@
   <xacro:rizon_robot
     rizon_type="$(arg rizon_type_left)"
-    robot_sn="$(arg robot_sn_left)"
+    robot_sn="$(arg robot_sn)"
     joint_limits_parameters_file="$(find flexiv_description)/config/$(arg rizon_type_left)/joint_limits.yaml"
     kinematics_parameters_file="$(find flexiv_description)/config/$(arg rizon_type_left)/default_kinematics.yaml"
@@ -46,5 +45,5 @@
   <xacro:rizon_robot
     rizon_type="$(arg rizon_type_right)"
-    robot_sn="$(arg robot_sn_right)"
+    robot_sn="$(arg robot_sn)"
     joint_limits_parameters_file="$(find flexiv_description)/config/$(arg rizon_type_right)/joint_limits.yaml"
     kinematics_parameters_file="$(find flexiv_description)/config/$(arg rizon_type_right)/default_kinematics.yaml"
@@ -65,6 +64,5 @@
       prefix_left="${prefix_left}"
       prefix_right="${prefix_right}"
-      robot_sn_left="$(arg robot_sn_left)"
-      robot_sn_right="$(arg robot_sn_right)"
+      robot_sn="$(arg robot_sn)"
       rdk_control_mode="$(arg rdk_control_mode)"
       use_fake_hardware="$(arg use_fake_hardware)"
