Commit message: Add platform parameters and joint configurations for AICO1 and AICO2 in URDF files

File: urdf/aico1.urdf.xacro (robot description, xacro)
@@ -61,4 +61,7 @@
     add_world_link="false"
     create_base_joint="false"
+    platform_name="aico1"
+    platform_type="$(arg platform_type)"
+    platform_prefix="$(arg platform_prefix)"
   />
 </robot>

File: urdf/aico2.urdf.xacro (robot description, xacro)
@@ -107,4 +107,7 @@
       translation_right_y="0"
       translation_right_z="0"
+      platform_name="aico2"
+      platform_type="$(arg platform_type)"
+      platform_prefix="$(arg platform_prefix)"
     />
   </xacro:if>

File: urdf/common/rizon.ros2_control.xacro (robot description, xacro)
@@ -9,4 +9,7 @@
     fake_sensor_commands:=false
     initial_positions_file
+    platform_name:=''
+    platform_type:=''
+    platform_prefix:=''
     ">
     <xacro:property name="initial_positions" value="${xacro.load_yaml(initial_positions_file)['initial_positions']}"/>
@@ -95,4 +98,51 @@
         <state_interface name="effort" />
       </joint>
+      <!-- Platform joints -->
+      <xacro:if value="${platform_name == 'aico1'}">
+        <xacro:if value="${platform_type == 'X1'}">
+          <joint name="${platform_prefix}aico1_x1_joint2">
+            <command_interface name="position" />
+            <command_interface name="velocity" />
+            <command_interface name="effort" />
+            <state_interface name="position">
+              <param name="initial_value">0.0</param>
+            </state_interface>
+            <state_interface name="velocity" />
+            <state_interface name="effort" />
+          </joint>
+        </xacro:if>
+        <xacro:if value="${platform_type == 'X2'}">
+          <joint name="${platform_prefix}aico1_x2_joint1">
+            <command_interface name="position" />
+            <command_interface name="velocity" />
+            <command_interface name="effort" />
+            <state_interface name="position">
+              <param name="initial_value">0.0</param>
+            </state_interface>
+            <state_interface name="velocity" />
+            <state_interface name="effort" />
+          </joint>
+          <joint name="${platform_prefix}aico1_x2_joint2">
+            <command_interface name="position" />
+            <command_interface name="velocity" />
+            <command_interface name="effort" />
+            <state_interface name="position">
+              <param name="initial_value">0.0</param>
+            </state_interface>
+            <state_interface name="velocity" />
+            <state_interface name="effort" />
+          </joint>
+          <joint name="${platform_prefix}aico1_x2_joint_head">
+            <command_interface name="position" />
+            <command_interface name="velocity" />
+            <command_interface name="effort" />
+            <state_interface name="position">
+              <param name="initial_value">0.0</param>
+            </state_interface>
+            <state_interface name="velocity" />
+            <state_interface name="effort" />
+          </joint>
+        </xacro:if>
+      </xacro:if>
       <!-- 18 digital IO ports (16 on control box + 2 inside the wrist connector) -->
       <gpio name="${prefix}gpio">

File: urdf/common/rizon_dual.ros2_control.xacro (robot description, xacro)
@@ -18,4 +18,7 @@
     translation_right_y:=0.0
     translation_right_z:=0.0
+    platform_name:=''
+    platform_type:=''
+    platform_prefix:=''
     ">
     <xacro:property name="initial_positions_left" value="${xacro.load_yaml(initial_positions_file_left)['initial_positions']}"/>
@@ -43,16 +46,4 @@
         </xacro:unless>
       </hardware>
-      <xacro:macro name="configure_joint" params="joint_name initial_pos">
-        <joint name="${joint_name}">
-          <command_interface name="position" />
-          <command_interface name="velocity" />
-          <command_interface name="effort" />
-          <state_interface name="position">
-            <param name="initial_value">${initial_pos}</param>
-          </state_interface>
-          <state_interface name="velocity" />
-          <state_interface name="effort" />
-        </joint>
-      </xacro:macro>
       <xacro:configure_joint joint_name="${prefix_left}joint1" initial_pos="${initial_positions_left['joint1']}" />
       <xacro:configure_joint joint_name="${prefix_left}joint2" initial_pos="${initial_positions_left['joint2']}" />
@@ -62,4 +53,51 @@
       <xacro:configure_joint joint_name="${prefix_left}joint6" initial_pos="${initial_positions_left['joint6']}" />
       <xacro:configure_joint joint_name="${prefix_left}joint7" initial_pos="${initial_positions_left['joint7']}" />
+      <!-- Platform joints -->
+      <xacro:if value="${platform_name == 'aico2'}">
+        <xacro:if value="${platform_type == 'X1'}">
+          <joint name="${platform_prefix}aico2_x1_joint1">
+            <command_interface name="position" />
+            <command_interface name="velocity" />
+            <command_interface name="effort" />
+            <state_interface name="position">
+              <param name="initial_value">0.0</param>
+            </state_interface>
+            <state_interface name="velocity" />
+            <state_interface name="effort" />
+          </joint>
+          <joint name="${platform_prefix}aico2_x1_joint2">
+            <command_interface name="position" />
+            <command_interface name="velocity" />
+            <command_interface name="effort" />
+            <state_interface name="position">
+              <param name="initial_value">0.0</param>
+            </state_interface>
+            <state_interface name="velocity" />
+            <state_interface name="effort" />
+          </joint>
+        </xacro:if>
+        <xacro:if value="${platform_type == 'X2'}">
+          <joint name="${platform_prefix}aico2_x2_joint1">
+            <command_interface name="position" />
+            <command_interface name="velocity" />
+            <command_interface name="effort" />
+            <state_interface name="position">
+              <param name="initial_value">0.0</param>
+            </state_interface>
+            <state_interface name="velocity" />
+            <state_interface name="effort" />
+          </joint>
+          <joint name="${platform_prefix}aico2_x2_joint2">
+            <command_interface name="position" />
+            <command_interface name="velocity" />
+            <command_interface name="effort" />
+            <state_interface name="position">
+              <param name="initial_value">0.0</param>
+            </state_interface>
+            <state_interface name="velocity" />
+            <state_interface name="effort" />
+          </joint>
+        </xacro:if>
+      </xacro:if>
       <xacro:configure_joint joint_name="${prefix_right}joint1" initial_pos="${initial_positions_right['joint1']}" />
       <xacro:configure_joint joint_name="${prefix_right}joint2" initial_pos="${initial_positions_right['joint2']}" />

File: urdf/common/rizon_robot.xacro (robot description, xacro)
@@ -22,4 +22,7 @@
     base_xyz:='0.0 0.0 0.0'
     base_rpy:='0.0 0.0 0.0'
+    platform_name:=''
+    platform_type:=''
+    platform_prefix:=''
     ">
     <!-- Prefix defaults to 'arm_prefix_robot_sn' -->
@@ -55,4 +58,7 @@
         fake_sensor_commands="${fake_sensor_commands}"
         initial_positions_file="${initial_positions_file}"
+        platform_name="${platform_name}"
+        platform_type="${platform_type}"
+        platform_prefix="${platform_prefix}"
       />
     </xacro:if>

Commit message: Update AICO1 and AICO2 URDF generation and visualization scripts to support specific Rizon types

File: urdf/aico1.urdf.xacro (robot description, xacro)
@@ -16,4 +16,8 @@
   <xacro:arg name="initial_positions_file"
     default="$(find flexiv_description)/config/initial_positions.yaml" />
+  <!-- Validate rizon_type -->
+  <xacro:if value="${'$(arg rizon_type)' != 'Rizon4' and '$(arg rizon_type)' != 'Rizon4s'}">
+    ${xacro.warning('AICO1 only supports Rizon4 and Rizon4s. You selected $(arg rizon_type).')}
+  </xacro:if>
   <xacro:include filename="$(find flexiv_description)/urdf/common/aico1_platform_x1.xacro" />
   <xacro:include filename="$(find flexiv_description)/urdf/common/aico1_platform_x2.xacro" />

File: urdf/aico2.urdf.xacro (robot description, xacro)
@@ -5,6 +5,13 @@
   <xacro:arg name="robot_sn_left" default="" />
   <xacro:arg name="robot_sn_right" default="" />
-  <xacro:arg name="rizon_type_left" default="Rizon4" />
-  <xacro:arg name="rizon_type_right" default="Rizon4R" />
+  <!-- Determine Rizon types based on platform_type -->
+  <xacro:if value="${'$(arg platform_type)' == 'X1'}">
+    <xacro:property name="rizon_type_left" value="Rizon4" />
+    <xacro:property name="rizon_type_right" value="Rizon4R" />
+  </xacro:if>
+  <xacro:if value="${'$(arg platform_type)' == 'X2'}">
+    <xacro:property name="rizon_type_left" value="Rizon10" />
+    <xacro:property name="rizon_type_right" value="Rizon10" />
+  </xacro:if>
   <xacro:arg name="load_gripper_left" default="false" />
   <xacro:arg name="gripper_name_left" default="Flexiv-GN01" />
@@ -59,10 +66,10 @@
   <!-- Left Robot -->
   <xacro:rizon_robot
-    rizon_type="$(arg rizon_type_left)"
+    rizon_type="${rizon_type_left}"
     robot_sn="$(arg robot_sn_left)"
-    joint_limits_parameters_file="$(find flexiv_description)/config/$(arg rizon_type_left)/joint_limits.yaml"
-    kinematics_parameters_file="$(find flexiv_description)/config/$(arg rizon_type_left)/default_kinematics.yaml"
-    inertia_parameters_file="$(find flexiv_description)/config/$(arg rizon_type_left)/inertia_parameters.yaml"
-    visual_parameters_file="$(find flexiv_description)/config/$(arg rizon_type_left)/visual_parameters.yaml"
+    joint_limits_parameters_file="$(find flexiv_description)/config/${rizon_type_left}/joint_limits.yaml"
+    kinematics_parameters_file="$(find flexiv_description)/config/${rizon_type_left}/default_kinematics.yaml"
+    inertia_parameters_file="$(find flexiv_description)/config/${rizon_type_left}/inertia_parameters.yaml"
+    visual_parameters_file="$(find flexiv_description)/config/${rizon_type_left}/visual_parameters.yaml"
     arm_prefix="${left_arm_prefix_arg}"
     load_gripper="$(arg load_gripper_left)"
@@ -75,10 +82,10 @@
   <!-- Right Robot -->
   <xacro:rizon_robot
-    rizon_type="$(arg rizon_type_right)"
+    rizon_type="${rizon_type_right}"
     robot_sn="$(arg robot_sn_right)"
-    joint_limits_parameters_file="$(find flexiv_description)/config/$(arg rizon_type_right)/joint_limits.yaml"
-    kinematics_parameters_file="$(find flexiv_description)/config/$(arg rizon_type_right)/default_kinematics.yaml"
-    inertia_parameters_file="$(find flexiv_description)/config/$(arg rizon_type_right)/inertia_parameters.yaml"
-    visual_parameters_file="$(find flexiv_description)/config/$(arg rizon_type_right)/visual_parameters.yaml"
+    joint_limits_parameters_file="$(find flexiv_description)/config/${rizon_type_right}/joint_limits.yaml"
+    kinematics_parameters_file="$(find flexiv_description)/config/${rizon_type_right}/default_kinematics.yaml"
+    inertia_parameters_file="$(find flexiv_description)/config/${rizon_type_right}/inertia_parameters.yaml"
+    visual_parameters_file="$(find flexiv_description)/config/${rizon_type_right}/visual_parameters.yaml"
     arm_prefix="${right_arm_prefix_arg}"
     load_gripper="$(arg load_gripper_right)"
