Commit message: Refactor AICO platform parameters to external axis terminology in launch files and URDFs

File: urdf/aico1.urdf.xacro (robot description, xacro)
@@ -2,6 +2,6 @@
 <robot xmlns:xacro="http://www.ros.org/wiki/xacro" name="aico1">
   <!-- Parameters -->
-  <xacro:arg name="platform_type" default="X1" />
-  <xacro:arg name="platform_prefix" default="" />
+  <xacro:arg name="external_axis_type" default="aico1_4_v1" />
+  <xacro:arg name="external_axis_prefix" default="" />
   <xacro:arg name="arm_prefix" default="" />
   <xacro:arg name="robot_sn" default="" />
@@ -17,30 +17,30 @@
     default="$(find flexiv_description)/config/initial_positions.yaml" />
   <!-- Validate rizon_type -->
-  <xacro:if value="${'$(arg rizon_type)' != 'Rizon4' and '$(arg rizon_type)' != 'Rizon4s'}">
-    ${xacro.warning('AICO1 only supports Rizon4 and Rizon4s. You selected $(arg rizon_type).')}
+  <xacro:if value="${'$(arg rizon_type)' != 'Rizon4' and '$(arg rizon_type)' != 'Rizon4s' and '$(arg rizon_type)' != 'Rizon4R'}">
+    ${xacro.warning('AICO1 only supports Rizon4, Rizon4s and Rizon4R. You selected $(arg rizon_type).')}
   </xacro:if>
-  <xacro:include filename="$(find flexiv_description)/urdf/common/aico1_platform_x1.xacro" />
-  <xacro:include filename="$(find flexiv_description)/urdf/common/aico1_platform_x2.xacro" />
+  <xacro:include filename="$(find flexiv_description)/urdf/common/aico1_4_v1.xacro" />
+  <xacro:include filename="$(find flexiv_description)/urdf/common/aico1_4_v2.xacro" />
   <xacro:include filename="$(find flexiv_description)/urdf/common/rizon_robot.xacro" />
   <!-- Calculate the actual prefix rizon_robot will use -->
   <xacro:property name="calculated_arm_prefix"
     value="${('$(arg arm_prefix)' + '_' + '$(arg robot_sn)' + '_') if '$(arg arm_prefix)' != '' and '$(arg robot_sn)' != '' else ('$(arg arm_prefix)' + '$(arg robot_sn)' + '_') if ('$(arg arm_prefix)' + '$(arg robot_sn)') != '' else ''}" />
-  <!-- Instantiate Platform -->
+  <!-- Instantiate External Axis -->
   <link name="world" />
-  <xacro:if value="${'$(arg platform_type)' == 'X1'}">
-    <xacro:aico1_platform_x1 prefix="$(arg platform_prefix)" arm_prefix="${calculated_arm_prefix}"
+  <xacro:if value="${'$(arg external_axis_type)' == 'aico1_4_v1'}">
+    <xacro:aico1_4_v1 prefix="$(arg external_axis_prefix)" arm_prefix="${calculated_arm_prefix}"
       mesh_prefix_path="package://flexiv_description/" />
     <joint name="world_to_platform" type="fixed">
       <parent link="world" />
-      <child link="$(arg platform_prefix)aico1_x1_base_link" />
+      <child link="$(arg external_axis_prefix)aico1_4_v1_base_link" />
       <origin xyz="0 0 0" rpy="0 0 0" />
     </joint>
   </xacro:if>
-  <xacro:if value="${'$(arg platform_type)' == 'X2'}">
-    <xacro:aico1_platform_x2 prefix="$(arg platform_prefix)" arm_prefix="${calculated_arm_prefix}"
+  <xacro:if value="${'$(arg external_axis_type)' == 'aico1_4_v2'}">
+    <xacro:aico1_4_v2 prefix="$(arg external_axis_prefix)" arm_prefix="${calculated_arm_prefix}"
       mesh_prefix_path="package://flexiv_description/" />
     <joint name="world_to_platform" type="fixed">
       <parent link="world" />
-      <child link="$(arg platform_prefix)aico1_x2_agv" />
+      <child link="$(arg external_axis_prefix)aico1_4_v2_base_link" />
       <origin xyz="0 0 0" rpy="0 0 0" />
     </joint>
@@ -65,7 +65,6 @@
     add_world_link="false"
     create_base_joint="false"
-    platform_name="aico1"
-    platform_type="$(arg platform_type)"
-    platform_prefix="$(arg platform_prefix)"
+    external_axis_type="$(arg external_axis_type)"
+    external_axis_prefix="$(arg external_axis_prefix)"
   />
 </robot>

File: urdf/aico2.urdf.xacro (robot description, xacro)
@@ -1,16 +1,18 @@
 <?xml version="1.0" encoding="utf-8"?>
 <robot xmlns:xacro="http://www.ros.org/wiki/xacro" name="aico2">
-  <xacro:arg name="platform_type" default="X1" />
-  <xacro:arg name="platform_prefix" default="" />
+  <xacro:arg name="rizon_type" default="Rizon4" />
+  <xacro:arg name="external_axis_prefix" default="" />
   <xacro:arg name="robot_sn_left" default="" />
   <xacro:arg name="robot_sn_right" default="" />
-  <!-- Determine Rizon types based on platform_type -->
-  <xacro:if value="${'$(arg platform_type)' == 'X1'}">
+  <!-- Determine Rizon left and right types based on rizon_type -->
+  <xacro:if value="${'$(arg rizon_type)' == 'Rizon4'}">
     <xacro:property name="rizon_type_left" value="Rizon4" />
     <xacro:property name="rizon_type_right" value="Rizon4R" />
+    <xacro:property name="external_axis_type" value="aico2_4_v2" />
   </xacro:if>
-  <xacro:if value="${'$(arg platform_type)' == 'X2'}">
+  <xacro:if value="${'$(arg rizon_type)' == 'Rizon10'}">
     <xacro:property name="rizon_type_left" value="Rizon10" />
     <xacro:property name="rizon_type_right" value="Rizon10" />
+    <xacro:property name="external_axis_type" value="aico2_10_v1" />
   </xacro:if>
   <xacro:arg name="load_gripper_left" default="false" />
@@ -28,6 +30,6 @@
   <xacro:arg name="initial_positions_file_right"
     default="$(find flexiv_description)/config/right_initial_positions.yaml" />
-  <xacro:include filename="$(find flexiv_description)/urdf/common/aico2_platform_x1.xacro" />
-  <xacro:include filename="$(find flexiv_description)/urdf/common/aico2_platform_x2.xacro" />
+  <xacro:include filename="$(find flexiv_description)/urdf/common/aico2_4_v2.xacro" />
+  <xacro:include filename="$(find flexiv_description)/urdf/common/aico2_10_v1.xacro" />
   <xacro:include filename="$(find flexiv_description)/urdf/common/rizon_robot.xacro" />
   <xacro:include filename="$(find flexiv_description)/urdf/common/rizon_dual.ros2_control.xacro" />
@@ -40,8 +42,8 @@
   <xacro:property name="calculated_right_arm_prefix"
     value="${(right_arm_prefix_arg + '_' + '$(arg robot_sn_right)' + '_') if right_arm_prefix_arg != '' and '$(arg robot_sn_right)' != '' else (right_arm_prefix_arg + '$(arg robot_sn_right)' + '_') if (right_arm_prefix_arg + '$(arg robot_sn_right)') != '' else ''}" />
-  <!-- Instantiate Platform -->
+  <!-- Instantiate External Axis -->
   <link name="world" />
-  <xacro:if value="${'$(arg platform_type)' == 'X1'}">
-    <xacro:aico2_platform_x1 prefix="$(arg platform_prefix)"
+  <xacro:if value="${'$(arg rizon_type)' == 'Rizon4'}">
+    <xacro:aico2_4_v2 prefix="$(arg external_axis_prefix)"
       left_arm_prefix="${calculated_left_arm_prefix}"
       right_arm_prefix="${calculated_right_arm_prefix}"
@@ -49,10 +51,10 @@
     <joint name="world_to_platform" type="fixed">
       <parent link="world" />
-      <child link="$(arg platform_prefix)aico2_x1_base_link" />
+      <child link="$(arg external_axis_prefix)aico2_4_v2_base_link" />
       <origin xyz="0 0 0" rpy="0 0 0" />
     </joint>
   </xacro:if>
-  <xacro:if value="${'$(arg platform_type)' == 'X2'}">
-    <xacro:aico2_platform_x2 prefix="$(arg platform_prefix)"
+  <xacro:if value="${'$(arg rizon_type)' == 'Rizon10'}">
+    <xacro:aico2_4_v2 prefix="$(arg external_axis_prefix)"
       left_arm_prefix="${calculated_left_arm_prefix}"
       right_arm_prefix="${calculated_right_arm_prefix}"
@@ -60,5 +62,5 @@
     <joint name="world_to_platform" type="fixed">
       <parent link="world" />
-      <child link="$(arg platform_prefix)aico2_x2_base_link" />
+      <child link="$(arg external_axis_prefix)aico2_4_v2_base_link" />
       <origin xyz="0 0 0" rpy="0 0 0" />
     </joint>
@@ -114,7 +116,6 @@
       translation_right_y="0"
       translation_right_z="0"
-      platform_name="aico2"
-      platform_type="$(arg platform_type)"
-      platform_prefix="$(arg platform_prefix)"
+      external_axis_type="${external_axis_type}"
+      external_axis_prefix="$(arg external_axis_prefix)"
     />
   </xacro:if>

File: urdf/common/aico2_4_v2.xacro (robot description, xacro)
@@ -1,33 +1,33 @@
 <?xml version="1.0" encoding="utf-8"?>
 <robot xmlns:xacro="http://wiki.ros.org/xacro">
-  <xacro:macro name="aico2_4_v1"
+  <xacro:macro name="aico2_4_v2"
     params="prefix left_arm_prefix right_arm_prefix mesh_prefix_path">
-    <joint name="${prefix}aico2_4_v1_joint1" type="revolute">
+    <joint name="${prefix}aico2_4_v2_joint1" type="revolute">
       <origin xyz="0 0 0.307" rpy="0 0 0" />
-      <parent link="${prefix}aico2_4_v1_base_link" />
-      <child link="${prefix}aico2_4_v1_link1" />
+      <parent link="${prefix}aico2_4_v2_base_link" />
+      <child link="${prefix}aico2_4_v2_link1" />
       <axis xyz="0 0 1" />
       <limit lower="-1.57" upper="1.57" effort="400" velocity="1.05" />
     </joint>
-    <joint name="${prefix}aico2_4_v1_joint2" type="revolute">
+    <joint name="${prefix}aico2_4_v2_joint2" type="revolute">
       <origin xyz="0.025 0 0" rpy="0 0 0" />
-      <parent link="${prefix}aico2_4_v1_link1" />
-      <child link="${prefix}aico2_4_v1_link2" />
+      <parent link="${prefix}aico2_4_v2_link1" />
+      <child link="${prefix}aico2_4_v2_link2" />
       <axis xyz="0 1 0" />
       <limit lower="0" upper="1.57" effort="365" velocity="1" />
     </joint>
-    <joint name="${prefix}aico2_4_v1_left_arm_adapter" type="fixed">
+    <joint name="${prefix}aico2_4_v2_left_arm_adapter" type="fixed">
       <origin xyz="0 -0.035 0.2885" rpy="-1.5708 0 0" />
-      <parent link="${prefix}aico2_4_v1_link2" />
+      <parent link="${prefix}aico2_4_v2_link2" />
       <child link="${left_arm_prefix}base_link" />
       <axis xyz="0 0 0" />
     </joint>
-    <joint name="${prefix}aico2_4_v1_right_arm_adapter" type="fixed">
+    <joint name="${prefix}aico2_4_v2_right_arm_adapter" type="fixed">
       <origin xyz="0 0.035 0.2885" rpy="1.5708 0 0" />
-      <parent link="${prefix}aico2_4_v1_link2" />
+      <parent link="${prefix}aico2_4_v2_link2" />
       <child link="${right_arm_prefix}base_link" />
       <axis xyz="0 0 0" />
     </joint>
-    <link name="${prefix}aico2_4_v1_base_link">
+    <link name="${prefix}aico2_4_v2_base_link">
       <inertial>
         <origin xyz="0.0052 -0.0154 0.258" rpy="0 0 0" />
@@ -38,5 +38,5 @@
         <origin xyz="0 0 0" rpy="0 0 1.5708" />
         <geometry>
-          <mesh filename="${mesh_prefix_path}meshes/AICO2-4-V1/visual/base_link.obj"
+          <mesh filename="${mesh_prefix_path}meshes/AICO2-4-V2/visual/base_link.obj"
             scale="0.001 0.001 0.001" />
         </geometry>
@@ -48,9 +48,9 @@
         <origin xyz="0 0 0" rpy="0 0 0" />
         <geometry>
-          <mesh filename="${mesh_prefix_path}meshes/AICO2-4-V1/collision/base_link.stl" />
+          <mesh filename="${mesh_prefix_path}meshes/AICO2-4-V2/collision/base_link.stl" />
         </geometry>
       </collision>
     </link>
-    <link name="${prefix}aico2_4_v1_link1">
+    <link name="${prefix}aico2_4_v2_link1">
       <inertial>
         <origin xyz="0.0484 -6.38E-05 -0.134" rpy="0 0 0" />
@@ -61,5 +61,5 @@
         <origin xyz="0 0 0" rpy="0 0 1.5708" />
         <geometry>
-          <mesh filename="${mesh_prefix_path}meshes/AICO2-4-V1/visual/link1.obj" />
+          <mesh filename="${mesh_prefix_path}meshes/AICO2-4-V2/visual/link1.obj" />
         </geometry>
         <material name="">
@@ -70,9 +70,9 @@
         <origin xyz="0 0 0" rpy="0 0 0" />
         <geometry>
-          <mesh filename="${mesh_prefix_path}meshes/AICO2-4-V1/collision/link1.stl" />
+          <mesh filename="${mesh_prefix_path}meshes/AICO2-4-V2/collision/link1.stl" />
         </geometry>
       </collision>
     </link>
-    <link name="${prefix}aico2_4_v1_link2">
+    <link name="${prefix}aico2_4_v2_link2">
       <inertial>
         <origin xyz="-0.0155 0.00056 0.25" rpy="0 0 0" />
@@ -83,5 +83,5 @@
         <origin xyz="0 0 0" rpy="0 0 1.5708" />
         <geometry>
-          <mesh filename="${mesh_prefix_path}meshes/AICO2-4-V1/visual/link2.obj" />
+          <mesh filename="${mesh_prefix_path}meshes/AICO2-4-V2/visual/link2.obj" />
         </geometry>
         <material name="">
@@ -92,5 +92,5 @@
         <origin xyz="0 0 0" rpy="0 0 0" />
         <geometry>
-          <mesh filename="${mesh_prefix_path}meshes/AICO2-4-V1/collision/link2.stl" />
+          <mesh filename="${mesh_prefix_path}meshes/AICO2-4-V2/collision/link2.stl" />
         </geometry>
       </collision>

File: urdf/common/rizon.ros2_control.xacro (robot description, xacro)
@@ -9,7 +9,6 @@
     fake_sensor_commands:=false
     initial_positions_file
-    platform_name:=''
-    platform_type:=''
-    platform_prefix:=''
+    external_axis_type:=''
+    external_axis_prefix:=''
     ">
     <xacro:property name="initial_positions" value="${xacro.load_yaml(initial_positions_file)['initial_positions']}"/>
@@ -98,50 +97,48 @@
         <state_interface name="effort" />
       </joint>
-      <!-- Platform joints -->
-      <xacro:if value="${platform_name == 'aico1'}">
-        <xacro:if value="${platform_type == 'X1'}">
-          <joint name="${platform_prefix}aico1_x1_joint2">
-            <command_interface name="position" />
-            <command_interface name="velocity" />
-            <command_interface name="effort" />
-            <state_interface name="position">
-              <param name="initial_value">0.0</param>
-            </state_interface>
-            <state_interface name="velocity" />
-            <state_interface name="effort" />
-          </joint>
-        </xacro:if>
-        <xacro:if value="${platform_type == 'X2'}">
-          <joint name="${platform_prefix}aico1_x2_joint1">
-            <command_interface name="position" />
-            <command_interface name="velocity" />
-            <command_interface name="effort" />
-            <state_interface name="position">
-              <param name="initial_value">0.0</param>
-            </state_interface>
-            <state_interface name="velocity" />
-            <state_interface name="effort" />
-          </joint>
-          <joint name="${platform_prefix}aico1_x2_joint2">
-            <command_interface name="position" />
-            <command_interface name="velocity" />
-            <command_interface name="effort" />
-            <state_interface name="position">
-              <param name="initial_value">0.0</param>
-            </state_interface>
-            <state_interface name="velocity" />
-            <state_interface name="effort" />
-          </joint>
-          <joint name="${platform_prefix}aico1_x2_joint_head">
-            <command_interface name="position" />
-            <command_interface name="velocity" />
-            <command_interface name="effort" />
-            <state_interface name="position">
-              <param name="initial_value">0.0</param>
-            </state_interface>
-            <state_interface name="velocity" />
-            <state_interface name="effort" />
-          </joint>
-        </xacro:if>
+      <!-- External axis joints -->
+      <xacro:if value="${external_axis_type == 'aico1_4_v1'}">
+        <joint name="${external_axis_prefix}aico1_4_v1_joint2">
+          <command_interface name="position" />
+          <command_interface name="velocity" />
+          <command_interface name="effort" />
+          <state_interface name="position">
+            <param name="initial_value">0.0</param>
+          </state_interface>
+          <state_interface name="velocity" />
+          <state_interface name="effort" />
+        </joint>
+      </xacro:if>
+      <xacro:if value="${external_axis_type == 'aico1_4_v2'}">
+        <joint name="${external_axis_prefix}aico1_4_v2_joint1">
+          <command_interface name="position" />
+          <command_interface name="velocity" />
+          <command_interface name="effort" />
+          <state_interface name="position">
+            <param name="initial_value">0.0</param>
+          </state_interface>
+          <state_interface name="velocity" />
+          <state_interface name="effort" />
+        </joint>
+        <joint name="${external_axis_prefix}aico1_4_v2_joint2">
+          <command_interface name="position" />
+          <command_interface name="velocity" />
+          <command_interface name="effort" />
+          <state_interface name="position">
+            <param name="initial_value">0.0</param>
+          </state_interface>
+          <state_interface name="velocity" />
+          <state_interface name="effort" />
+        </joint>
+        <joint name="${external_axis_prefix}aico1_4_v2_joint_head">
+          <command_interface name="position" />
+          <command_interface name="velocity" />
+          <command_interface name="effort" />
+          <state_interface name="position">
+            <param name="initial_value">0.0</param>
+          </state_interface>
+          <state_interface name="velocity" />
+          <state_interface name="effort" />
+        </joint>
       </xacro:if>
       <!-- 18 digital IO ports (16 on control box + 2 inside the wrist connector) -->

File: urdf/common/rizon_dual.ros2_control.xacro (robot description, xacro)
@@ -18,7 +18,6 @@
     translation_right_y:=0.0
     translation_right_z:=0.0
-    platform_name:=''
-    platform_type:=''
-    platform_prefix:=''
+    external_axis_type:=''
+    external_axis_prefix:=''
     ">
     <xacro:property name="initial_positions_left" value="${xacro.load_yaml(initial_positions_file_left)['initial_positions']}"/>
@@ -65,50 +64,48 @@
       <xacro:configure_joint joint_name="${prefix_left}joint6" initial_pos="${initial_positions_left['joint6']}" />
       <xacro:configure_joint joint_name="${prefix_left}joint7" initial_pos="${initial_positions_left['joint7']}" />
-      <!-- Platform joints -->
-      <xacro:if value="${platform_name == 'aico2'}">
-        <xacro:if value="${platform_type == 'X1'}">
-          <joint name="${platform_prefix}aico2_x1_joint1">
-            <command_interface name="position" />
-            <command_interface name="velocity" />
-            <command_interface name="effort" />
-            <state_interface name="position">
-              <param name="initial_value">0.0</param>
-            </state_interface>
-            <state_interface name="velocity" />
-            <state_interface name="effort" />
-          </joint>
-          <joint name="${platform_prefix}aico2_x1_joint2">
-            <command_interface name="position" />
-            <command_interface name="velocity" />
-            <command_interface name="effort" />
-            <state_interface name="position">
-              <param name="initial_value">0.0</param>
-            </state_interface>
-            <state_interface name="velocity" />
-            <state_interface name="effort" />
-          </joint>
-        </xacro:if>
-        <xacro:if value="${platform_type == 'X2'}">
-          <joint name="${platform_prefix}aico2_x2_joint1">
-            <command_interface name="position" />
-            <command_interface name="velocity" />
-            <command_interface name="effort" />
-            <state_interface name="position">
-              <param name="initial_value">0.0</param>
-            </state_interface>
-            <state_interface name="velocity" />
-            <state_interface name="effort" />
-          </joint>
-          <joint name="${platform_prefix}aico2_x2_joint2">
-            <command_interface name="position" />
-            <command_interface name="velocity" />
-            <command_interface name="effort" />
-            <state_interface name="position">
-              <param name="initial_value">0.0</param>
-            </state_interface>
-            <state_interface name="velocity" />
-            <state_interface name="effort" />
-          </joint>
-        </xacro:if>
+      <!-- External axis joints -->
+      <xacro:if value="${external_axis_type == 'aico2_4_v2'}">
+        <joint name="${external_axis_prefix}aico2_4_v2_joint1">
+          <command_interface name="position" />
+          <command_interface name="velocity" />
+          <command_interface name="effort" />
+          <state_interface name="position">
+            <param name="initial_value">0.0</param>
+          </state_interface>
+          <state_interface name="velocity" />
+          <state_interface name="effort" />
+        </joint>
+        <joint name="${external_axis_prefix}aico2_4_v2_joint2">
+          <command_interface name="position" />
+          <command_interface name="velocity" />
+          <command_interface name="effort" />
+          <state_interface name="position">
+            <param name="initial_value">0.0</param>
+          </state_interface>
+          <state_interface name="velocity" />
+          <state_interface name="effort" />
+        </joint>
+      </xacro:if>
+      <xacro:if value="${external_axis_type == 'aico2_10_v1'}">
+        <joint name="${external_axis_prefix}aico2_10_v1_joint1">
+          <command_interface name="position" />
+          <command_interface name="velocity" />
+          <command_interface name="effort" />
+          <state_interface name="position">
+            <param name="initial_value">0.0</param>
+          </state_interface>
+          <state_interface name="velocity" />
+          <state_interface name="effort" />
+        </joint>
+        <joint name="${external_axis_prefix}aico2_10_v1_joint2">
+          <command_interface name="position" />
+          <command_interface name="velocity" />
+          <command_interface name="effort" />
+          <state_interface name="position">
+            <param name="initial_value">0.0</param>
+          </state_interface>
+          <state_interface name="velocity" />
+          <state_interface name="effort" />
+        </joint>
       </xacro:if>
       <xacro:configure_joint joint_name="${prefix_right}joint1" initial_pos="${initial_positions_right['joint1']}" />

File: urdf/common/rizon_robot.xacro (robot description, xacro)
@@ -22,7 +22,6 @@
     base_xyz:='0.0 0.0 0.0'
     base_rpy:='0.0 0.0 0.0'
-    platform_name:=''
-    platform_type:=''
-    platform_prefix:=''
+    external_axis_type:=''
+    external_axis_prefix:=''
     ">
     <!-- Prefix defaults to 'arm_prefix_robot_sn' -->
@@ -58,7 +57,6 @@
         fake_sensor_commands="${fake_sensor_commands}"
         initial_positions_file="${initial_positions_file}"
-        platform_name="${platform_name}"
-        platform_type="${platform_type}"
-        platform_prefix="${platform_prefix}"
+        external_axis_type="${external_axis_type}"
+        external_axis_prefix="${external_axis_prefix}"
       />
     </xacro:if>

Commit message: Enhance AICO launch and URDF files: normalize external_axis_type and update AICO1 joint link

File: urdf/aico1.urdf.xacro (robot description, xacro)
@@ -42,5 +42,5 @@
     <joint name="world_to_platform" type="fixed">
       <parent link="world" />
-      <child link="$(arg external_axis_prefix)aico1_4_v2_base_link" />
+      <child link="$(arg external_axis_prefix)aico1_4_v2_agv" />
       <origin xyz="0 0 0" rpy="0 0 0" />
     </joint>
