Commit message: Update xacro argument to external_axis_type

File: urdf/aico1.urdf.xacro (robot description, xacro)
@@ -2,6 +2,6 @@
 <robot xmlns:xacro="http://www.ros.org/wiki/xacro" name="aico1">
   <!-- Parameters -->
-  <xacro:arg name="platform_type" default="X1" />
-  <xacro:arg name="platform_prefix" default="" />
+  <xacro:arg name="external_axis_type" default="aico1_platform_x1" />
+  <xacro:arg name="external_axis_prefix" default="" />
   <xacro:arg name="arm_prefix" default="" />
   <xacro:arg name="robot_sn" default="" />
@@ -17,6 +17,6 @@
     default="$(find flexiv_description)/config/initial_positions.yaml" />
   <!-- Validate rizon_type -->
-  <xacro:if value="${'$(arg rizon_type)' != 'Rizon4' and '$(arg rizon_type)' != 'Rizon4s'}">
-    ${xacro.warning('AICO1 only supports Rizon4 and Rizon4s. You selected $(arg rizon_type).')}
+  <xacro:if value="${'$(arg rizon_type)' != 'Rizon4' and '$(arg rizon_type)' != 'Rizon4s' and '$(arg rizon_type)' != 'Rizon4R'}">
+    ${xacro.warning('AICO1 only supports Rizon4, Rizon4s and Rizon4R. You selected $(arg rizon_type).')}
   </xacro:if>
   <xacro:include filename="$(find flexiv_description)/urdf/common/aico1_platform_x1.xacro" />
@@ -26,21 +26,21 @@
   <xacro:property name="calculated_arm_prefix"
     value="${('$(arg arm_prefix)' + '_' + '$(arg robot_sn)' + '_') if '$(arg arm_prefix)' != '' and '$(arg robot_sn)' != '' else ('$(arg arm_prefix)' + '$(arg robot_sn)' + '_') if ('$(arg arm_prefix)' + '$(arg robot_sn)') != '' else ''}" />
-  <!-- Instantiate Platform -->
+  <!-- Instantiate External Axis -->
   <link name="world" />
-  <xacro:if value="${'$(arg platform_type)' == 'X1'}">
-    <xacro:aico1_platform_x1 prefix="$(arg platform_prefix)" arm_prefix="${calculated_arm_prefix}"
+  <xacro:if value="${'$(arg external_axis_type)' == 'aico1_platform_x1'}">
+    <xacro:aico1_platform_x1 prefix="$(arg external_axis_prefix)" arm_prefix="${calculated_arm_prefix}"
       mesh_prefix_path="package://flexiv_description/" />
     <joint name="world_to_platform" type="fixed">
       <parent link="world" />
-      <child link="$(arg platform_prefix)aico1_x1_base_link" />
+      <child link="$(arg external_axis_prefix)aico1_x1_base_link" />
       <origin xyz="0 0 0" rpy="0 0 0" />
     </joint>
   </xacro:if>
-  <xacro:if value="${'$(arg platform_type)' == 'X2'}">
-    <xacro:aico1_platform_x2 prefix="$(arg platform_prefix)" arm_prefix="${calculated_arm_prefix}"
+  <xacro:if value="${'$(arg external_axis_type)' == 'aico1_platform_x2'}">
+    <xacro:aico1_platform_x2 prefix="$(arg external_axis_prefix)" arm_prefix="${calculated_arm_prefix}"
       mesh_prefix_path="package://flexiv_description/" />
     <joint name="world_to_platform" type="fixed">
       <parent link="world" />
-      <child link="$(arg platform_prefix)aico1_x2_agv" />
+      <child link="$(arg external_axis_prefix)aico1_x2_agv" />
       <origin xyz="0 0 0" rpy="0 0 0" />
     </joint>
@@ -65,7 +65,6 @@
     add_world_link="false"
     create_base_joint="false"
-    platform_name="aico1"
-    platform_type="$(arg platform_type)"
-    platform_prefix="$(arg platform_prefix)"
+    external_axis_type="$(arg external_axis_type)"
+    external_axis_prefix="$(arg external_axis_prefix)"
   />
 </robot>

File: urdf/aico2.urdf.xacro (robot description, xacro)
@@ -1,16 +1,23 @@
 <?xml version="1.0" encoding="utf-8"?>
 <robot xmlns:xacro="http://www.ros.org/wiki/xacro" name="aico2">
-  <xacro:arg name="platform_type" default="X1" />
-  <xacro:arg name="platform_prefix" default="" />
+  <xacro:arg name="external_axis_type" default="aico2_platform_x1" />
+  <xacro:arg name="external_axis_prefix" default="" />
+  <xacro:arg name="rizon_type" default="Rizon4" />
   <xacro:arg name="robot_sn_left" default="" />
   <xacro:arg name="robot_sn_right" default="" />
-  <!-- Determine Rizon types based on platform_type -->
-  <xacro:if value="${'$(arg platform_type)' == 'X1'}">
+  <!-- Determine Rizon left and right types based on rizon_type -->
+  <xacro:if value="${'$(arg rizon_type)' == 'Rizon4'}">
     <xacro:property name="rizon_type_left" value="Rizon4" />
     <xacro:property name="rizon_type_right" value="Rizon4R" />
+    <xacro:if value="${'$(arg external_axis_type)' != 'aico2_platform_x1'}">
+      ${xacro.warning('AICO2 with Rizon4 configuration only supports aico2_platform_x1 external axis. You selected $(arg external_axis_type).')}
+    </xacro:if>
   </xacro:if>
-  <xacro:if value="${'$(arg platform_type)' == 'X2'}">
+  <xacro:if value="${'$(arg rizon_type)' == 'Rizon10'}">
     <xacro:property name="rizon_type_left" value="Rizon10" />
     <xacro:property name="rizon_type_right" value="Rizon10" />
+    <xacro:if value="${'$(arg external_axis_type)' != 'aico2_platform_x2'}">
+      ${xacro.warning('AICO2 with Rizon10 configuration only supports aico2_platform_x2 external axis. You selected $(arg external_axis_type).')}
+    </xacro:if>
   </xacro:if>
   <xacro:arg name="load_gripper_left" default="false" />
@@ -40,8 +47,8 @@
   <xacro:property name="calculated_right_arm_prefix"
     value="${(right_arm_prefix_arg + '_' + '$(arg robot_sn_right)' + '_') if right_arm_prefix_arg != '' and '$(arg robot_sn_right)' != '' else (right_arm_prefix_arg + '$(arg robot_sn_right)' + '_') if (right_arm_prefix_arg + '$(arg robot_sn_right)') != '' else ''}" />
-  <!-- Instantiate Platform -->
+  <!-- Instantiate External Axis -->
   <link name="world" />
-  <xacro:if value="${'$(arg platform_type)' == 'X1'}">
-    <xacro:aico2_platform_x1 prefix="$(arg platform_prefix)"
+  <xacro:if value="${'$(arg external_axis_type)' == 'aico2_platform_x1'}">
+    <xacro:aico2_platform_x1 prefix="$(arg external_axis_prefix)"
       left_arm_prefix="${calculated_left_arm_prefix}"
       right_arm_prefix="${calculated_right_arm_prefix}"
@@ -49,10 +56,10 @@
     <joint name="world_to_platform" type="fixed">
       <parent link="world" />
-      <child link="$(arg platform_prefix)aico2_x1_base_link" />
+      <child link="$(arg external_axis_prefix)aico2_x1_base_link" />
       <origin xyz="0 0 0" rpy="0 0 0" />
     </joint>
   </xacro:if>
-  <xacro:if value="${'$(arg platform_type)' == 'X2'}">
-    <xacro:aico2_platform_x2 prefix="$(arg platform_prefix)"
+  <xacro:if value="${'$(arg external_axis_type)' == 'aico2_platform_x2'}">
+    <xacro:aico2_platform_x2 prefix="$(arg external_axis_prefix)"
       left_arm_prefix="${calculated_left_arm_prefix}"
       right_arm_prefix="${calculated_right_arm_prefix}"
@@ -60,5 +67,5 @@
     <joint name="world_to_platform" type="fixed">
       <parent link="world" />
-      <child link="$(arg platform_prefix)aico2_x2_base_link" />
+      <child link="$(arg external_axis_prefix)aico2_x2_base_link" />
       <origin xyz="0 0 0" rpy="0 0 0" />
     </joint>
@@ -114,7 +121,6 @@
       translation_right_y="0"
       translation_right_z="0"
-      platform_name="aico2"
-      platform_type="$(arg platform_type)"
-      platform_prefix="$(arg platform_prefix)"
+      external_axis_type="$(arg external_axis_type)"
+      external_axis_prefix="$(arg external_axis_prefix)"
     />
   </xacro:if>

File: urdf/common/rizon.ros2_control.xacro (robot description, xacro)
@@ -9,7 +9,6 @@
     fake_sensor_commands:=false
     initial_positions_file
-    platform_name:=''
-    platform_type:=''
-    platform_prefix:=''
+    external_axis_type:=''
+    external_axis_prefix:=''
     ">
     <xacro:property name="initial_positions" value="${xacro.load_yaml(initial_positions_file)['initial_positions']}"/>
@@ -98,50 +97,48 @@
         <state_interface name="effort" />
       </joint>
-      <!-- Platform joints -->
-      <xacro:if value="${platform_name == 'aico1'}">
-        <xacro:if value="${platform_type == 'X1'}">
-          <joint name="${platform_prefix}aico1_x1_joint2">
-            <command_interface name="position" />
-            <command_interface name="velocity" />
-            <command_interface name="effort" />
-            <state_interface name="position">
-              <param name="initial_value">0.0</param>
-            </state_interface>
-            <state_interface name="velocity" />
-            <state_interface name="effort" />
-          </joint>
-        </xacro:if>
-        <xacro:if value="${platform_type == 'X2'}">
-          <joint name="${platform_prefix}aico1_x2_joint1">
-            <command_interface name="position" />
-            <command_interface name="velocity" />
-            <command_interface name="effort" />
-            <state_interface name="position">
-              <param name="initial_value">0.0</param>
-            </state_interface>
-            <state_interface name="velocity" />
-            <state_interface name="effort" />
-          </joint>
-          <joint name="${platform_prefix}aico1_x2_joint2">
-            <command_interface name="position" />
-            <command_interface name="velocity" />
-            <command_interface name="effort" />
-            <state_interface name="position">
-              <param name="initial_value">0.0</param>
-            </state_interface>
-            <state_interface name="velocity" />
-            <state_interface name="effort" />
-          </joint>
-          <joint name="${platform_prefix}aico1_x2_joint_head">
-            <command_interface name="position" />
-            <command_interface name="velocity" />
-            <command_interface name="effort" />
-            <state_interface name="position">
-              <param name="initial_value">0.0</param>
-            </state_interface>
-            <state_interface name="velocity" />
-            <state_interface name="effort" />
-          </joint>
-        </xacro:if>
+      <!-- External axis joints -->
+      <xacro:if value="${external_axis_type == 'aico1_platform_x1'}">
+        <joint name="${external_axis_prefix}aico1_x1_joint2">
+          <command_interface name="position" />
+          <command_interface name="velocity" />
+          <command_interface name="effort" />
+          <state_interface name="position">
+            <param name="initial_value">0.0</param>
+          </state_interface>
+          <state_interface name="velocity" />
+          <state_interface name="effort" />
+        </joint>
+      </xacro:if>
+      <xacro:if value="${external_axis_type == 'aico1_platform_x2'}">
+        <joint name="${external_axis_prefix}aico1_x2_joint1">
+          <command_interface name="position" />
+          <command_interface name="velocity" />
+          <command_interface name="effort" />
+          <state_interface name="position">
+            <param name="initial_value">0.0</param>
+          </state_interface>
+          <state_interface name="velocity" />
+          <state_interface name="effort" />
+        </joint>
+        <joint name="${external_axis_prefix}aico1_x2_joint2">
+          <command_interface name="position" />
+          <command_interface name="velocity" />
+          <command_interface name="effort" />
+          <state_interface name="position">
+            <param name="initial_value">0.0</param>
+          </state_interface>
+          <state_interface name="velocity" />
+          <state_interface name="effort" />
+        </joint>
+        <joint name="${external_axis_prefix}aico1_x2_joint_head">
+          <command_interface name="position" />
+          <command_interface name="velocity" />
+          <command_interface name="effort" />
+          <state_interface name="position">
+            <param name="initial_value">0.0</param>
+          </state_interface>
+          <state_interface name="velocity" />
+          <state_interface name="effort" />
+        </joint>
       </xacro:if>
       <!-- 18 digital IO ports (16 on control box + 2 inside the wrist connector) -->

File: urdf/common/rizon_dual.ros2_control.xacro (robot description, xacro)
@@ -18,7 +18,6 @@
     translation_right_y:=0.0
     translation_right_z:=0.0
-    platform_name:=''
-    platform_type:=''
-    platform_prefix:=''
+    external_axis_type:=''
+    external_axis_prefix:=''
     ">
     <xacro:property name="initial_positions_left" value="${xacro.load_yaml(initial_positions_file_left)['initial_positions']}"/>
@@ -65,50 +64,48 @@
       <xacro:configure_joint joint_name="${prefix_left}joint6" initial_pos="${initial_positions_left['joint6']}" />
       <xacro:configure_joint joint_name="${prefix_left}joint7" initial_pos="${initial_positions_left['joint7']}" />
-      <!-- Platform joints -->
-      <xacro:if value="${platform_name == 'aico2'}">
-        <xacro:if value="${platform_type == 'X1'}">
-          <joint name="${platform_prefix}aico2_x1_joint1">
-            <command_interface name="position" />
-            <command_interface name="velocity" />
-            <command_interface name="effort" />
-            <state_interface name="position">
-              <param name="initial_value">0.0</param>
-            </state_interface>
-            <state_interface name="velocity" />
-            <state_interface name="effort" />
-          </joint>
-          <joint name="${platform_prefix}aico2_x1_joint2">
-            <command_interface name="position" />
-            <command_interface name="velocity" />
-            <command_interface name="effort" />
-            <state_interface name="position">
-              <param name="initial_value">0.0</param>
-            </state_interface>
-            <state_interface name="velocity" />
-            <state_interface name="effort" />
-          </joint>
-        </xacro:if>
-        <xacro:if value="${platform_type == 'X2'}">
-          <joint name="${platform_prefix}aico2_x2_joint1">
-            <command_interface name="position" />
-            <command_interface name="velocity" />
-            <command_interface name="effort" />
-            <state_interface name="position">
-              <param name="initial_value">0.0</param>
-            </state_interface>
-            <state_interface name="velocity" />
-            <state_interface name="effort" />
-          </joint>
-          <joint name="${platform_prefix}aico2_x2_joint2">
-            <command_interface name="position" />
-            <command_interface name="velocity" />
-            <command_interface name="effort" />
-            <state_interface name="position">
-              <param name="initial_value">0.0</param>
-            </state_interface>
-            <state_interface name="velocity" />
-            <state_interface name="effort" />
-          </joint>
-        </xacro:if>
+      <!-- External axis joints -->
+      <xacro:if value="${external_axis_type == 'aico2_platform_x1'}">
+        <joint name="${external_axis_prefix}aico2_x1_joint1">
+          <command_interface name="position" />
+          <command_interface name="velocity" />
+          <command_interface name="effort" />
+          <state_interface name="position">
+            <param name="initial_value">0.0</param>
+          </state_interface>
+          <state_interface name="velocity" />
+          <state_interface name="effort" />
+        </joint>
+        <joint name="${external_axis_prefix}aico2_x1_joint2">
+          <command_interface name="position" />
+          <command_interface name="velocity" />
+          <command_interface name="effort" />
+          <state_interface name="position">
+            <param name="initial_value">0.0</param>
+          </state_interface>
+          <state_interface name="velocity" />
+          <state_interface name="effort" />
+        </joint>
+      </xacro:if>
+      <xacro:if value="${external_axis_type == 'aico2_platform_x2'}">
+        <joint name="${external_axis_prefix}aico2_x2_joint1">
+          <command_interface name="position" />
+          <command_interface name="velocity" />
+          <command_interface name="effort" />
+          <state_interface name="position">
+            <param name="initial_value">0.0</param>
+          </state_interface>
+          <state_interface name="velocity" />
+          <state_interface name="effort" />
+        </joint>
+        <joint name="${external_axis_prefix}aico2_x2_joint2">
+          <command_interface name="position" />
+          <command_interface name="velocity" />
+          <command_interface name="effort" />
+          <state_interface name="position">
+            <param name="initial_value">0.0</param>
+          </state_interface>
+          <state_interface name="velocity" />
+          <state_interface name="effort" />
+        </joint>
       </xacro:if>
       <xacro:configure_joint joint_name="${prefix_right}joint1" initial_pos="${initial_positions_right['joint1']}" />
