Commit message: Update AICO robot configurations and URDF files for different AICO model names

File: urdf/aico1.urdf.xacro (robot description, xacro)
@@ -2,5 +2,5 @@
 <robot xmlns:xacro="http://www.ros.org/wiki/xacro" name="aico1">
   <!-- Parameters -->
-  <xacro:arg name="external_axis_type" default="aico1_platform_x1" />
+  <xacro:arg name="external_axis_type" default="aico1_4_v1" />
   <xacro:arg name="external_axis_prefix" default="" />
   <xacro:arg name="arm_prefix" default="" />
@@ -20,6 +20,6 @@
     ${xacro.warning('AICO1 only supports Rizon4, Rizon4s and Rizon4R. You selected $(arg rizon_type).')}
   </xacro:if>
-  <xacro:include filename="$(find flexiv_description)/urdf/common/aico1_platform_x1.xacro" />
-  <xacro:include filename="$(find flexiv_description)/urdf/common/aico1_platform_x2.xacro" />
+  <xacro:include filename="$(find flexiv_description)/urdf/common/aico1_4_v1.xacro" />
+  <xacro:include filename="$(find flexiv_description)/urdf/common/aico1_4_v2.xacro" />
   <xacro:include filename="$(find flexiv_description)/urdf/common/rizon_robot.xacro" />
   <!-- Calculate the actual prefix rizon_robot will use -->
@@ -28,19 +28,19 @@
   <!-- Instantiate External Axis -->
   <link name="world" />
-  <xacro:if value="${'$(arg external_axis_type)' == 'aico1_platform_x1'}">
-    <xacro:aico1_platform_x1 prefix="$(arg external_axis_prefix)" arm_prefix="${calculated_arm_prefix}"
+  <xacro:if value="${'$(arg external_axis_type)' == 'aico1_4_v1'}">
+    <xacro:aico1_4_v1 prefix="$(arg external_axis_prefix)" arm_prefix="${calculated_arm_prefix}"
       mesh_prefix_path="package://flexiv_description/" />
     <joint name="world_to_platform" type="fixed">
       <parent link="world" />
-      <child link="$(arg external_axis_prefix)aico1_x1_base_link" />
+      <child link="$(arg external_axis_prefix)aico1_4_v1_base_link" />
       <origin xyz="0 0 0" rpy="0 0 0" />
     </joint>
   </xacro:if>
-  <xacro:if value="${'$(arg external_axis_type)' == 'aico1_platform_x2'}">
-    <xacro:aico1_platform_x2 prefix="$(arg external_axis_prefix)" arm_prefix="${calculated_arm_prefix}"
+  <xacro:if value="${'$(arg external_axis_type)' == 'aico1_4_v2'}">
+    <xacro:aico1_4_v2 prefix="$(arg external_axis_prefix)" arm_prefix="${calculated_arm_prefix}"
       mesh_prefix_path="package://flexiv_description/" />
     <joint name="world_to_platform" type="fixed">
       <parent link="world" />
-      <child link="$(arg external_axis_prefix)aico1_x2_agv" />
+      <child link="$(arg external_axis_prefix)aico1_4_v2_agv" />
       <origin xyz="0 0 0" rpy="0 0 0" />
     </joint>

File: urdf/aico2.urdf.xacro (robot description, xacro)
@@ -1,5 +1,5 @@
 <?xml version="1.0" encoding="utf-8"?>
 <robot xmlns:xacro="http://www.ros.org/wiki/xacro" name="aico2">
-  <xacro:arg name="external_axis_type" default="aico2_platform_x1" />
+  <xacro:arg name="external_axis_type" default="aico2_4_v1" />
   <xacro:arg name="external_axis_prefix" default="" />
   <xacro:arg name="rizon_type" default="Rizon4" />
@@ -10,6 +10,6 @@
     <xacro:property name="rizon_type_left" value="Rizon4" />
     <xacro:property name="rizon_type_right" value="Rizon4R" />
-    <xacro:if value="${'$(arg external_axis_type)' != 'aico2_platform_x1'}">
-      ${xacro.warning('AICO2 with Rizon4 configuration only supports aico2_platform_x1 external axis. You selected $(arg external_axis_type).')}
+    <xacro:if value="${'$(arg external_axis_type)' != 'aico2_4_v1' and '$(arg external_axis_type)' != 'aico2_4_v2'}">
+      ${xacro.warning('AICO2 with Rizon4 configuration only supports AICO2-4-V1 or AICO2-4-V2 external axis. You selected $(arg external_axis_type).')}
     </xacro:if>
   </xacro:if>
@@ -17,6 +17,6 @@
     <xacro:property name="rizon_type_left" value="Rizon10" />
     <xacro:property name="rizon_type_right" value="Rizon10" />
-    <xacro:if value="${'$(arg external_axis_type)' != 'aico2_platform_x2'}">
-      ${xacro.warning('AICO2 with Rizon10 configuration only supports aico2_platform_x2 external axis. You selected $(arg external_axis_type).')}
+    <xacro:if value="${'$(arg external_axis_type)' != 'aico2_10_v1'}">
+      ${xacro.warning('AICO2 with Rizon10 configuration only supports AICO2-10-V1 external axis. You selected $(arg external_axis_type).')}
     </xacro:if>
   </xacro:if>
@@ -35,6 +35,6 @@
   <xacro:arg name="initial_positions_file_right"
     default="$(find flexiv_description)/config/right_initial_positions.yaml" />
-  <xacro:include filename="$(find flexiv_description)/urdf/common/aico2_platform_x1.xacro" />
-  <xacro:include filename="$(find flexiv_description)/urdf/common/aico2_platform_x2.xacro" />
+  <xacro:include filename="$(find flexiv_description)/urdf/common/aico2_4_v1.xacro" />
+  <xacro:include filename="$(find flexiv_description)/urdf/common/aico2_10_v1.xacro" />
   <xacro:include filename="$(find flexiv_description)/urdf/common/rizon_robot.xacro" />
   <xacro:include filename="$(find flexiv_description)/urdf/common/rizon_dual.ros2_control.xacro" />
@@ -49,6 +49,6 @@
   <!-- Instantiate External Axis -->
   <link name="world" />
-  <xacro:if value="${'$(arg external_axis_type)' == 'aico2_platform_x1'}">
-    <xacro:aico2_platform_x1 prefix="$(arg external_axis_prefix)"
+  <xacro:if value="${'$(arg external_axis_type)' == 'aico2_4_v1'}">
+    <xacro:aico2_4_v1 prefix="$(arg external_axis_prefix)"
       left_arm_prefix="${calculated_left_arm_prefix}"
       right_arm_prefix="${calculated_right_arm_prefix}"
@@ -56,10 +56,10 @@
     <joint name="world_to_platform" type="fixed">
       <parent link="world" />
-      <child link="$(arg external_axis_prefix)aico2_x1_base_link" />
+      <child link="$(arg external_axis_prefix)aico2_4_v1_base_link" />
       <origin xyz="0 0 0" rpy="0 0 0" />
     </joint>
   </xacro:if>
-  <xacro:if value="${'$(arg external_axis_type)' == 'aico2_platform_x2'}">
-    <xacro:aico2_platform_x2 prefix="$(arg external_axis_prefix)"
+  <xacro:if value="${'$(arg external_axis_type)' == 'aico2_10_v1'}">
+    <xacro:aico2_10_v1 prefix="$(arg external_axis_prefix)"
       left_arm_prefix="${calculated_left_arm_prefix}"
       right_arm_prefix="${calculated_right_arm_prefix}"
@@ -67,5 +67,5 @@
     <joint name="world_to_platform" type="fixed">
       <parent link="world" />
-      <child link="$(arg external_axis_prefix)aico2_x2_base_link" />
+      <child link="$(arg external_axis_prefix)aico2_10_v1_base_link" />
       <origin xyz="0 0 0" rpy="0 0 0" />
     </joint>

File: urdf/common/aico1_4_v1.xacro (robot description, xacro)
@@ -1,26 +1,26 @@
 <?xml version="1.0" encoding="utf-8"?>
 <robot xmlns:xacro="http://wiki.ros.org/xacro">
-  <xacro:macro name="aico1_platform_x1" params="prefix arm_prefix mesh_prefix_path">
-    <joint name="${prefix}aico1_x1_joint1" type="fixed">
+  <xacro:macro name="aico1_4_v1" params="prefix arm_prefix mesh_prefix_path">
+    <joint name="${prefix}aico1_4_v1_joint1" type="fixed">
       <origin xyz="0 0 0.768" rpy="0 0 0" />
-      <parent link="${prefix}aico1_x1_base_link" />
-      <child link="${prefix}aico1_x1_link1" />
+      <parent link="${prefix}aico1_4_v1_base_link" />
+      <child link="${prefix}aico1_4_v1_link1" />
       <axis xyz="0 0 1" />
       <limit lower="0" upper="0.3" effort="100" velocity="1" />
     </joint>
-    <joint name="${prefix}aico1_x1_joint2" type="revolute">
+    <joint name="${prefix}aico1_4_v1_joint2" type="revolute">
       <origin xyz="0.1385 0.204 0.183" rpy="0 0 0" />
-      <parent link="${prefix}aico1_x1_link1" />
-      <child link="${prefix}aico1_x1_link2" />
+      <parent link="${prefix}aico1_4_v1_link1" />
+      <child link="${prefix}aico1_4_v1_link2" />
       <axis xyz="0 1 0" />
       <limit lower="0" upper="1.57" effort="365" velocity="1" />
     </joint>
-    <joint name="${prefix}aico1_x1_arm_adapter" type="fixed">
+    <joint name="${prefix}aico1_4_v1_arm_adapter" type="fixed">
       <origin xyz="0.0037763 0.0 0.3214" rpy="1.5708 0 0" />
-      <parent link="${prefix}aico1_x1_link2" />
+      <parent link="${prefix}aico1_4_v1_link2" />
       <child link="${arm_prefix}base_link" />
       <axis xyz="0 0 0" />
     </joint>
-    <link name="${prefix}aico1_x1_base_link">
+    <link name="${prefix}aico1_4_v1_base_link">
       <inertial>
         <origin xyz="0.00266 0.000754 0.34" rpy="0 0 0" />
@@ -32,5 +32,5 @@
         <geometry>
           <mesh
-            filename="${mesh_prefix_path}meshes/AICO1-X1/visual/base_link.obj" />
+            filename="${mesh_prefix_path}meshes/AICO1-4-V1/visual/base_link.obj" />
         </geometry>
         <material name="">
@@ -42,9 +42,9 @@
         <geometry>
           <mesh
-            filename="${mesh_prefix_path}meshes/AICO1-X1/collision/base_link.stl" />
+            filename="${mesh_prefix_path}meshes/AICO1-4-V1/collision/base_link.stl" />
         </geometry>
       </collision>
     </link>
-    <link name="${prefix}aico1_x1_link1">
+    <link name="${prefix}aico1_4_v1_link1">
       <inertial>
         <origin xyz="0.017 0.014 -0.075" rpy="0 0 0" />
@@ -56,5 +56,5 @@
         <geometry>
           <mesh
-            filename="${mesh_prefix_path}meshes/AICO1-X1/visual/rise_link.obj" />
+            filename="${mesh_prefix_path}meshes/AICO1-4-V1/visual/rise_link.obj" />
         </geometry>
         <material name="">
@@ -66,5 +66,5 @@
         <geometry>
           <mesh
-            filename="${mesh_prefix_path}meshes/AICO1-X1/collision/rise_link_bottom.stl" />
+            filename="${mesh_prefix_path}meshes/AICO1-4-V1/collision/rise_link_bottom.stl" />
         </geometry>
       </collision>
@@ -73,9 +73,9 @@
         <geometry>
           <mesh
-            filename="${mesh_prefix_path}meshes/AICO1-X1/collision/rise_link_top.stl" />
+            filename="${mesh_prefix_path}meshes/AICO1-4-V1/collision/rise_link_top.stl" />
         </geometry>
       </collision>
     </link>
-    <link name="${prefix}aico1_x1_link2">
+    <link name="${prefix}aico1_4_v1_link2">
       <inertial>
         <origin xyz="0.0303 -0.092 0.255" rpy="0 0 0" />
@@ -87,5 +87,5 @@
         <geometry>
           <mesh
-            filename="${mesh_prefix_path}meshes/AICO1-X1/visual/pitch_link.obj" />
+            filename="${mesh_prefix_path}meshes/AICO1-4-V1/visual/pitch_link.obj" />
         </geometry>
         <material name="">
@@ -97,5 +97,5 @@
         <geometry>
           <mesh
-            filename="${mesh_prefix_path}meshes/AICO1-X1/collision/pitch_link.stl" />
+            filename="${mesh_prefix_path}meshes/AICO1-4-V1/collision/pitch_link.stl" />
         </geometry>
       </collision>

File: urdf/common/aico1_4_v2.xacro (robot description, xacro)
@@ -1,39 +1,39 @@
 <?xml version="1.0" encoding="utf-8"?>
 <robot xmlns:xacro="http://wiki.ros.org/xacro">
-  <xacro:macro name="aico1_platform_x2" params="prefix arm_prefix mesh_prefix_path">
-    <joint name="${prefix}aico1_x2_base_to_agv" type="fixed">
+  <xacro:macro name="aico1_4_v2" params="prefix arm_prefix mesh_prefix_path">
+    <joint name="${prefix}aico1_4_v2_base_to_agv" type="fixed">
       <origin xyz="0.004 0.1255 0.695" rpy="0.0 0.0 0.0" />
-      <parent link="${prefix}aico1_x2_agv" />
-      <child link="${prefix}aico1_x2_base_link" />
+      <parent link="${prefix}aico1_4_v2_agv" />
+      <child link="${prefix}aico1_4_v2_base_link" />
       <axis xyz="0 0 0" />
     </joint>
-    <joint name="${prefix}aico1_x2_joint1" type="revolute">
+    <joint name="${prefix}aico1_4_v2_joint1" type="revolute">
       <origin xyz="-0.122 0.1066 0.164" rpy="0 0 0" />
-      <parent link="${prefix}aico1_x2_base_link" />
-      <child link="${prefix}aico1_x2_link1" />
+      <parent link="${prefix}aico1_4_v2_base_link" />
+      <child link="${prefix}aico1_4_v2_link1" />
       <axis xyz="0 1 0" />
       <limit lower="-0.523598775598" upper="1.57079632679" effort="1000"
         velocity="1" />
     </joint>
-    <joint name="${prefix}aico1_x2_joint2" type="revolute">
+    <joint name="${prefix}aico1_4_v2_joint2" type="revolute">
       <origin xyz="-0.005 -0.0991 0.47875" rpy="0 0 0" />
-      <parent link="${prefix}aico1_x2_link1" />
-      <child link="${prefix}aico1_x2_neck_link" />
+      <parent link="${prefix}aico1_4_v2_link1" />
+      <child link="${prefix}aico1_4_v2_neck_link" />
       <axis xyz="0 0 1" />
       <limit lower="-1.57079632679" upper="1.57079632679" effort="50" velocity="1" />
     </joint>
-    <joint name="${prefix}aico1_x2_joint_head" type="revolute">
+    <joint name="${prefix}aico1_4_v2_joint_head" type="revolute">
       <origin xyz="-0.025 0 0.088" rpy="0 0 0" />
-      <parent link="${prefix}aico1_x2_neck_link" />
-      <child link="${prefix}aico1_x2_head_link" />
+      <parent link="${prefix}aico1_4_v2_neck_link" />
+      <child link="${prefix}aico1_4_v2_head_link" />
       <axis xyz="0 1 0" />
       <limit lower="0" upper="0.436332312999" effort="80" velocity="1" />
     </joint>
-    <joint name="${prefix}aico1_x2_arm_adapter" type="fixed">
-      <parent link="${prefix}aico1_x2_link1" />
+    <joint name="${prefix}aico1_4_v2_arm_adapter" type="fixed">
+      <parent link="${prefix}aico1_4_v2_link1" />
       <child link="${arm_prefix}base_link" />
       <origin xyz="0.0 0.016 0.320" rpy="1.57079632679 0.0 0.0" />
     </joint>
-    <link name="${prefix}aico1_x2_agv">
+    <link name="${prefix}aico1_4_v2_agv">
       <inertial>
         <origin xyz="0 0 0" rpy="0 0 0" />
@@ -45,5 +45,5 @@
         <geometry>
           <mesh
-            filename="${mesh_prefix_path}meshes/AICO1-X2/visual/agv.obj" />
+            filename="${mesh_prefix_path}meshes/AICO1-4-V2/visual/agv.obj" />
         </geometry>
         <material name="">
@@ -55,9 +55,9 @@
         <geometry>
           <mesh
-            filename="${mesh_prefix_path}meshes/AICO1-X2/collision/agv.stl" />
+            filename="${mesh_prefix_path}meshes/AICO1-4-V2/collision/agv.stl" />
         </geometry>
       </collision>
     </link>
-    <link name="${prefix}aico1_x2_base_link">
+    <link name="${prefix}aico1_4_v2_base_link">
       <inertial>
         <origin xyz="-0.0372 -0.00251 0.0448" rpy="0 0 0" />
@@ -69,5 +69,5 @@
         <geometry>
           <mesh
-            filename="${mesh_prefix_path}meshes/AICO1-X2/visual/base_link.obj" />
+            filename="${mesh_prefix_path}meshes/AICO1-4-V2/visual/base_link.obj" />
         </geometry>
         <material name="">
@@ -79,9 +79,9 @@
         <geometry>
           <mesh
-            filename="${mesh_prefix_path}meshes/AICO1-X2/collision/base_link.stl" />
+            filename="${mesh_prefix_path}meshes/AICO1-4-V2/collision/base_link.stl" />
         </geometry>
       </collision>
     </link>
-    <link name="${prefix}aico1_x2_link1">
+    <link name="${prefix}aico1_4_v2_link1">
       <inertial>
         <origin xyz="-0.00141 -0.0922 0.106" rpy="0 0 0" />
@@ -93,5 +93,5 @@
         <geometry>
           <mesh
-            filename="${mesh_prefix_path}meshes/AICO1-X2/visual/link1.obj" />
+            filename="${mesh_prefix_path}meshes/AICO1-4-V2/visual/link1.obj" />
         </geometry>
         <material name="">
@@ -103,9 +103,9 @@
         <geometry>
           <mesh
-            filename="${mesh_prefix_path}meshes/AICO1-X2/collision/link1.stl" />
+            filename="${mesh_prefix_path}meshes/AICO1-4-V2/collision/link1.stl" />
         </geometry>
       </collision>
     </link>
-    <link name="${prefix}aico1_x2_neck_link">
+    <link name="${prefix}aico1_4_v2_neck_link">
       <inertial>
         <origin xyz="-0.0149 7E-07 0.0547" rpy="0 0 0" />
@@ -117,5 +117,5 @@
         <geometry>
           <mesh
-            filename="${mesh_prefix_path}meshes/AICO1-X2/visual/neck_link.obj" />
+            filename="${mesh_prefix_path}meshes/AICO1-4-V2/visual/neck_link.obj" />
         </geometry>
         <material name="">
@@ -127,9 +127,9 @@
         <geometry>
           <mesh
-            filename="${mesh_prefix_path}meshes/AICO1-X2/collision/neck_link.stl" />
+            filename="${mesh_prefix_path}meshes/AICO1-4-V2/collision/neck_link.stl" />
         </geometry>
       </collision>
     </link>
-    <link name="${prefix}aico1_x2_head_link">
+    <link name="${prefix}aico1_4_v2_head_link">
       <inertial>
         <origin xyz="0.017 0.000125 0.0594" rpy="0 0 0" />
@@ -141,5 +141,5 @@
         <geometry>
           <mesh
-            filename="${mesh_prefix_path}meshes/AICO1-X2/visual/head_link.obj" />
+            filename="${mesh_prefix_path}meshes/AICO1-4-V2/visual/head_link.obj" />
         </geometry>
         <material name="">
@@ -151,5 +151,5 @@
         <geometry>
           <mesh
-            filename="${mesh_prefix_path}meshes/AICO1-X2/collision/head_link.stl" />
+            filename="${mesh_prefix_path}meshes/AICO1-4-V2/collision/head_link.stl" />
         </geometry>
       </collision>

File: urdf/common/rizon.ros2_control.xacro (robot description, xacro)
@@ -98,6 +98,6 @@
       </joint>
       <!-- External axis joints -->
-      <xacro:if value="${external_axis_type == 'aico1_platform_x1'}">
-        <joint name="${external_axis_prefix}aico1_x1_joint2">
+      <xacro:if value="${external_axis_type == 'aico1_4_v1'}">
+        <joint name="${external_axis_prefix}aico1_4_v1_joint2">
           <command_interface name="position" />
           <command_interface name="velocity" />
@@ -110,6 +110,6 @@
         </joint>
       </xacro:if>
-      <xacro:if value="${external_axis_type == 'aico1_platform_x2'}">
-        <joint name="${external_axis_prefix}aico1_x2_joint1">
+      <xacro:if value="${external_axis_type == 'aico1_4_v2'}">
+        <joint name="${external_axis_prefix}aico1_4_v2_joint1">
           <command_interface name="position" />
           <command_interface name="velocity" />
@@ -121,5 +121,5 @@
           <state_interface name="effort" />
         </joint>
-        <joint name="${external_axis_prefix}aico1_x2_joint2">
+        <joint name="${external_axis_prefix}aico1_4_v2_joint2">
           <command_interface name="position" />
           <command_interface name="velocity" />
@@ -131,5 +131,5 @@
           <state_interface name="effort" />
         </joint>
-        <joint name="${external_axis_prefix}aico1_x2_joint_head">
+        <joint name="${external_axis_prefix}aico1_4_v2_joint_head">
           <command_interface name="position" />
           <command_interface name="velocity" />

File: urdf/common/rizon_dual.ros2_control.xacro (robot description, xacro)
@@ -66,6 +66,6 @@
       <xacro:configure_joint joint_name="${prefix_left}joint7" initial_pos="${initial_positions_left['joint7']}" />
       <!-- External axis joints -->
-      <xacro:if value="${external_axis_type == 'aico2_platform_x1'}">
-        <joint name="${external_axis_prefix}aico2_x1_joint1">
+      <xacro:if value="${external_axis_type == 'aico2_4_v1'}">
+        <joint name="${external_axis_prefix}aico2_4_v1_joint1">
           <command_interface name="position" />
           <command_interface name="velocity" />
@@ -77,5 +77,5 @@
           <state_interface name="effort" />
         </joint>
-        <joint name="${external_axis_prefix}aico2_x1_joint2">
+        <joint name="${external_axis_prefix}aico2_4_v1_joint2">
           <command_interface name="position" />
           <command_interface name="velocity" />
@@ -88,6 +88,6 @@
         </joint>
       </xacro:if>
-      <xacro:if value="${external_axis_type == 'aico2_platform_x2'}">
-        <joint name="${external_axis_prefix}aico2_x2_joint1">
+      <xacro:if value="${external_axis_type == 'aico2_10_v1'}">
+        <joint name="${external_axis_prefix}aico2_10_v1_joint1">
           <command_interface name="position" />
           <command_interface name="velocity" />
@@ -99,5 +99,5 @@
           <state_interface name="effort" />
         </joint>
-        <joint name="${external_axis_prefix}aico2_x2_joint2">
+        <joint name="${external_axis_prefix}aico2_10_v1_joint2">
           <command_interface name="position" />
           <command_interface name="velocity" />

Commit message: Update AICO1-4-V2 meshes file and fix the correct reference link

File: urdf/aico1.urdf.xacro (robot description, xacro)
@@ -42,5 +42,5 @@
     <joint name="world_to_platform" type="fixed">
       <parent link="world" />
-      <child link="$(arg external_axis_prefix)aico1_4_v2_agv" />
+      <child link="$(arg external_axis_prefix)aico1_4_v2_base_link" />
       <origin xyz="0 0 0" rpy="0 0 0" />
     </joint>
