Commit message: Update kinematics params property names

File: urdf/flexiv.urdf.xacro (robot description, xacro)
@@ -83,5 +83,5 @@
   <xacro:if value="${is_single}">
     <xacro:property name="mounting" value="${xacro.load_yaml('$(arg mounting_file)')}" />
-    <xacro:property name="single_kin"
+    <xacro:property name="single_kinematics"
       value="${'$(arg kinematics_parameters_file)' if '$(arg kinematics_parameters_file)' != ''
                else cfg + '/' + robot_type_str + '/default_kinematics.yaml'}" />
@@ -90,5 +90,5 @@
       robot_sn="$(arg robot_sn)"
       joint_limits_parameters_file="$(arg joint_limits_parameters_file)"
-      kinematics_parameters_file="${single_kin}"
+      kinematics_parameters_file="${single_kinematics}"
       inertia_parameters_file="$(arg inertia_parameters_file)"
       visual_parameters_file="$(arg visual_parameters_file)"
@@ -209,5 +209,5 @@
         mesh_prefix_path="package://flexiv_description/" />
     </xacro:if>
-    <xacro:property name="aico1_kin"
+    <xacro:property name="aico1_kinematics"
       value="${'$(arg kinematics_parameters_file)' if '$(arg kinematics_parameters_file)' != ''
                else cfg + '/' + aico1_arm + '/default_kinematics.yaml'}" />
@@ -216,5 +216,5 @@
       robot_sn="$(arg robot_sn)"
       joint_limits_parameters_file="${cfg}/${aico1_arm}/joint_limits.yaml"
-      kinematics_parameters_file="${aico1_kin}"
+      kinematics_parameters_file="${aico1_kinematics}"
       inertia_parameters_file="${cfg}/${aico1_arm}/inertia_parameters.yaml"
       visual_parameters_file="${cfg}/${aico1_arm}/visual_parameters.yaml"
@@ -304,8 +304,8 @@
       <xacro:property name="paired_base_joint" value="true" />
     </xacro:if>
-    <xacro:property name="paired_kin_left"
+    <xacro:property name="paired_kinematics_left"
       value="${'$(arg kinematics_parameters_file_left)' if '$(arg kinematics_parameters_file_left)' != ''
                else cfg + '/' + arm_left + '/default_kinematics.yaml'}" />
-    <xacro:property name="paired_kin_right"
+    <xacro:property name="paired_kinematics_right"
       value="${'$(arg kinematics_parameters_file_right)' if '$(arg kinematics_parameters_file_right)' != ''
                else cfg + '/' + arm_right + '/default_kinematics.yaml'}" />
@@ -314,5 +314,5 @@
       robot_sn="$(arg robot_sn_left)"
       joint_limits_parameters_file="${cfg}/${arm_left}/joint_limits.yaml"
-      kinematics_parameters_file="${paired_kin_left}"
+      kinematics_parameters_file="${paired_kinematics_left}"
       inertia_parameters_file="${cfg}/${arm_left}/inertia_parameters.yaml"
       visual_parameters_file="${cfg}/${arm_left}/visual_parameters.yaml"
@@ -329,5 +329,5 @@
       robot_sn="$(arg robot_sn_right)"
       joint_limits_parameters_file="${cfg}/${arm_right}/joint_limits.yaml"
-      kinematics_parameters_file="${paired_kin_right}"
+      kinematics_parameters_file="${paired_kinematics_right}"
       inertia_parameters_file="${cfg}/${arm_right}/inertia_parameters.yaml"
       visual_parameters_file="${cfg}/${arm_right}/visual_parameters.yaml"
@@ -340,5 +340,4 @@
       base_xyz="${paired_right_xyz}"
       base_rpy="${paired_right_rpy}" />
-    <!-- One interface spanning both robots plus any external axis joints. -->
   </xacro:if>
 </robot>

Commit message: Update dual-arm setup robot kinematics parameter files (#34)

File: urdf/flexiv.urdf.xacro (robot description, xacro)
@@ -27,6 +27,6 @@
   <xacro:arg name="joint_limits_parameters_file"
     default="$(find flexiv_description)/config/$(arg robot_type)/joint_limits.yaml" />
-  <xacro:arg name="kinematics_parameters_file"
-    default="$(find flexiv_description)/config/$(arg robot_type)/default_kinematics.yaml" />
+  <!-- Empty means 'use the arm's default_kinematics.yaml'. -->
+  <xacro:arg name="kinematics_parameters_file" default="" />
   <xacro:arg name="inertia_parameters_file"
     default="$(find flexiv_description)/config/$(arg robot_type)/inertia_parameters.yaml" />
@@ -54,4 +54,7 @@
   <xacro:arg name="load_mounted_ft_sensor_left" default="false" />
   <xacro:arg name="load_mounted_ft_sensor_right" default="false" />
+  <!-- Empty means 'use the arm's default_kinematics.yaml'. -->
+  <xacro:arg name="kinematics_parameters_file_left" default="" />
+  <xacro:arg name="kinematics_parameters_file_right" default="" />
   <!-- Boolean flags for dispatch -->
   <xacro:property name="robot_type_str" value="$(arg robot_type)" />
@@ -80,9 +83,12 @@
   <xacro:if value="${is_single}">
     <xacro:property name="mounting" value="${xacro.load_yaml('$(arg mounting_file)')}" />
+    <xacro:property name="single_kinematics"
+      value="${'$(arg kinematics_parameters_file)' if '$(arg kinematics_parameters_file)' != ''
+               else cfg + '/' + robot_type_str + '/default_kinematics.yaml'}" />
     <xacro:flexiv_robot
       robot_type="$(arg robot_type)"
       robot_sn="$(arg robot_sn)"
       joint_limits_parameters_file="$(arg joint_limits_parameters_file)"
-      kinematics_parameters_file="$(arg kinematics_parameters_file)"
+      kinematics_parameters_file="${single_kinematics}"
       inertia_parameters_file="$(arg inertia_parameters_file)"
       visual_parameters_file="$(arg visual_parameters_file)"
@@ -101,4 +107,8 @@
     <!-- Each arm of a dual-arm product is an Enlight-L: reuse its config + meshes for both arms. -->
     <xacro:property name="arm_cfg" value="$(find flexiv_description)/config/Enlight-L" />
+    <!-- Kinematics are per-robot and live in this product's own file, one section per arm. -->
+    <xacro:property name="ll_kinematics_file"
+      value="${'$(arg kinematics_parameters_file)' if '$(arg kinematics_parameters_file)' != ''
+               else cfg + '/Enlight-LL/default_kinematics.yaml'}" />
     <!-- Left arm: owns the shared world link + its base joint. -->
     <xacro:flexiv_robot
@@ -106,5 +116,6 @@
       robot_sn="$(arg robot_sn)"
       joint_limits_parameters_file="${arm_cfg}/joint_limits.yaml"
-      kinematics_parameters_file="${arm_cfg}/default_kinematics.yaml"
+      kinematics_parameters_file="${ll_kinematics_file}"
+      kinematics_section="ARM_1"
       inertia_parameters_file="${arm_cfg}/inertia_parameters.yaml"
       visual_parameters_file="${arm_cfg}/visual_parameters.yaml"
@@ -123,5 +134,6 @@
       robot_sn="$(arg robot_sn)"
       joint_limits_parameters_file="${arm_cfg}/joint_limits.yaml"
-      kinematics_parameters_file="${arm_cfg}/default_kinematics.yaml"
+      kinematics_parameters_file="${ll_kinematics_file}"
+      kinematics_section="ARM_2"
       inertia_parameters_file="${arm_cfg}/inertia_parameters.yaml"
       visual_parameters_file="${arm_cfg}/visual_parameters.yaml"
@@ -144,6 +156,10 @@
     <xacro:include filename="$(find flexiv_description)/urdf/common/mico_core.xacro" />
     <xacro:property name="arm_cfg" value="$(find flexiv_description)/config/Enlight-L" />
+    <xacro:property name="mico_core_kin"
+      value="${'$(arg kinematics_parameters_file)' if '$(arg kinematics_parameters_file)' != ''
+               else cfg + '/MICO-Core/default_kinematics.yaml'}" />
     <xacro:mico_core
       robot_sn="$(arg robot_sn)"
+      kinematics_parameters_file="${mico_core_kin}"
       load_gripper="$(arg load_gripper)"
       gripper_name="$(arg gripper_name)"
@@ -155,6 +171,10 @@
     <xacro:include filename="$(find flexiv_description)/urdf/common/mico_plus.xacro" />
     <xacro:property name="arm_cfg" value="$(find flexiv_description)/config/Enlight-L" />
+    <xacro:property name="mico_plus_kin"
+      value="${'$(arg kinematics_parameters_file)' if '$(arg kinematics_parameters_file)' != ''
+               else cfg + '/MICO-Plus/default_kinematics.yaml'}" />
     <xacro:mico_plus
       robot_sn="$(arg robot_sn)"
+      kinematics_parameters_file="${mico_plus_kin}"
       load_gripper="$(arg load_gripper)"
       gripper_name="$(arg gripper_name)"
@@ -166,6 +186,10 @@
     <xacro:include filename="$(find flexiv_description)/urdf/common/mico_ultra.xacro" />
     <xacro:property name="arm_cfg" value="$(find flexiv_description)/config/Enlight-L" />
+    <xacro:property name="mico_ultra_kin"
+      value="${'$(arg kinematics_parameters_file)' if '$(arg kinematics_parameters_file)' != ''
+               else cfg + '/MICO-Ultra/default_kinematics.yaml'}" />
     <xacro:mico_ultra
       robot_sn="$(arg robot_sn)"
+      kinematics_parameters_file="${mico_ultra_kin}"
       load_gripper="$(arg load_gripper)"
       gripper_name="$(arg gripper_name)"
@@ -203,9 +227,12 @@
         mesh_prefix_path="package://flexiv_description/" />
     </xacro:if>
+    <xacro:property name="aico1_kinematics"
+      value="${'$(arg kinematics_parameters_file)' if '$(arg kinematics_parameters_file)' != ''
+               else cfg + '/' + aico1_arm + '/default_kinematics.yaml'}" />
     <xacro:flexiv_robot
       robot_type="${aico1_arm}"
       robot_sn="$(arg robot_sn)"
       joint_limits_parameters_file="${cfg}/${aico1_arm}/joint_limits.yaml"
-      kinematics_parameters_file="${cfg}/${aico1_arm}/default_kinematics.yaml"
+      kinematics_parameters_file="${aico1_kinematics}"
       inertia_parameters_file="${cfg}/${aico1_arm}/inertia_parameters.yaml"
       visual_parameters_file="${cfg}/${aico1_arm}/visual_parameters.yaml"
@@ -295,9 +322,15 @@
       <xacro:property name="paired_base_joint" value="true" />
     </xacro:if>
+    <xacro:property name="paired_kinematics_left"
+      value="${'$(arg kinematics_parameters_file_left)' if '$(arg kinematics_parameters_file_left)' != ''
+               else cfg + '/' + arm_left + '/default_kinematics.yaml'}" />
+    <xacro:property name="paired_kinematics_right"
+      value="${'$(arg kinematics_parameters_file_right)' if '$(arg kinematics_parameters_file_right)' != ''
+               else cfg + '/' + arm_right + '/default_kinematics.yaml'}" />
     <xacro:flexiv_robot
       robot_type="${arm_left}"
       robot_sn="$(arg robot_sn_left)"
       joint_limits_parameters_file="${cfg}/${arm_left}/joint_limits.yaml"
-      kinematics_parameters_file="${cfg}/${arm_left}/default_kinematics.yaml"
+      kinematics_parameters_file="${paired_kinematics_left}"
       inertia_parameters_file="${cfg}/${arm_left}/inertia_parameters.yaml"
       visual_parameters_file="${cfg}/${arm_left}/visual_parameters.yaml"
@@ -314,5 +347,5 @@
       robot_sn="$(arg robot_sn_right)"
       joint_limits_parameters_file="${cfg}/${arm_right}/joint_limits.yaml"
-      kinematics_parameters_file="${cfg}/${arm_right}/default_kinematics.yaml"
+      kinematics_parameters_file="${paired_kinematics_right}"
       inertia_parameters_file="${cfg}/${arm_right}/inertia_parameters.yaml"
       visual_parameters_file="${cfg}/${arm_right}/visual_parameters.yaml"
@@ -325,5 +358,4 @@
       base_xyz="${paired_right_xyz}"
       base_rpy="${paired_right_rpy}" />
-    <!-- One interface spanning both robots plus any external axis joints. -->
   </xacro:if>
 </robot>

Commit message: Feature/Add AICO2 external axis types (#36)

File: urdf/flexiv.urdf.xacro (robot description, xacro)
@@ -13,5 +13,6 @@
     Two paired robots (robot_sn_left + robot_sn_right, 'arm_type_left/right'):
       Rizon-Dual   two arms on a shared mount, no external axis
-      AICO2-4-V1, AICO2-4-V2, AICO2-10-V1
+      AICO2-4-V1, AICO2-4-V2, AICO2-4-D3, AICO2-4E-D1, AICO2-4U-D1
+      AICO2-10-V1, AICO2-10-D2, AICO2-10E-D1, AICO2-10U-D1
   -->
   <xacro:arg name="robot_type" default="Enlight-L" />
@@ -66,6 +67,8 @@
   <xacro:property name="is_dual" value="${is_enlight_ll or is_mico}" />
   <xacro:property name="is_aico1" value="${robot_type_str in ['AICO1-4-V1', 'AICO1-4-V2']}" />
-  <xacro:property name="is_aico2"
-    value="${robot_type_str in ['AICO2-4-V1', 'AICO2-4-V2', 'AICO2-10-V1']}" />
+  <xacro:property name="aico2_types"
+    value="${['AICO2-4-V1', 'AICO2-4-V2', 'AICO2-4-D3', 'AICO2-4E-D1', 'AICO2-4U-D1',
+              'AICO2-10-V1', 'AICO2-10-D2', 'AICO2-10E-D1', 'AICO2-10U-D1']}" />
+  <xacro:property name="is_aico2" value="${robot_type_str in aico2_types}" />
   <xacro:property name="is_rizon_dual" value="${robot_type_str == 'Rizon-Dual'}" />
   <!-- 'Paired' means two robots with two serial numbers, as opposed to one robot
@@ -248,22 +251,22 @@
        one robot with two arms on a single robot_sn. -->
   <xacro:if value="${is_paired}">
-    <!-- AICO2-10-V1 carries two Rizon10; the -4- variants carry a Rizon4 / Rizon4R
-         mirrored pair, which is also the default for a plain Rizon-Dual. -->
-    <xacro:property name="paired_default_left"
-      value="${'Rizon10' if robot_type_str == 'AICO2-10-V1' else 'Rizon4'}" />
+    <!-- The AICO2-10 variants carry two Rizon10; the AICO2-4 ones carry a Rizon4 /
+         Rizon4R mirrored pair, which is also the default for a plain Rizon-Dual. -->
+    <xacro:property name="is_aico2_10" value="${robot_type_str.startswith('AICO2-10')}" />
+    <xacro:property name="paired_default_left" value="${'Rizon10' if is_aico2_10 else 'Rizon4'}" />
     <xacro:property name="paired_default_right"
-      value="${'Rizon10R' if robot_type_str == 'AICO2-10-V1' else 'Rizon4R'}" />
+      value="${'Rizon10R' if is_aico2_10 else 'Rizon4R'}" />
     <xacro:property name="arm_left"
       value="${'$(arg arm_type_left)' if '$(arg arm_type_left)' != '' else paired_default_left}" />
     <xacro:property name="arm_right"
       value="${'$(arg arm_type_right)' if '$(arg arm_type_right)' != '' else paired_default_right}" />
-    <xacro:if value="${robot_type_str in ['AICO2-4-V1', 'AICO2-4-V2']}">
+    <xacro:if value="${is_aico2 and not is_aico2_10}">
       <xacro:unless value="${arm_left in ['Rizon4', 'Rizon4s', 'Rizon4R'] and arm_right in ['Rizon4', 'Rizon4s', 'Rizon4R']}">
         ${xacro.warning(robot_type_str + ' carries Rizon4-class arms. You selected ' + arm_left + ' and ' + arm_right + '.')}
       </xacro:unless>
     </xacro:if>
-    <xacro:if value="${robot_type_str == 'AICO2-10-V1'}">
+    <xacro:if value="${is_aico2_10}">
       <xacro:unless value="${arm_left in ['Rizon10', 'Rizon10R'] and arm_right in ['Rizon10', 'Rizon10R']}">
-        ${xacro.warning('AICO2-10-V1 carries Rizon10-class arms. You selected ' + arm_left + ' and ' + arm_right + '.')}
+        ${xacro.warning(robot_type_str + ' carries Rizon10-class arms. You selected ' + arm_left + ' and ' + arm_right + '.')}
       </xacro:unless>
     </xacro:if>
@@ -280,5 +283,11 @@
       <xacro:include filename="$(find flexiv_description)/urdf/common/aico2_4_v1.xacro" />
       <xacro:include filename="$(find flexiv_description)/urdf/common/aico2_4_v2.xacro" />
+      <xacro:include filename="$(find flexiv_description)/urdf/common/aico2_4_d3.xacro" />
+      <xacro:include filename="$(find flexiv_description)/urdf/common/aico2_4e_d1.xacro" />
+      <xacro:include filename="$(find flexiv_description)/urdf/common/aico2_4u_d1.xacro" />
       <xacro:include filename="$(find flexiv_description)/urdf/common/aico2_10_v1.xacro" />
+      <xacro:include filename="$(find flexiv_description)/urdf/common/aico2_10_d2.xacro" />
+      <xacro:include filename="$(find flexiv_description)/urdf/common/aico2_10e_d1.xacro" />
+      <xacro:include filename="$(find flexiv_description)/urdf/common/aico2_10u_d1.xacro" />
       <joint name="world_to_platform" type="fixed">
         <parent link="world" />
@@ -286,19 +295,9 @@
         <origin xyz="0 0 0" rpy="0 0 0" />
       </joint>
-      <xacro:if value="${robot_type_str == 'AICO2-4-V1'}">
-        <xacro:aico2_4_v1 prefix="$(arg external_axis_prefix)"
-          left_arm_prefix="${prefix_left}" right_arm_prefix="${prefix_right}"
-          mesh_prefix_path="package://flexiv_description/" />
-      </xacro:if>
-      <xacro:if value="${robot_type_str == 'AICO2-4-V2'}">
-        <xacro:aico2_4_v2 prefix="$(arg external_axis_prefix)"
-          left_arm_prefix="${prefix_left}" right_arm_prefix="${prefix_right}"
-          mesh_prefix_path="package://flexiv_description/" />
-      </xacro:if>
-      <xacro:if value="${robot_type_str == 'AICO2-10-V1'}">
-        <xacro:aico2_10_v1 prefix="$(arg external_axis_prefix)"
-          left_arm_prefix="${prefix_left}" right_arm_prefix="${prefix_right}"
-          mesh_prefix_path="package://flexiv_description/" />
-      </xacro:if>
+      <!-- Every AICO2 macro is named after its robot type and takes the same
+           parameters, so the selected one can be called by name. -->
+      <xacro:call macro="${external_axis_type}" prefix="$(arg external_axis_prefix)"
+        left_arm_prefix="${prefix_left}" right_arm_prefix="${prefix_right}"
+        mesh_prefix_path="package://flexiv_description/" />
       <xacro:property name="paired_left_xyz" value="0.0 0.0 0.0" />
       <xacro:property name="paired_left_rpy" value="0.0 0.0 0.0" />
